File: Hardware/VariometerV2.sch (KiCad schematic (older format))
At the start: 5 parts

Commit message: Fast fertig
Parts:
- added AE?: Antenna, symbol Device:Antenna
- added C?: 4.7uF, symbol Device:C_Small
- added C? (x11): 100nF, symbol Device:C_Small
- added C? (x2): 1uF, symbol Device:C_Small
- added C?: 10nF, symbol Device:C_Small
- added C? (x2): 8 pF, symbol Device:C_Small
- added C? (x3): 0.1uF, symbol Device:C_Small
- added C?: 0.1 uF, symbol Device:C_Small
- added C?: 100n, symbol Device:C_Small
- added C? (x4): 10uF, symbol Device:C_Small
- added C?: 100 nF, symbol Device:C_Small
- added C?: 2.2 uF, symbol Device:C_Small
- added C?: 2.2uF, symbol Device:C_Small
- added D?: RE, symbol Device:LED_Small
- added D?: BL, symbol Device:LED_Small
- added D?: GR, symbol Device:LED_Small
- added D? (x2): B5819W SL, symbol Device:D_Schottky_Small
- added D? (x2): RCLAMP0521P-N, symbol Device:D_TVS_ALT
- added D? (x4): TVS, symbol Device:D_TVS_ALT
- added F?: 500mA, symbol Device:Polyfuse_Small
- added FB?: 600 @ 600MHz, symbol Device:Ferrite_Bead_Small
- added FB?: 100 @ 100 MHz, symbol Device:Ferrite_Bead_Small
- added H?: LED_CHRG+, symbol Mechanical:MountingHole_Pad
- added H?: LED_CHRG-, symbol Mechanical:MountingHole_Pad
- added H?: LED_STBY+, symbol Mechanical:MountingHole_Pad
- added H?: LED_STBY-, symbol Mechanical:MountingHole_Pad
- added IC?: DW01A-G, SOT95P280X135-6N, symbol VariometerV2-rescue:DW01A-G-DW01A-G
- added IC?: TP4056, symbol Vario2_Library:TP4056
- added J?: SWD, symbol Connector_Generic:Conn_02x05_Odd_Even
- added J?: Conn_01x04, symbol Connector_Generic:Conn_01x04
- added J?: USB_B_Micro, symbol Connector:USB_B_Micro
- added J?: Screw_Terminal_01x02, symbol Connector:Screw_Terminal_01x02
- added J?: Micro_SD_Card_Det, symbol Connector:Micro_SD_Card_Det
- added L?: 39nF, symbol Device:L_Small
- added L?: 47nH, symbol Device:L_Small
- added Q? (x2): AO3400A, Package_TO_SOT_SMD:SOT-23, symbol Transistor_FET:AO3400A
- added R? (x2): 1.2k, symbol Device:R_Small
- added R?: 47, symbol Device:R_Small
- added R? (x5): 1k, symbol Device:R_Small
- added R? (x3): 2.2k, symbol Device:R_Small
- added R? (x4): 22, symbol Device:R_Small
- added R?: 100, symbol Device:R_Small
- added R?: 51k, symbol Device:R_Small
- added R?: 27k, symbol Device:R_Small
- added R?: 1.5k, symbol Device:R_Small
- added R? (x5): 10k, symbol Device:R_Small
- added R?: 100k, symbol Device:R_Small
- added R?: 1M, symbol Device:R_Small
- added U?: USBLC6-2SC6, Package_TO_SOT_SMD:SOT-23-6, symbol Power_Protection:USBLC6-2SC6
- added U?: BMI088, symbol Vario2_Library:BMI088
- added U?: E104-BT51, symbol Vario2_Library:E104-BT51
- added U?: TPS76801QDR, symbol Vario2_Library:TPS76801QDR
- added U?: MS5611-01BA, Package_LGA:LGA-8_3x5mm_P1.25mm, symbol Sensor_Pressure:MS5611-01BA
- added U?: ATGM336H-5N31, symbol Vario2_Library:ATGM336H-5N31
- added Y?: 16MHz, symbol Device:Crystal_GND24_Small
Connections:
- net labels added: +5V, ACC_INT, BATT+, BATT_CONN+, BATT_CONN-, BAT_ADC, BLE_DATA, BLE_LED, BLE_MODE, BLE_SLEEP, BLE_nRESET, DW01A_OC, DW01A_OD, ERROR_LED, GPS_LED, GPS_PPS, GYR_INT, I2C4_SCL, I2C4_SDA, IMU_ACC_CS, IMU_GYR_CS, PresSens_CS, SDCARD_DETECT, SD_CS, SPI1_MISO, SPI1_MOSI, SPI1_SCK, SPI2_MISO, SPI2_MOSI, SPI2_SCK, TP4056_CHRG, TP4056_STBY, USART2_RX, USART2_TX, USART6_RX, USART6_TX, USB_CONN_D+, USB_CONN_D-, VREF+
- net labels removed: BLE_RX, BLE_TX, GPS_RX, GPS_TX, IMU_MISO, IMU_MOSI, IMU_SCK, MS5611_MISO, MS5611_MOSI, MS5611_SCK, SDCARD_MISO, SDCARD_MOSI, SDCARD_SCK, VBATT_MSR
- wire segments 32 -> 344
- no-connect marks 0 -> 44
Other:
- note added: "Power"
- note added: "STM32 Microcontroller"
- moved on the sheet: C?, R?, SW?, U?

Commit message: Fast fertig
Parts:
- added Q?: AO3401A, Package_TO_SOT_SMD:SOT-23, symbol Transistor_FET:AO3401A
- added Q?: AO3400A, Package_TO_SOT_SMD:SOT-23, symbol Transistor_FET:AO3400A
- added R?: 1M, symbol Device:R_Small
- added R?: 33k, symbol Device:R_Small
- added R?: 10k, symbol Device:R_Small
- IC?: symbol Vario2_Library:TP4056 -> VariometerV2-rescue:TP4056-Vario2_Library
- U?: symbol Vario2_Library:BMI088 -> VariometerV2-rescue:BMI088-Vario2_Library
- U?: symbol Vario2_Library:E104-BT51 -> VariometerV2-rescue:E104-BT51-Vario2_Library
- U?: symbol Vario2_Library:TPS76801QDR -> VariometerV2-rescue:TPS76801QDR-Vario2_Library
- U?: symbol Vario2_Library:ATGM336H-5N31 -> VariometerV2-rescue:ATGM336H-5N31-Vario2_Library
Connections:
- net labels added: BAT_MS
- wire segments 344 -> 357
Changed lines of the file:
@@
 	5550 3800 5750 3800
 $Comp
-L Vario2_Library:TPS76801QDR U?
+L VariometerV2-rescue:TPS76801QDR-Vario2_Library U?
 U 1 1 61A53EF8
 P 4300 2950
@@
 	650  1800 2200 1800
 $Comp
-L Vario2_Library:TP4056 IC?
+L VariometerV2-rescue:TP4056-Vario2_Library IC?
 U 1 1 61A54DF9
 P 2200 1250
@@
 SPI1_SCK
 $Comp
-L Vario2_Library:BMI088 U?
+L VariometerV2-rescue:BMI088-Vario2_Library U?
 U 1 1 6198EA40
 P 8750 1550
@@
 Connection ~ 13250 1200
 $Comp
-L Vario2_Library:ATGM336H-5N31 U?
+L VariometerV2-rescue:ATGM336H-5N31-Vario2_Library U?
 U 1 1 620A5AC0
 P 11200 5200
@@
 	11800 4900 12150 4900
 $Comp
-L Vario2_Library:E104-BT51 U?
+L VariometerV2-rescue:E104-BT51-Vario2_Library U?
 U 1 1 619E049C
 P 6700 5650
@@
 Wire Wire Line
 	8600 5700 8600 5750
+Text GLabel 6150 2500 1    50   Input ~ 0
+BATT+
+$Comp
+L Device:R_Small R?
+U 1 1 619C2CC4
+P 6800 2600
+F 0 "R?" V 6700 2600 50  0000 C CNN
+F 1 "1M" H 6905 2600 50  0000 C CNN
+F 2 "" H 6800 2600 50  0001 C CNN
+F 3 "~" H 6800 2600 50  0001 C CNN
+	1    6800 2600
+	-1   0    0    1
+$EndComp
+$Comp
+L Device:R_Small R?
+U 1 1 619C3D54
+P 6400 3200
+F 0 "R?" V 6300 3200 50  0000 C CNN
+F 1 "10k" H 6505 3200 50  0000 C CNN
+F 2 "" H 6400 3200 50  0001 C CNN
+F 3 "~" H 6400 3200 50  0001 C CNN
+	1    6400 3200
+	-1   0    0    1
+$EndComp
+$Comp
+L Device:R_Small R?
+U 1 1 619C3321
+P 6400 3550
+F 0 "R?" V 6300 3550 50  0000 C CNN
+F 1 "33k" H 6505 3550 50  0000 C CNN
+F 2 "" H 6400 3550 50  0001 C CNN
+F 3 "~" H 6400 3550 50  0001 C CNN
+	1    6400 3550
+	-1   0    0    1
+$EndComp
+$Comp
+L Transistor_FET:AO3401A Q?
+U 1 1 619C5BA0
+P 6500 2800
+F 0 "Q?" H 6705 2754 50  0000 L CNN
+F 1 "AO3401A" H 6705 2845 50  0000 L CNN
+F 2 "Package_TO_SOT_SMD:SOT-23" H 6700 2725 50  0001 L CIN
+F 3 "http://www.aosmd.com/pdfs/datasheet/AO3401A.pdf" H 6500 2800 50  0001 L CNN
+	1    6500 2800
+	-1   0    0    1
+$EndComp
+$Comp
+L Transistor_FET:AO3400A Q?
+U 1 1 61AA11B0
+P 6900 3400
+F 0 "Q?" H 6750 3550 50  0000 L CNN
+F 1 "AO3400A" H 6600 3250 50  0000 L CNN
+F 2 "Package_TO_SOT_SMD:SOT-23" H 7100 3325 50  0001 L CIN
+F 3 "http://www.aosmd.com/pdfs/datasheet/AO3400A.pdf" H 6900 3400 50  0001 L CNN
+	1    6900 3400
+	-1   0    0    1
+$EndComp
+Wire Wire Line
+	6150 2500 6400 2500
+Wire Wire Line
+	6400 2500 6400 2600
+Wire Wire Line
+	6400 3000 6400 3100
+Wire Wire Line
+	6400 3300 6400 3350
+Text GLabel 6250 3350 0    50   Input ~ 0
+BAT_ADC
+Wire Wire Line
+	6250 3350 6400 3350
+Connection ~ 6400 3350
+Wire Wire Line
+	6400 3350 6400 3450
+Text GLabel 3050 10250 2    50   Input ~ 0
+BAT_MS
+Text GLabel 7100 3400 2    50   Input ~ 0
+BAT_MS
+Wire Wire Line
+	6400 2500 6800 2500
+Connection ~ 6400 2500
+Wire Wire Line
+	6800 2700 6800 2800
+Wire Wire Line
+	6700 2800 6800 2800
+Connection ~ 6800 2800
+Wire Wire Line
+	6800 2800 6800 3200
+$Comp
+L power:GND #PWR?
+U 1 1 61B744F6
+P 6800 3750
+F 0 "#PWR?" H 6800 3500 50  0001 C CNN
+F 1 "GND" H 6805 3577 50  0000 C CNN
+F 2 "" H 6800 3750 50  0001 C CNN
+F 3 "" H 6800 3750 50  0001 C CNN
+	1    6800 3750
+	1    0    0    -1
+$EndComp
+Wire Wire Line
+	6400 3650 6800 3650
+Wire Wire Line
+	6800 3650 6800 3600
+Wire Wire Line
+	6800 3650 6800 3750
+Connection ~ 6800 3650
 $EndSCHEMATC

Commit message: update
Parts:
- added C?: 1uF, symbol Device:C_Small
- added C?: 0.1uF, symbol Device:C_Small
- added C?: 10uF, symbol Device:C_Small
- added D?: B5819W SL, symbol Device:D_Schottky_Small
- added Q?: AO3401A, Package_TO_SOT_SMD:SOT-23, symbol Transistor_FET:AO3401A
- added Q?: AO3400A, Package_TO_SOT_SMD:SOT-23, symbol Transistor_FET:AO3400A
- added R?: 10k, symbol Device:R_Small
- added R? (x2): 100k, symbol Device:R_Small
- added R?: 300k, symbol Device:R_Small
- added SW?: SW_Push, symbol Switch:SW_Push
Connections:
- net labels added: POW_SW+, POW_UNSW+, SDMMC1_CK, SDMMC1_CMD, SDMMC1_D0, SDMMC1_D1, SDMMC1_D2, SDMMC1_D3, USART1_RX, USART1_TX
- net labels removed: USART6_RX, USART6_TX
- wire segments 357 -> 389
Other:
- note added: "AO340A: N-Channel Mosfet (acitve high)\nAO3401A: P-Channel Mosfet"
- note added: "Battery Charge/Protection"
- note added: "Battery Voltage Measure"
- note added: "LDO"
- note added: "ON/OFF CIRCUIT"
- moved on the sheet: C?, D?, F?, FB?, J?, L?, Q?, R?, U?

Commit message: Fertig
Parts:
- removed D?: RCLAMP0521P-N, symbol Device:D_TVS_ALT
- removed D? (x4): TVS, symbol Device:D_TVS_ALT
- removed H?: LED_CHRG+, symbol Mechanical:MountingHole_Pad
- removed H?: LED_CHRG-, symbol Mechanical:MountingHole_Pad
- removed H?: LED_STBY+, symbol Mechanical:MountingHole_Pad
- removed H?: LED_STBY-, symbol Mechanical:MountingHole_Pad
- removed R? (x4): 10k, symbol Device:R_Small
- removed R?: 1M, symbol Device:R_Small
- removed U?: USBLC6-2SC6, Package_TO_SOT_SMD:SOT-23-6, symbol Power_Protection:USBLC6-2SC6
- added J?: BUZZER_1, symbol Connector_Generic:Conn_01x01
- added J?: BUZZER_2, symbol Connector_Generic:Conn_01x01
- added J?: LED_CHRG+, symbol Connector_Generic:Conn_01x01
- added J?: LED_CHRG-, symbol Connector_Generic:Conn_01x01
- added J?: LED_STBY+, symbol Connector_Generic:Conn_01x01
- added J?: LED_STBY-, symbol Connector_Generic:Conn_01x01
- added Q? (x2): AO3400A, Package_TO_SOT_SMD:SOT-23, symbol Transistor_FET:AO3400A
- added Q? (x2): AO3401A, Package_TO_SOT_SMD:SOT-23, symbol Transistor_FET:AO3401A
- added R? (x9): 10k, symbol Device:R_Small
- added R?: 1M, symbol Device:R_Small
- added R?: 22, symbol Device:R_Small
- added R?: 100k, symbol Device:R_Small
- added U? (x3): SRV05-4, Package_TO_SOT_SMD:SOT-23-6, symbol Power_Protection:SRV05-4
- J?: value Screw_Terminal_01x02 -> BATT_CONN
Connections:
- net labels added: TIM1_CH1, TIM1_CH1N
- net labels removed: BUZZER_PWM, SPI2_SCK, USB_CONN_D+, USB_CONN_D-
- wire segments 389 -> 439
- no-connect marks 44 -> 47
Other:
- note added: "Analog Filtering"
- note added: "Bluetooth Low Energy"
- note added: "Boot Selection"
- note added: "Buzzer mit H-Bridge"
- note added: "Connectors"
- note added: "Ext. Crystal"
- note added: "GPS"
- note added: "I2C Pullups"
- note added: "IMU Sensor"
- note added: "LEDS"
- note added: "Micro SD Card"
- note added: "Power Filtering"
- note added: "Pressure Sensor"
- note added: "VREF+ Filtering"
- moved on the sheet: C?, D?, FB?, J?, L?, Q?, R?, U?

Commit message: f
Parts:
- removed AE?: Antenna, symbol Device:Antenna
- removed L?: 39nF, symbol Device:L_Small
- removed R?: 100k, symbol Device:R_Small
- added C?: 100nF, symbol Device:C_Small
- added D?: GREEN, symbol Device:LED_Small
- added FB?: 600 @ 100MHz, symbol Device:Ferrite_Bead_Small
- added J?: 5-1814832-1, TE_5-1814832-1, symbol 5-1814832-1:5-1814832-1
- added R?: 1.5k, symbol Device:R_Small
- added R? (x2): 22, symbol Device:R_Small
- added TP?: GND TP, symbol Connector:TestPoint
- added TP?: 3.3V TP, symbol Connector:TestPoint
- added U?: M24C64, symbol Vario2_Library:M24C64
- FB?: value 600 @ 600MHz -> 600 @ 100MHz
- FB?: value 100 @ 100 MHz -> 600 @ 100 MHz
Connections:
- net labels added: GPS_ON, I2C_GPS_SCL, I2C_GPS_SDA
- net labels removed: SD_CS, SPI2_MISO, SPI2_MOSI
- wire segments 439 -> 457
- no-connect marks 47 -> 85
Other:
- note added: "Power LED"
- note added: "Step-Down Converter (3.3V) LDO"
- note removed: "LDO"
- moved on the sheet: C?, J?, L?, Q?, R?, U?

Commit message: Schematic Finish
Parts:
- removed C?: 10uF, symbol Device:C_Small
- removed D?: RCLAMP0521P-N, symbol Device:D_TVS_ALT
- added C32: 10uF, symbol Device:C_Small
- added H1, H2, H3, H4: MountingHole_Pad, symbol Mechanical:MountingHole_Pad
- added R32, R39, R40: 10k, symbol Device:R_Small
- C31: renamed from C?; value 0.1uF -> 100nF
- F1: renamed from F?; value 500mA -> 700mA
- J12: renamed from J?; symbol 5-1814832-1:5-1814832-1 -> VariometerV2-rescue:5-1814832-1-5-1814832-1
- R20: renamed from R?; value 1.2k -> 22
- U8: renamed from U?; symbol Vario2_Library:M24C64 -> VariometerV2-rescue:M24C64-Vario2_Library
- gave numbers to parts that had none: 123
Connections:
- net +3V3: now also C32.1, R39.1, R40.2; no longer U4.5 (VP), U5.5 (VP)
- net +5V: now also R32.1; no longer U3.5 (VP)
- net GND: now also C32.2, H1.1, H2.1, H3.1, H4.1
- net BLE_LINK: now reaches U2.58 (PD11)
- net BLE_LINK: now also U7.19 (DIO_15_LINK)
- net 3.3V_SDCARD: now reaches C25.1, C26.1, FB3.2, J9.4 (VDD)
- net 3.3V_SDCARD: now also U5.6 (IO4)
- new net: R39.2, U4.5 (VP)
- new net: R40.1, U5.5 (VP)
- new net: R32.2, U3.5 (VP)
- no-connect marks 85 -> 84
Other:
- moved on the sheet: C31

Commit message: hg
Parts:
- removed FB1: 600 @ 100MHz, symbol Device:Ferrite_Bead_Small
- added JP1: Jumper_2_Open, symbol Jumper:Jumper_2_Open
- C1, C10, C11, C12, C13, C14, C15, C16, C17, C18, C19, C2, C25, C26, C27, C28, C29, C30, C31, C33, C35, C4, C5, C7: footprint (none) -> Capacitor_SMD:C_0402_1005Metric
- C20, C21, C32, C34, C6, C8, C9: footprint (none) -> Capacitor_SMD:C_0603_1608Metric
- C22, C23: value 8 pF -> 6pF; footprint (none) -> Capacitor_SMD:C_0603_1608Metric
- C24: value 100n -> 100nF; footprint (none) -> Capacitor_SMD:C_0402_1005Metric
- C3: footprint (none) -> Capacitor_SMD:C_0201_0603Metric
- D1, D2, D3: footprint (none) -> Diode_SMD:D_SOD-123
- D4, D5, D6, D7: footprint (none) -> LED_SMD:LED_0603_1608Metric
- F1: footprint (none) -> Fuse:Fuse_0603_1608Metric
- FB1: renamed from FB2; footprint (none) -> Inductor_SMD:L_0805_2012Metric
- FB2: renamed from FB3; footprint (none) -> Inductor_SMD:L_0805_2012Metric
- H1, H2, H3, H4: footprint (none) -> MountingHole:MountingHole_2.5mm_Pad_Via
- IC1: footprint (none) -> Hardware:SOIC127P600X175-9N
- IC2: footprint SOT95P280X135-6N -> Hardware:SOT95P280X135-6N
- J1, J2, J3, J4: footprint (none) -> Connector_Wire:SolderWire-0.1sqmm_1x01_D0.4mm_OD1mm
- J5: footprint (none) -> TerminalBlock_Phoenix:TerminalBlock_Phoenix_PT-1,5-2-3.5-H_1x02_P3.50mm_Horizontal
- J6: footprint (none) -> Connector_Molex:Molex_PicoBlade_53048-0410_1x04_P1.25mm_Horizontal
- J7: footprint (none) -> Connector_PinSocket_1.27mm:PinSocket_2x05_P1.27mm_Horizontal
- R20: value 22 -> 47
Connections:
- net POW_SW+: now also JP1.2 (B)
- net POW_UNSW+: now also D1.1 (K), D2.1 (K), JP1.1 (A)

Commit message: PCb
Parts:
- added SW3: SW_Push, symbol Switch:SW_Push
Connections:
- net +3V3: now also SW3.2
- net Button_Input: now reaches U2.97 (PE0)
- net Button_Input: now also SW3.1
- no-connect marks 84 -> 83
Changed lines of the file:
@@
 Wire Wire Line
 	4300 7450 4300 7700
-NoConn ~ 1350 7150
 NoConn ~ 1350 7250
 NoConn ~ 1350 7350
@@
 Wire Wire Line
 	1650 2950 2150 2950
+Text GLabel 1350 7150 0    50   Input ~ 0
+Button_Input
+$Comp
+L power:+3.3V #PWR0181
+U 1 1 61C02EA8
+P 7450 7750
+F 0 "#PWR0181" H 7450 7600 50  0001 C CNN
+F 1 "+3.3V" H 7450 7900 50  0000 C CNN
+F 2 "" H 7450 7750 50  0001 C CNN
+F 3 "" H 7450 7750 50  0001 C CNN
+	1    7450 7750
+	1    0    0    -1
+$EndComp
+$Comp
+L Switch:SW_Push SW3
+U 1 1 61C035A8
+P 7450 7950
+F 0 "SW3" H 7450 8235 50  0000 C CNN
+F 1 "SW_Push" H 7450 8144 50  0000 C CNN
+F 2 "" H 7450 8150 50  0001 C CNN
+F 3 "~" H 7450 8150 50  0001 C CNN
+	1    7450 7950
+	0    -1   -1   0
+$EndComp
+Text GLabel 7450 8350 0    50   Input ~ 0
+Button_Input
+Wire Wire Line
+	7450 8350 7450 8150
 $EndSCHEMATC
