File: Hardware/VariometerV2.sch (KiCad schematic (older format))
At the start: 137 parts, among them IC1 TP4056, IC2 DW01A-G, J1 LED_CHRG+, J10 BUZZER_1, J11 BUZZER_2, J12 5-1814832-1, J2 LED_CHRG-, J3 LED_STBY+, J4 LED_STBY-, J5 BATT_CONN, J6 Conn_01x04, J7 SWD, J8 USB_B_Micro, J9 Micro_SD_Card_Det, Q1 AO3400A, Q10 AO3400A, Q2 AO3400A, Q3 AO3401A, Q4 AO3400A, Q5 AO3401A, Q6 AO3400A, Q7 AO3401A, Q8 AO3400A, Q9 AO3401A, SW1 SW_Push, SW2 SW_SPDT, SW3 SW_Push, U1 TPS76801QDR, U10 MS5611-01BA, U2 STM32F745VET6, U3 SRV05-4, U4 SRV05-4, U5 SRV05-4, U6 BMI088, U7 E104-BT51, U8 M24C64, U9 ATGM336H-5N31, Y1 16MHz

Commit message: PCB fast fertig
Parts:
- removed J1: LED_CHRG+, Connector_Wire:SolderWire-0.1sqmm_1x01_D0.4mm_OD1mm, symbol Connector_Generic:Conn_01x01
- removed J10: BUZZER_1, symbol Connector_Generic:Conn_01x01
- removed J11: BUZZER_2, symbol Connector_Generic:Conn_01x01
- removed J2: LED_CHRG-, Connector_Wire:SolderWire-0.1sqmm_1x01_D0.4mm_OD1mm, symbol Connector_Generic:Conn_01x01
- removed J3: LED_STBY+, Connector_Wire:SolderWire-0.1sqmm_1x01_D0.4mm_OD1mm, symbol Connector_Generic:Conn_01x01
- removed J4: LED_STBY-, Connector_Wire:SolderWire-0.1sqmm_1x01_D0.4mm_OD1mm, symbol Connector_Generic:Conn_01x01
- removed J5: BATT_CONN, TerminalBlock_Phoenix:TerminalBlock_Phoenix_PT-1,5-2-3.5-H_1x02_P3.50mm_Horizontal, symbol Connector:Screw_Terminal_01x02
- removed J8: USB_B_Micro, symbol Connector:USB_B_Micro
- removed J9: Micro_SD_Card_Det, symbol Connector:Micro_SD_Card_Det
- added J1: LED_CHRG, Connector_PinHeader_2.00mm:PinHeader_2x01_P2.00mm_Vertical, symbol Connector_Generic:Conn_02x01
- added J2: LED_STBY, Connector_PinHeader_2.00mm:PinHeader_2x01_P2.00mm_Vertical, symbol Connector_Generic:Conn_02x01
- added J3: Conn_01x02_Male, Connector_PinSocket_2.54mm:PinSocket_1x02_P2.54mm_Vertical, symbol Connector:Conn_01x02_Male
- added J6: USB3135-30-A, USB313530A, symbol SamacSys_Parts:USB3135-30-A
- added J7: TF-15X15, Hardware:TF15X15, symbol SamacSys_Parts:TF-15X15
- added J8: Conn_02x01, Connector_PinHeader_2.00mm:PinHeader_2x01_P2.00mm_Vertical, symbol Connector_Generic:Conn_02x01
- H1, H2, H3, H4: footprint MountingHole:MountingHole_2.5mm_Pad_Via -> MountingHole:MountingHole_2.2mm_M2_DIN965_Pad
- J4: renamed from J6; footprint Connector_Molex:Molex_PicoBlade_53048-0410_1x04_P1.25mm_Horizontal -> Connector_PinHeader_1.27mm:PinHeader_1x04_P1.27mm_Vertical
- J5: renamed from J7; footprint Connector_PinSocket_1.27mm:PinSocket_2x05_P1.27mm_Horizontal -> Connector_PinHeader_1.27mm:PinHeader_2x05_P1.27mm_Vertical
- J9: renamed from J12; footprint TE_5-1814832-1 -> Hardware:5-1814832-1
- JP1: footprint (none) -> TestPoint:TestPoint_2Pads_Pitch2.54mm_Drill0.8mm
- L1: footprint (none) -> Inductor_SMD:L_0603_1608Metric
- R1, R10, R11, R12, R13, R2, R21, R22, R23, R3, R4, R5, R6, R7, R8, R9: footprint (none) -> Resistor_SMD:R_0603_1608Metric
- R14, R15, R16, R17, R18, R19, R24, R25, R26, R27, R28, R29, R30, R31, R32, R33, R34, R35, R36, R37, R38, R39, R40, R41, R42, R43, R44, R45, R46: footprint (none) -> Resistor_SMD:R_0402_1005Metric
- R20: footprint (none) -> Resistor_SMD:R_0805_2012Metric
- SW1, SW3: footprint (none) -> Connector_Wire:SolderWire-0.25sqmm_1x02_P4.2mm_D0.65mm_OD1.7mm
- SW2: footprint (none) -> Hardware:MINISPDTSW
- TP1, TP2: footprint (none) -> Connector_Pin:Pin_D0.7mm_L6.5mm_W1.8mm_FlatFork
- U1: footprint (none) -> Hardware:SOIC127P600X175-8N
- U6: footprint (none) -> Hardware:BMI088
- U7: footprint (none) -> Hardware:WIRELM-SMD_E180-ZG120A
- U8: footprint (none) -> Package_SO:SOIC-8_3.9x4.9mm_P1.27mm
- U9: footprint (none) -> Hardware:ATGM336H5N31
- Y1: footprint (none) -> Crystal:Crystal_SMD_3225-4Pin_3.2x2.5mm
Connections:
- wire segments 464 -> 474
- no-connect marks 83 -> 84
Other:
- moved on the sheet: D1, D2, F1, R32, U3

Commit message: PCB fertig
Parts:
- C3: footprint Capacitor_SMD:C_0201_0603Metric -> Capacitor_SMD:C_0402_1005Metric
- F1: value 700mA -> 1A
- J6: footprint USB313530A -> Hardware:USB313530A; symbol SamacSys_Parts:USB3135-30-A -> VariometerV2-rescue:USB3135-30-A-SamacSys_Parts
- J7: symbol SamacSys_Parts:TF-15X15 -> VariometerV2-rescue:TF-15X15-SamacSys_Parts
Connections:
- wire segments 474 -> 472
Changed lines of the file:
@@
 F 0 "C3" H 6450 1650 50  0000 L CNN
 F 1 "10uF" H 6450 1550 50  0000 L CNN
-F 2 "Capacitor_SMD:C_0201_0603Metric" H 6400 1500 50  0001 C CNN
+F 2 "Capacitor_SMD:C_0402_1005Metric" H 6400 1500 50  0001 C CNN
 F 3 "~" H 6400 1500 50  0001 C CNN
 	1    6400 1500
@@
 P 1750 2950
 F 0 "F1" V 1650 2950 50  0000 C CNN
-F 1 "700mA" V 1850 2950 50  0000 C CNN
+F 1 "1A" V 1850 2950 50  0000 C CNN
 F 2 "Fuse:Fuse_0603_1608Metric" H 1800 2750 50  0001 L CNN
 F 3 "~" H 1750 2950 50  0001 C CNN
@@
 $EndComp
 Wire Wire Line
-	13200 2550 14100 2550
+	13200 2550 13450 2550
 Wire Wire Line
 	13850 1650 13850 1450
@@
 Wire Wire Line
 	13400 4050 13450 4050
-Wire Wire Line
-	13450 4050 13450 3050
-Wire Wire Line
-	13450 3050 12800 3050
-Wire Wire Line
-	12800 3050 12800 2550
-Wire Wire Line
-	12800 2550 13000 2550
-Wire Wire Line
-	12550 2550 12800 2550
-Connection ~ 12800 2550
 Wire Wire Line
 	12550 2750 13550 2750
@@
 $EndComp
 $Comp
-L SamacSys_Parts:TF-15X15 J7
+L VariometerV2-rescue:TF-15X15-SamacSys_Parts J7
 U 1 1 61E50C19
 P 14100 2150
@@
 	7150 5150 7450 5150
 $Comp
-L SamacSys_Parts:USB3135-30-A J6
+L VariometerV2-rescue:USB3135-30-A-SamacSys_Parts J6
 U 1 1 622240A6
 P 5300 9800
 F 0 "J6" H 5750 9135 50  0000 C CNN
 F 1 "USB3135-30-A" H 5750 9226 50  0000 C CNN
-F 2 "USB313530A" H 6050 9900 50  0001 L CNN
+F 2 "Hardware:USB313530A" H 6050 9900 50  0001 L CNN
 F 3 "https://gct.co/Files/Drawings/USB3135.pdf?v=9f17ad4b-b3da-4f3d-b4d5-eb94b5d526c5" H 6050 9800 50  0001 L CNN
 F 4 "GCT (GLOBAL CONNECTOR TECHNOLOGY) - USB3135-30-A - USB Connector, Micro USB Type B, USB 2.0, Receptacle, 5 Ways, Surface Mount, Right Angle" H 6050 9700 50  0001 L CNN "Description"
@@
 	1    0    0    -1
 $EndComp
+Wire Wire Line
+	12550 2550 13000 2550
+Wire Wire Line
+	13450 2550 13450 4050
+Connection ~ 13450 2550
+Wire Wire Line
+	13450 2550 14100 2550
 $EndSCHEMATC

Commit message: update
Parts:
- J3: footprint Connector_PinSocket_2.54mm:PinSocket_1x02_P2.54mm_Vertical -> Connector_PinHeader_2.54mm:PinHeader_1x02_P2.54mm_Vertical
Changed lines of the file:
@@
 F 0 "J3" H 5772 6982 50  0000 R CNN
 F 1 "Conn_01x02_Male" H 5772 7073 50  0000 R CNN
-F 2 "Connector_PinSocket_2.54mm:PinSocket_1x02_P2.54mm_Vertical" H 5800 7100 50  0001 C CNN
+F 2 "Connector_PinHeader_2.54mm:PinHeader_1x02_P2.54mm_Vertical" H 5800 7100 50  0001 C CNN
 F 3 "~" H 5800 7100 50  0001 C CNN
 	1    5800 7100

Commit message: Fertig
Parts:
- R46: footprint Resistor_SMD:R_0402_1005Metric -> Resistor_SMD:R_0805_2012Metric
Changed lines of the file:
@@
 F 0 "R46" H 14950 6300 50  0000 C CNN
 F 1 "100k" H 15200 6300 50  0000 C CNN
-F 2 "Resistor_SMD:R_0402_1005Metric" H 15050 6300 50  0001 C CNN
+F 2 "Resistor_SMD:R_0805_2012Metric" H 15050 6300 50  0001 C CNN
 F 3 "~" H 15050 6300 50  0001 C CNN
 	1    15050 6300

Commit message: esp32 start
Parts:
- removed C10, C11, C12, C13, C14, C15, C19, C24, C30, C31: 100nF, Capacitor_SMD:C_0402_1005Metric, symbol Device:C_Small
- removed C16, C18: 1uF, Capacitor_SMD:C_0402_1005Metric, symbol Device:C_Small
- removed C17: 10nF, Capacitor_SMD:C_0402_1005Metric, symbol Device:C_Small
- removed C20, C21: 2.2uF, Capacitor_SMD:C_0603_1608Metric, symbol Device:C_Small
- removed C22, C23: 6pF, Capacitor_SMD:C_0603_1608Metric, symbol Device:C_Small
- removed C32: 10uF, Capacitor_SMD:C_0603_1608Metric, symbol Device:C_Small
- removed C9: 4.7uF, Capacitor_SMD:C_0603_1608Metric, symbol Device:C_Small
- removed D5: RE, LED_SMD:LED_0603_1608Metric, symbol Device:LED_Small
- removed D6: BL, LED_SMD:LED_0603_1608Metric, symbol Device:LED_Small
- removed D7: GR, LED_SMD:LED_0603_1608Metric, symbol Device:LED_Small
- removed FB1: 600 @ 100MHz, Inductor_SMD:L_0805_2012Metric, symbol Device:Ferrite_Bead_Small
- removed R18: 47, Resistor_SMD:R_0402_1005Metric, symbol Device:R_Small
- removed R19: 10k, Resistor_SMD:R_0402_1005Metric, symbol Device:R_Small
- removed R20: 47, Resistor_SMD:R_0805_2012Metric, symbol Device:R_Small
- removed R21, R22: 1k, Resistor_SMD:R_0603_1608Metric, symbol Device:R_Small
- removed R23: 2.2k, Resistor_SMD:R_0603_1608Metric, symbol Device:R_Small
- removed R24, R25: 2.2k, Resistor_SMD:R_0402_1005Metric, symbol Device:R_Small
- removed R31: 22, Resistor_SMD:R_0402_1005Metric, symbol Device:R_Small
- removed R46: 100k, Resistor_SMD:R_0805_2012Metric, symbol Device:R_Small
- removed SW2: SW_SPDT, Hardware:MINISPDTSW, symbol Switch:SW_SPDT
- removed U2: STM32F745VET6, Package_QFP:LQFP-100_14x14mm_P0.5mm, symbol MCU_ST_STM32F7:STM32F745VETx
- removed U7: E104-BT51, Hardware:WIRELM-SMD_E180-ZG120A, symbol VariometerV2-rescue:E104-BT51-Vario2_Library
- removed Y1: 16MHz, Crystal:Crystal_SMD_3225-4Pin_3.2x2.5mm, symbol Device:Crystal_GND24_Small
- added C? (x2): 22uF, symbol Device:C_Small
- added C?: 0.1uF, symbol Device:C_Small
- added IC?: ESP32-WROOM-32E, ESP32WROOM32EM113EH2800PH3Q0, symbol SamacSys_Parts:ESP32-WROOM-32E_M113EH2800PH3Q0_
- added R?: 22, Resistor_SMD:R_0402_1005Metric, symbol Device:R_Small
- added R?: 10k, Resistor_SMD:R_0603_1608Metric, symbol Device:R_Small
Connections:
- net labels added: EN, IO0, JTAG_TCLK, JTAG_TDI, JTAG_TDO, JTAG_TMS, SDCARD_CS
- net labels removed: +3.3VA, BLE_DATA, BLE_LED, BLE_LINK, BLE_MODE, BLE_SLEEP, BLE_nRESET, BOOT0, ERROR_LED, GPS_LED, HSE_IN, HSE_OUT, NRST, SDMMC1_CK, SDMMC1_CMD, SDMMC1_D0, SDMMC1_D1, SDMMC1_D2, SDMMC1_D3, SWCLK, SWDIO, SWO, USART1_RX, USART1_TX, VREF+
- wire segments 472 -> 374
- no-connect marks 84 -> 25
Other:
- note removed: "Analog Filtering"
- note removed: "Bluetooth Low Energy"
- note removed: "Boot Selection"
- note removed: "Ext. Crystal"
- note removed: "I2C Pullups"
- note removed: "LEDS"
- note removed: "Power Filtering"
- note removed: "STM32 Microcontroller"
- note removed: "VREF+ Filtering"
- moved on the sheet: R26, R27

Commit message: fast fertig
Parts:
- removed IC?: ESP32-WROOM-32E, ESP32WROOM32EM113EH2800PH3Q0, symbol SamacSys_Parts:ESP32-WROOM-32E_M113EH2800PH3Q0_
- removed J4: Conn_01x04, Connector_PinHeader_1.27mm:PinHeader_1x04_P1.27mm_Vertical, symbol Connector_Generic:Conn_01x04
- removed R26, R27: 22, Resistor_SMD:R_0402_1005Metric, symbol Device:R_Small
- added C?: 10uF, symbol Device:C_Small
- added C?: 0.1uF, symbol Device:C_Small
- added IC?: ESP32-S3-WROOM-1, ESP32S3WROOM1, symbol SamacSys_Parts:ESP32-S3-WROOM-1
- added J?: TFT_LCD_CONNECTOR, symbol Connector_Generic:Conn_01x08
- added R?: 4.7k, symbol Device:R_Small
- added SW? (x2): Switch_SW_Push, symbol VariometerV2-cache:Switch_SW_Push
- C?: renamed from C7; value 0.1 uF -> 0.1uF
- C?: value 22uF -> 10uF
- C?: renamed from C25; value 100 nF -> 100nF
- C?: renamed from C26; value 2.2 uF -> 2.2uF
- C?: value 22uF -> 1uF
- renumbered C1 to C?, C28 to C?, C29 to C?, C8 to C?, C3 to C?, C2 to C?, C35 to C?, C4 to C?, C5 to C?, C33 to C?, C6 to C?, C27 to C?, C34 to C?, D1 to D?, D3 to D?, D2 to D?, D4 to D?, F1 to F?, FB2 to FB?, H1 to H?, H2 to H?, H3 to H?, H4 to H?, IC2 to IC?, IC1 to IC?, J5 to J?, J7 to J?, J9 to J?, J6 to J?, J3 to J?, J1 to J?, J2 to J?, J8 to J?, JP1 to JP?, L1 to L?, Q5 to Q?, Q1 to Q?, Q2 to Q?, Q8 to Q?, Q7 to Q?, Q6 to Q?, Q3 to Q?, Q9 to Q?, Q4 to Q?, Q10 to Q?, R28 to R?, R29 to R?, R30 to R?, R4 to R?, R1 to R?, R2 to R?, R14 to R?, R16 to R?, R15 to R?, R3 to R?, R10 to R?, R11 to R?, R12 to R?, R42 to R?, R43 to R?, R17 to R?, R6 to R?, R7 to R?, R5 to R?, R39 to R?, R40 to R?, R32 to R?, R33 to R?, R9 to R?, R8 to R?, R44 to R?, R45 to R?, R13 to R?, R41 to R?, R34 to R?, R35 to R?, R36 to R?, R37 to R?, R38 to R?, SW1 to SW?, SW3 to SW?, TP2 to TP?, TP1 to TP?, U6 to U?, U1 to U?, U10 to U?, U8 to U?, U9 to U?, U3 to U?, U4 to U?, U5 to U?
Connections:
- net labels added: LCD_CS, LCD_DC, LCD_RST, SPI2_MISO, SPI2_MOSI, SPI2_SCK
- net labels removed: I2C4_SCL, I2C4_SDA
- wire segments 374 -> 380
- no-connect marks 25 -> 23
Other:
- note added: "Boot-Switch"
- note added: "ESP32"
- note added: "Reset-Switch"
- moved on the sheet: C?, D?, F?, H?, J?, JP?, Q?, R?, SW?, TP?, U?

Commit message: Change
Parts:
- removed C?: 100nF, Capacitor_SMD:C_0402_1005Metric, symbol Device:C_Small
- removed J?: TF-15X15, Hardware:TF15X15, symbol VariometerV2-rescue:TF-15X15-SamacSys_Parts
- removed TP?: GND TP, Connector_Pin:Pin_D0.7mm_L6.5mm_W1.8mm_FlatFork, symbol Connector:TestPoint
- removed U?: M24C64, Package_SO:SOIC-8_3.9x4.9mm_P1.27mm, symbol VariometerV2-rescue:M24C64-Vario2_Library
- added D5: BLUE, LED_SMD:LED_0603_1608Metric, symbol Device:LED_Small
- added J9: MEM2075-00-140-01-A, Hardware:MEM20750014001A, symbol SamacSys_Parts:MEM2075-00-140-01-A
- added R25: 1k, Resistor_SMD:R_0603_1608Metric, symbol Device:R_Small
- added R39, R40: 4.7k, Resistor_SMD:R_0402_1005Metric, symbol Device:R_Small
- C1, C2, C5, C7: renamed from C?; value 0.1uF -> 100nF
- C10, C13: renamed from C?; value 0.1uF -> 100nF; footprint (none) -> Capacitor_SMD:C_0402_1005Metric
- C11: renamed from C?; footprint (none) -> Capacitor_SMD:C_0402_1005Metric
- C12, C9: renamed from C?; footprint (none) -> Capacitor_SMD:C_0603_1608Metric
- C3: renamed from C?; footprint Capacitor_SMD:C_0402_1005Metric -> Capacitor_SMD:C_0603_1608Metric
- FB1: renamed from FB?; footprint Inductor_SMD:L_0805_2012Metric -> Inductor_SMD:L_0603_1608Metric
- IC3: renamed from IC?; footprint ESP32S3WROOM1 -> Hardware:ESP32S3WROOM1; symbol SamacSys_Parts:ESP32-S3-WROOM-1 -> VariometerV2-rescue:ESP32-S3-WROOM-1-SamacSys_Parts
- J3: renamed from J?; footprint (none) -> Connector_PinHeader_2.54mm:PinHeader_1x08_P2.54mm_Vertical
- R19: renamed from R?; footprint (none) -> Resistor_SMD:R_0402_1005Metric
- SW2, SW3: renamed from SW?; footprint (none) -> Button_Switch_THT:SW_PUSH_6mm; symbol VariometerV2-cache:Switch_SW_Push -> VariometerV2-rescue:Switch_SW_Push-VariometerV2-cache
- gave numbers to parts that had none: 86
Connections:
- net +3V3: now also D5.2 (A), R39.1, R40.1; no longer C11.1, C12.1, IC3.3 (EN), R18.2, SW2.1
- net 3.3V_SDCARD: now also J9.P4 (VDD)
- net GND: now also Q1.2 (S), J9.P6 (VSS); no longer Q1.3 (D)
- net GPS_PPS: now also R25.2
- net IO0: now also R40.2
- net SDCARD_CS: now also J9.P2 (CD/DAT3)
- net SDCARD_DETECT: now also J9.P9 (CD)
- net SPI2_MISO: now also J9.P7 (DAT0)
- net SPI2_MOSI: now also J9.P3 (CMD)
- net at Q2.3 (D): now also Q1.3 (D); no longer Q1.2 (S)
- net at R30.2, U5.3 (IO2): now also J9.P1 (DAT2)
- net at R35.2, U5.6 (IO4): now also J9.P5 (CLK)
- net at R34.2, U6.3 (IO2): now also J9.P8 (DAT1)
- net I2C_GPS_SCL: no longer names the net of U4.17 (SCL)
- net I2C_GPS_SDA: no longer names the net of U4.16 (SDA)
- new net: D5.1 (K), R25.1
- new net EN: C11.1, C12.1, IC3.3 (EN), R18.2, R39.2, SW2.1
- no-connect marks 23 -> 25
Other:
- moved on the sheet: C15, H1, H2, H3, H4, J7, L1, U4

Commit message: update
Parts:
- removed J9: MEM2075-00-140-01-A, Hardware:MEM20750014001A, symbol SamacSys_Parts:MEM2075-00-140-01-A
- added J9: TFP09-2-12B, Hardware:TFP09212B, symbol SamacSys_Parts:TFP09-2-12B
Connections:
- net 3.3V_SDCARD: now also J9.4 (VDD)
- net GND: now also J9.10 (GND), J9.6 (VSS)
- net SDCARD_CS: now also J9.2 (CD/DAT3)
- net SDCARD_DETECT: now also J9.9 (CARD_DETECTION)
- net SPI2_MISO: now also J9.7 (DAT0)
- net SPI2_MOSI: now also J9.3 (CMD)
- net at R30.2, U5.3 (IO2): now also J9.1 (DAT2)
- net at R35.2, U5.6 (IO4): now also J9.5 (CLK)
- net at R34.2, U6.3 (IO2): now also J9.8 (DAT1)
- no-connect marks 25 -> 24
Other:
- moved on the sheet: C16, C17, C18, FB1, R30, R31, R32, R33, R34, R35, R36, R37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
