File: Hardware/VariometerV2.sch (KiCad schematic (older format))
At the start: 107 parts, among them IC1 TP4056, IC2 DW01A-G, IC3 ESP32-S3-WROOM-1, J1 LED_CHRG, J2 LED_STBY, J3 TFT_LCD_CONNECTOR, J4 Conn_01x02_Male, J5 SWD, J6 USB3135-30-A, J7 5-1814832-1, J8 Conn_02x01, J9 TFP09-2-12B, Q1 AO3400A, Q10 AO3400A, Q2 AO3400A, Q3 AO3401A, Q4 AO3400A, Q5 AO3401A, Q6 AO3400A, Q7 AO3401A, Q8 AO3400A, Q9 AO3401A, SW1 SW_Push, SW2 Switch_SW_Push, SW3 Switch_SW_Push, SW4 SW_Push, U1 TPS76801QDR, U2 SRV05-4, U4 ATGM336H-5N31, U5 SRV05-4, U6 SRV05-4, U7 BMI088, U8 MS5611-01BA

Commit message: Update VariometerV2.sch
Parts:
- R40: value 4.7k -> 0k
Other:
- moved on the sheet: C11, R18
Changed lines of the file:
@@
 L power:+3.3V #PWR0153
 U 1 1 622FD041
-P 750 7050
-F 0 "#PWR0153" H 750 6900 50  0001 C CNN
-F 1 "+3.3V" H 765 7223 50  0000 C CNN
-F 2 "" H 750 7050 50  0001 C CNN
-F 3 "" H 750 7050 50  0001 C CNN
-	1    750  7050
+P 900 7150
+F 0 "#PWR0153" H 900 7000 50  0001 C CNN
+F 1 "+3.3V" H 915 7323 50  0000 C CNN
+F 2 "" H 900 7150 50  0001 C CNN
+F 3 "" H 900 7150 50  0001 C CNN
+	1    900  7150
 	1    0    0    -1
 $EndComp
@@
 L Device:R_Small R18
 U 1 1 622FD801
-P 750 7150
-F 0 "R18" H 809 7196 50  0000 L CNN
-F 1 "10k" H 809 7105 50  0000 L CNN
-F 2 "Resistor_SMD:R_0603_1608Metric" H 750 7150 50  0001 C CNN
-F 3 "~" H 750 7150 50  0001 C CNN
-	1    750  7150
+P 900 7250
+F 0 "R18" H 959 7296 50  0000 L CNN
+F 1 "10k" H 959 7205 50  0000 L CNN
+F 2 "Resistor_SMD:R_0603_1608Metric" H 900 7250 50  0001 C CNN
+F 3 "~" H 900 7250 50  0001 C CNN
+	1    900  7250
 	1    0    0    -1
 $EndComp
@@
 L Device:C_Small C11
 U 1 1 622FF342
-P 750 7550
-F 0 "C11" H 842 7596 50  0000 L CNN
-F 1 "1uF" H 842 7505 50  0000 L CNN
-F 2 "Capacitor_SMD:C_0402_1005Metric" H 750 7550 50  0001 C CNN
-F 3 "~" H 750 7550 50  0001 C CNN
-	1    750  7550
-	1    0    0    -1
-$EndComp
-Wire Wire Line
-	750  7450 750  7350
+P 900 7650
+F 0 "C11" H 992 7696 50  0000 L CNN
+F 1 "1uF" H 992 7605 50  0000 L CNN
+F 2 "Capacitor_SMD:C_0402_1005Metric" H 900 7650 50  0001 C CNN
+F 3 "~" H 900 7650 50  0001 C CNN
+	1    900  7650
+	1    0    0    -1
+$EndComp
+Wire Wire Line
+	900  7550 900  7450
 $Comp
 L power:GND #PWR0154
 U 1 1 6232633B
-P 750 7650
-F 0 "#PWR0154" H 750 7400 50  0001 C CNN
-F 1 "GND" H 755 7477 50  0000 C CNN
-F 2 "" H 750 7650 50  0001 C CNN
-F 3 "" H 750 7650 50  0001 C CNN
-	1    750  7650
-	1    0    0    -1
-$EndComp
-Text GLabel 850  7350 2    50   Input ~ 0
+P 900 7750
+F 0 "#PWR0154" H 900 7500 50  0001 C CNN
+F 1 "GND" H 905 7577 50  0000 C CNN
+F 2 "" H 900 7750 50  0001 C CNN
+F 3 "" H 900 7750 50  0001 C CNN
+	1    900  7750
+	1    0    0    -1
+$EndComp
+Text GLabel 1000 7450 2    50   Input ~ 0
 EN
 Wire Wire Line
-	750  7350 850  7350
-Connection ~ 750  7350
-Wire Wire Line
-	750  7350 750  7250
+	900  7450 1000 7450
+Connection ~ 900  7450
+Wire Wire Line
+	900  7450 900  7350
 $Comp
 L VariometerV2-rescue:ESP32-S3-WROOM-1-SamacSys_Parts IC3
@@
 P 2800 9650
 F 0 "R40" H 2859 9696 50  0000 L CNN
-F 1 "4.7k" H 2859 9605 50  0000 L CNN
+F 1 "0k" H 2859 9605 50  0000 L CNN
 F 2 "Resistor_SMD:R_0402_1005Metric" H 2800 9650 50  0001 C CNN
 F 3 "~" H 2800 9650 50  0001 C CNN

Commit message: k
Parts:
- J7: footprint Hardware:5-1814832-1 -> Hardware:518148322
Changed lines of the file:
@@
 F 0 "J7" H 7912 10014 50  0000 C CNN
 F 1 "5-1814832-1" H 8000 9950 50  0000 C CNN
-F 2 "Hardware:5-1814832-1" H 7950 9700 50  0001 L BNN
+F 2 "Hardware:518148322" H 7950 9700 50  0001 L BNN
 F 3 "https://www.te.com/usa-en/product-518148321.html?te_bu=Cor&te_type=disp&te_campaign=seda_glo_cor-seda-global-disp-prtnr-fy19-seda-model-bom-cta_sma-317_1&elqCampaignId=32493" H 7950 9700 50  0001 L BNN
 F 4 "TE Connectivity" H 7950 9700 50  0001 L BNN "Field4"
