File: Hardware/VariometerV2.kicad_pcb (KiCad board)
At the start: 4 copper layers, 61.2 x 69.8 mm, 134 parts, among them IC1 TP4056, IC2 DW01A-G, J1 LED_CHRG, J2 LED_STBY, J3 Conn_01x02_Male, J4 Conn_01x04, J5 SWD, J6 USB3135-30-A, J7 TF-15X15, J8 Conn_02x01, J9 5-1814832-1, Q1 AO3400A, Q10 AO3400A, Q2 AO3400A, Q3 AO3401A, Q4 AO3400A, Q5 AO3401A, Q6 AO3400A, Q7 AO3401A, Q8 AO3400A, Q9 AO3401A, SW1 SW_Push, SW2 SW_SPDT, SW3 SW_Push, U1 TPS76801QDR, U10 MS5611-01BA, U2 STM32F745VET6, U3 SRV05-4, U4 SRV05-4, U5 SRV05-4, U6 BMI088, U7 E104-BT51, U8 M24C64, U9 ATGM336H-5N31, Y1 16MHz

Commit message: PCB fertig
Parts:
- C3: footprint Capacitor_SMD:C_0201_0603Metric -> Capacitor_SMD:C_0402_1005Metric
- F1: value 700mA -> 1A
- moved U3 0.52 mm to (119.9, 122.1)
- moved R1 0.40 mm to (120.5, 126.4)
- moved U6 0.35 mm to (92.5, 143.2)
- moved C28 0.34 mm to (92.6, 146.9)
- moved C3 0.31 mm to (125.4, 132.2), turned to 0 degrees
- moved R32 0.21 mm to (120.3, 124.8)
Connections:
- U4 pad 6: SDMMC1_CK -> Net-(J7-Pad5)
Routing:
- net GND: track 73.4 -> 201.6 mm, vias 18 -> 87
- net BATT+: track 27.9 -> 54.3 mm, vias 0 -> 2
- net SDCARD_DETECT: track 10.4 -> 25.7 mm, vias 2 -> 4
- net BATT_CONN-: track 6.85 -> 21.5 mm, vias 0 -> 2
- net Net-(J7-Pad5): track 3.33 -> 17.7 mm, vias 0 -> 2
- net +3V3: track 111.3 -> 124.8 mm, vias 45 -> 46
- net USB_D-: track 47.5 -> 36.8 mm
- net USB_D+: track 48.5 -> 39.9 mm
- net Net-(D4-Pad1): track 0.00 -> 2.30 mm
- net Net-(R19-Pad1): track 17.4 -> 15.9 mm
- net SDMMC1_CMD: track 26.1 -> 27.0 mm
- net SDMMC1_D1: track 35.3 -> 34.4 mm
- net Button_Input: track 11.9 -> 12.7 mm
- net ACC_INT: track 19.4 -> 20.1 mm
- net Net-(J9-Pad1): track 10.2 -> 10.9 mm
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- added copper zone on F.Cu, net GND
Other:
- rule trace_min: 0.0889 -> 0.2

Commit message: update
Parts:
- J3: footprint Connector_PinSocket_2.54mm:PinSocket_1x02_P2.54mm_Vertical -> Connector_PinHeader_2.54mm:PinHeader_1x02_P2.54mm_Vertical
Routing:
- net GND: track 201.6 -> 200.2 mm, vias 87 -> 88
- net +3V3: track 124.8 -> 123.4 mm
Other:
- rule via_min_size: 0.2 -> 0.4

Commit message: hg
Routing:
- net USB_D-: track 36.8 -> 38.7 mm
- net GND: track 200.2 -> 201.3 mm, vias 88 -> 89
Other:
- board text added: "+"
- board text added: "3.3V"
- board text added: "Charge"
- board text added: "GND"
- board text added: "Input"
- board text added: "Standby"

Commit message: jh
Parts:
- moved C29 1.22 mm to (90.8, 140.4)
- moved C20 1.04 mm to (90.7, 138.0)
Routing:
- net Net-(C20-Pad1): track 2.36 -> 4.04 mm
- net Net-(J9-Pad1): track 10.9 -> 10.3 mm
- net GND: track 201.3 -> 201.7 mm, vias 89 -> 90
- net +3V3: track 123.4 -> 123.7 mm, vias 46 -> 45

Commit message: Fertig
Parts:
- R46: footprint Resistor_SMD:R_0402_1005Metric -> Resistor_SMD:R_0805_2012Metric
- moved C30 0.81 mm to (115.4, 161.4)
- moved R46 0.27 mm to (112.0, 161.8)
Routing:
- net +3V3: track 123.7 -> 114.5 mm, vias 45 -> 44
- net BLE_nRESET: track 48.9 -> 49.9 mm
Other:
- board text added: "-"
- board text added: "BATTERY"
- board text added: "BLE"
- board text added: "BOOT"
- board text added: "BUZZER"
- board text added: "ERROR"
- board text added: "GPS"
- board text added: "I2C"
- board text added: "JUMPER"
- board text added: "ON/OFF"
- board text added: "Power"
- board text added: "RUN"
- board text added: "SD-CARD"
- board text added: "SWD"
- board text added: "USB"
- board text added: "Variometer | V. 1"

Commit message: hg
Other:
- board text added: "5V"
- board text added: "INPUT"
- board text added: "NC"
- board text added: "NRST"
- board text added: "RF_IN"
- board text added: "SCL"
- board text added: "SDA"
- board text added: "SWCLK"
- board text added: "SWDIO"
- board text added: "SWO"
- board text added: "USB_D+"
- board text added: "USB_D-"
- board text added: "X"
- board text added: "Y"
- board text removed: "Input"

Commit message: gerber added
Other:
- outline, holes or cut-outs redrawn
- board text added: "JLCJLCJLCJLC"

Commit message: Change
Parts:
- removed C14, C24, C28, C29, C30, C31, C33, C35: 100nF, Capacitor_SMD:C_0402_1005Metric
- removed C22, C23: 6pF, Capacitor_SMD:C_0603_1608Metric
- removed C25: 100 nF, Capacitor_SMD:C_0402_1005Metric
- removed C26: 2.2 uF, Capacitor_SMD:C_0402_1005Metric
- removed C27: 2.2uF, Capacitor_SMD:C_0402_1005Metric
- removed C32, C34: 10uF, Capacitor_SMD:C_0603_1608Metric
- removed D6: BL, LED_SMD:LED_0603_1608Metric
- removed D7: GR, LED_SMD:LED_0603_1608Metric
- removed FB2: 600 @ 100 MHz, Inductor_SMD:L_0805_2012Metric
- removed R41: 1M, Resistor_SMD:R_0402_1005Metric
- removed R42, R43, R44, R45: 10k, Resistor_SMD:R_0402_1005Metric
- removed R46: 100k, Resistor_SMD:R_0805_2012Metric
- removed TP2: GND TP, Connector_Pin:Pin_D0.7mm_L6.5mm_W1.8mm_FlatFork
- removed U10: MS5611-01BA, Package_LGA:LGA-8_3x5mm_P1.25mm
- removed U3: SRV05-4, Package_TO_SOT_SMD:SOT-23-6
- removed U9: ATGM336H-5N31, Hardware:ATGM336H5N31
- removed Y1: 16MHz, Crystal:Crystal_SMD_3225-4Pin_3.2x2.5mm
- added IC3: ESP32-S3-WROOM-1, Hardware:ESP32S3WROOM1, F.Cu at (35.1, 56.3)
- added SW4: SW_Push, Connector_Wire:SolderWire-0.25sqmm_1x02_P4.2mm_D0.65mm_OD1.7mm, F.Cu at (25.7, 78.4)
- C1, C2, C5: value 0.1uF -> 100nF
- C11: value 100nF -> 1uF
- C12, C15: value 100nF -> 10uF; footprint Capacitor_SMD:C_0402_1005Metric -> Capacitor_SMD:C_0603_1608Metric
- C16: value 1uF -> 2.2uF
- C17: value 10nF -> 2.2uF
- C18: value 1uF -> 100nF
- C20, C21: value 2.2uF -> 100nF; footprint Capacitor_SMD:C_0603_1608Metric -> Capacitor_SMD:C_0402_1005Metric
- C3: footprint Capacitor_SMD:C_0402_1005Metric -> Capacitor_SMD:C_0603_1608Metric
- C7: value 0.1 uF -> 100nF
- C9: value 4.7uF -> 10uF
- D5: value RE -> BLUE
- FB1: value 600 @ 100MHz -> 600 @ 100 MHz; footprint Inductor_SMD:L_0805_2012Metric -> Inductor_SMD:L_0603_1608Metric
- J3: value Conn_01x02_Male -> TFT_LCD_CONNECTOR; footprint Connector_PinHeader_2.54mm:PinHeader_1x02_P2.54mm_Vertical -> Connector_PinHeader_2.54mm:PinHeader_1x08_P2.54mm_Vertical
- J4: value Conn_01x04 -> Conn_01x02_Male; footprint Connector_PinHeader_1.27mm:PinHeader_1x04_P1.27mm_Vertical -> Connector_PinHeader_2.54mm:PinHeader_1x02_P2.54mm_Vertical
- J7: value TF-15X15 -> 5-1814832-1; footprint Hardware:TF15X15 -> Hardware:5-1814832-1
- J9: value 5-1814832-1 -> MEM2075-00-140-01-A; footprint Hardware:5-1814832-1 -> Hardware:MEM20750014001A
- R13: value 1.5k -> 1M; footprint Resistor_SMD:R_0603_1608Metric -> Resistor_SMD:R_0402_1005Metric
- R14: value 1M -> 10k
- R15: value 10k -> 33k
- R16: value 33k -> 10k
- R17: value 10k -> 1.5k; footprint Resistor_SMD:R_0402_1005Metric -> Resistor_SMD:R_0603_1608Metric
- R18: value 47 -> 10k; footprint Resistor_SMD:R_0402_1005Metric -> Resistor_SMD:R_0603_1608Metric
- R19, R39, R40: value 10k -> 4.7k
- R20: value 47 -> 22; footprint Resistor_SMD:R_0805_2012Metric -> Resistor_SMD:R_0402_1005Metric
- R21, R22: value 1k -> 22; footprint Resistor_SMD:R_0603_1608Metric -> Resistor_SMD:R_0402_1005Metric
- R23: value 2.2k -> 22; footprint Resistor_SMD:R_0603_1608Metric -> Resistor_SMD:R_0402_1005Metric
- R24: value 2.2k -> 10k
- R25: value 2.2k -> 1k; footprint Resistor_SMD:R_0402_1005Metric -> Resistor_SMD:R_0603_1608Metric
- R26, R27, R28, R29, R30, R31: value 22 -> 10k
- R35: value 10k -> 22
- R38: value 22 -> 1M
- R8: value 100k -> 300k
- R9: value 300k -> 100k
- SW2: value SW_SPDT -> Switch_SW_Push; footprint Hardware:MINISPDTSW -> Button_Switch_THT:SW_PUSH_6mm
- SW3: value SW_Push -> Switch_SW_Push; footprint Connector_Wire:SolderWire-0.25sqmm_1x02_P4.2mm_D0.65mm_OD1.7mm -> Button_Switch_THT:SW_PUSH_6mm
- U2: value STM32F745VET6 -> SRV05-4; footprint Package_QFP:LQFP-100_14x14mm_P0.5mm -> Package_TO_SOT_SMD:SOT-23-6
- U4: value SRV05-4 -> ATGM336H-5N31; footprint Package_TO_SOT_SMD:SOT-23-6 -> Hardware:ATGM336H5N31
- U6: value BMI088 -> SRV05-4; footprint Hardware:BMI088 -> Package_TO_SOT_SMD:SOT-23-6
- U7: value E104-BT51 -> BMI088; footprint Hardware:WIRELM-SMD_E180-ZG120A -> Hardware:BMI088
- U8: value M24C64 -> MS5611-01BA; footprint Package_SO:SOIC-8_3.9x4.9mm_P1.27mm -> Package_LGA:LGA-8_3x5mm_P1.25mm
- moved H2 174.5 mm to (25.1, 20.7)
- moved J9 139.7 mm to (38.7, 26.0), turned to 180 degrees
- moved J8 128.7 mm to (68.0, 38.0), turned to 270 degrees
- moved Q7 128.6 mm to (71.0, 33.9), turned to 180 degrees
- moved Q8 127.0 mm to (66.5, 34.1), turned to 0 degrees
- moved J3 124.5 mm to (69.5, 19.0), turned to 270 degrees
- moved Q9 123.0 mm to (72.1, 39.0), turned to 180 degrees
- moved U6 122.2 mm to (51.1, 28.1), turned to 0 degrees
- moved R32 118.8 mm to (39.3, 37.9), turned to 90 degrees
- moved C13 117.5 mm to (62.8, 22.3), turned to 180 degrees
- moved Q10 113.8 mm to (71.1, 44.3), turned to 0 degrees
- moved R30 112.1 mm to (35.4, 37.6), turned to 0 degrees
- moved R31 108.6 mm to (37.6, 37.9), turned to 90 degrees
- moved C16 105.6 mm to (30.1, 37.9), turned to 0 degrees
- moved TP1 105.4 mm to (62.5, 35.5), turned to 0 degrees
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Connections:
- C11 pad 1: +3V3 -> EN
- C12 pad 1: +3V3 -> EN
- C13 pad 1: +3V3 -> IO0
- C16 pad 1: +3.3VA -> +3V3
- C17 pad 1: +3.3VA -> 3.3V_SDCARD
- C18 pad 1: VREF+ -> 3.3V_SDCARD
- C19 pad 1: VREF+ -> +3V3
- C20 pad 1: Net-(C20-Pad1) -> +3V3
- C21 pad 1: Net-(C21-Pad1) -> +3V3
- D5 pad 2: ERROR_LED -> +3V3
- FB1 pad 1: +3.3VA -> +3V3
- FB1 pad 2: +3V3 -> 3.3V_SDCARD
- IC2 pad 4: Net-(IC2-Pad4) -> (no net)
- J3 pad 1: BATT_CONN- -> GND
- J3 pad 2: BATT+ -> +3V3
- J4 pad 1: +3V3 -> BATT_CONN-
- J4 pad 2: Net-(J4-Pad2) -> BATT+
- J5 pad 10: Net-(J5-Pad10) -> (no net)
- J5 pad 7: Net-(J5-Pad7) -> (no net)
- J6 pad 4: Net-(J6-Pad4) -> (no net)
- J7 pad 1: SDMMC1_D2 -> Net-(J7-Pad1)
- J7 pad 2: SDMMC1_D3 -> GND
- J7 pad 3: SDMMC1_CMD -> GND
- J7 pad 4: 3.3V_SDCARD -> GND
- J7 pad 5: Net-(J7-Pad5) -> GND
- L1 pad 1: Net-(J9-Pad1) -> Net-(J7-Pad1)
- Q1 pad 2: Net-(Q1-Pad2) -> GND
- Q1 pad 3: GND -> Net-(Q1-Pad3)
- Q2 pad 3: Net-(Q1-Pad2) -> Net-(Q1-Pad3)
- R13 pad 1: Net-(D4-Pad1) -> Net-(Q5-Pad1)
- R13 pad 2: GND -> BATT+
- R14 pad 1: Net-(Q5-Pad1) -> BAT_ADC
- R14 pad 2: BATT+ -> Net-(Q5-Pad3)
- R15 pad 1: BAT_ADC -> GND
- R15 pad 2: Net-(Q5-Pad3) -> BAT_ADC
- R16 pad 1: GND -> BAT_MS
- R16 pad 2: BAT_ADC -> Net-(Q6-Pad1)
- R17 pad 1: BAT_MS -> Net-(D4-Pad1)
- R17 pad 2: Net-(Q6-Pad1) -> GND
- R18 pad 1: VREF+ -> +3V3
- R18 pad 2: +3.3VA -> EN
- R19 pad 1: Net-(R19-Pad1) -> +3V3
- R19 pad 2: BOOT0 -> Button_Input
- R20 pad 1: HSE_OUT -> Net-(J5-Pad2)
- R20 pad 2: Net-(C23-Pad1) -> JTAG_TMS
- R21 pad 1: Net-(D5-Pad1) -> Net-(J5-Pad4)
- R21 pad 2: GND -> JTAG_TCLK
- R22 pad 1: Net-(D6-Pad1) -> Net-(J5-Pad6)
- R22 pad 2: GND -> JTAG_TDO
- R23 pad 1: Net-(D7-Pad1) -> Net-(J5-Pad8)
- R23 pad 2: GND -> JTAG_TDI
- R24 pad 1: +3V3 -> +5V
- R24 pad 2: I2C4_SCL -> Net-(R24-Pad2)
- R25 pad 1: +3V3 -> Net-(D5-Pad1)
- R25 pad 2: I2C4_SDA -> GPS_PPS
- R26 pad 1: I2C4_SCL -> Net-(Q7-Pad1)
- R26 pad 2: Net-(J4-Pad2) -> TIM1_CH1
- R27 pad 1: I2C4_SDA -> Net-(Q8-Pad1)
- R27 pad 2: Net-(J4-Pad3) -> TIM1_CH1
- R28 pad 1: Net-(J5-Pad2) -> TIM1_CH1N
- R28 pad 2: SWDIO -> Net-(Q9-Pad1)
- R29 pad 1: Net-(J5-Pad4) -> TIM1_CH1N
- R29 pad 2: SWCLK -> Net-(Q10-Pad1)
- R30 pad 1: Net-(J5-Pad6) -> +3V3
- R30 pad 2: SWO -> Net-(J9-PadP1)
- R31 pad 1: Net-(J5-Pad10) -> +3V3
- R31 pad 2: NRST -> SDCARD_CS
- R32 pad 1: +5V -> +3V3
- R32 pad 2: Net-(R32-Pad2) -> SPI2_MOSI
- R33 pad 2: SDMMC1_D2 -> SPI2_MISO
- R34 pad 2: SDMMC1_D3 -> Net-(J9-PadP8)
- R35 pad 1: +3V3 -> SPI2_SCK
- R35 pad 2: SDMMC1_CMD -> Net-(J9-PadP5)
- R36 pad 2: SDMMC1_D0 -> Net-(R36-Pad2)
- R37 pad 1: +3V3 -> Net-(R37-Pad1)
- R37 pad 2: SDMMC1_D1 -> +3V3
- R38 pad 1: SDMMC1_CK -> SDCARD_DETECT
- R38 pad 2: Net-(J7-Pad5) -> GND
- R39 pad 2: Net-(R39-Pad2) -> EN
- R40 pad 1: Net-(R40-Pad1) -> +3V3
- R40 pad 2: +3V3 -> IO0
- R8 pad 1: POW_SW+ -> Net-(D3-Pad2)
- R8 pad 2: Net-(D3-Pad2) -> Net-(C6-Pad1)
- R9 pad 1: Net-(D3-Pad2) -> POW_SW+
- R9 pad 2: Net-(C6-Pad1) -> Net-(D3-Pad2)
- SW2 pad 1: +3V3 -> EN
- SW2 pad 2: Net-(R19-Pad1) -> GND
- SW3 pad 1: Button_Input -> IO0
- SW3 pad 2: +3V3 -> GND
- U1 pad 8: Net-(U1-Pad8) -> (no net)
- U2 pad 1: Net-(U2-Pad1) -> USB_D+
- U2 pad 2: Net-(U2-Pad2) -> GND
- U2 pad 3: Net-(U2-Pad3) -> USB_D-
- U2 pad 4: Net-(U2-Pad4) -> (no net)
- U2 pad 5: Net-(U2-Pad5) -> Net-(R24-Pad2)
- U2 pad 6: +3V3 -> (no net)
- U4 pad 1: SDMMC1_D3 -> GND
- U4 pad 2: GND -> USART2_RX
- U4 pad 3: SDMMC1_D2 -> USART2_TX
- U4 pad 4: SDMMC1_CMD -> GPS_PPS
- U4 pad 5: Net-(R39-Pad2) -> GPS_ON
- U4 pad 6: Net-(J7-Pad5) -> +3V3
- U5 pad 1: SDMMC1_D0 -> SDCARD_CS
- U5 pad 3: SDMMC1_D1 -> Net-(J9-PadP1)
- U5 pad 4: SDCARD_DETECT -> SPI2_MOSI
- U5 pad 5: Net-(R40-Pad1) -> Net-(R36-Pad2)
- U5 pad 6: 3.3V_SDCARD -> Net-(J9-PadP5)
- U6 pad 1: Net-(U6-Pad1) -> SPI2_MISO
- U6 pad 3: +3V3 -> Net-(J9-PadP8)
- U6 pad 4: GND -> SDCARD_DETECT
- U6 pad 5: IMU_GYR_CS -> Net-(R37-Pad1)
- U6 pad 6: GND -> 3.3V_SDCARD
- U7 pad 1: GND -> (no net)
- U7 pad 10: Net-(U7-Pad10) -> SPI1_MISO
- U7 pad 11: Net-(U7-Pad11) -> +3V3
- U7 pad 12: Net-(U7-Pad12) -> GYR_INT
- U7 pad 13: Net-(U7-Pad13) -> (no net)
- U7 pad 14: Net-(U7-Pad14) -> IMU_ACC_CS
- U7 pad 15: Net-(U7-Pad15) -> SPI1_MISO
- U7 pad 16: BLE_SLEEP -> ACC_INT
- U7 pad 3: GND -> +3V3
- U7 pad 4: Net-(U7-Pad4) -> GND
- U7 pad 5: Net-(U7-Pad5) -> IMU_GYR_CS
- U7 pad 6: USART1_TX -> GND
- U7 pad 7: USART1_RX -> GND
- U7 pad 8: Net-(U7-Pad8) -> SPI1_SCK
- U7 pad 9: Net-(U7-Pad9) -> SPI1_MOSI
- U8 pad 1: GND -> +3V3
- U8 pad 4: GND -> PresSens_CS
- U8 pad 5: I2C_GPS_SDA -> PresSens_CS
- U8 pad 6: I2C_GPS_SCL -> SPI1_MISO
- U8 pad 7: GND -> SPI1_MOSI
- U8 pad 8: +3V3 -> SPI1_SCK
Routing:
- net GND: track 201.6 -> 0.00 mm, vias 90 -> 0
- net +3V3: track 114.5 -> 0.00 mm, vias 44 -> 0
- net BLE_LED: track 74.0 -> 0.00 mm, vias 2 -> 0
- net GPS_LED: track 69.1 -> 0.00 mm, vias 2 -> 0
- net NRST: track 66.9 -> 0.00 mm, vias 2 -> 0
- net BAT_MS: track 63.6 -> 0.00 mm, vias 2 -> 0
- net ERROR_LED: track 63.2 -> 0.00 mm, vias 2 -> 0
- net +5V: track 57.4 -> 0.00 mm, vias 5 -> 0
- net BAT_ADC: track 57.0 -> 0.00 mm, vias 2 -> 0
- net BATT+: track 54.3 -> 0.00 mm, vias 2 -> 0
- net BLE_nRESET: track 49.9 -> 0.00 mm, vias 2 -> 0
- net SWO: track 48.7 -> 0.00 mm, vias 2 -> 0
- net SWCLK: track 45.6 -> 0.00 mm, vias 2 -> 0
- net I2C4_SCL: track 44.7 -> 0.00 mm, vias 2 -> 0
- net I2C4_SDA: track 44.3 -> 0.00 mm, vias 2 -> 0
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- removed copper zone on In2.Cu, net +3V3
- removed copper zone on F.Cu, net GND
- removed copper zone on In1.Cu, net GND
Other:
- board outline removed
- board text removed: "+"
- board text removed: "-"
- board text removed: "3.3V"
- board text removed: "5V"
- board text removed: "BATTERY"
- board text removed: "BLE"
- board text removed: "BOOT"
- board text removed: "BUZZER"
- board text removed: "Charge"
- board text removed: "ERROR"
- board text removed: "GND"
- board text removed: "GPS"
- board text removed: "I2C"
- board text removed: "INPUT"
- board text removed: "JLCJLCJLCJLC"
- board text removed: "JUMPER"
- board text removed: "NC"
- board text removed: "NRST"
- board text removed: "ON/OFF"
- board text removed: "Power"
- board text removed: "RF_IN"
- board text removed: "RUN"
- board text removed: "SCL"
- board text removed: "SD-CARD"
- board text removed: "SDA"
- board text removed: "SWCLK"
- board text removed: "SWD"
- board text removed: "SWDIO"
- board text removed: "SWO"
- board text removed: "Standby"
- board text removed: "USB"
- board text removed: "USB_D+"
- board text removed: "USB_D-"
- board text removed: "Variometer | V. 1"
- board text removed: "X"
- board text removed: "Y"
