File: Hardware/VariometerV2.kicad_pcb (KiCad board)
At the start: 4 copper layers, 107 parts, among them IC1 TP4056, IC2 DW01A-G, IC3 ESP32-S3-WROOM-1, J1 LED_CHRG, J2 LED_STBY, J3 TFT_LCD_CONNECTOR, J4 Conn_01x02_Male, J5 SWD, J6 USB3135-30-A, J7 5-1814832-1, J8 Conn_02x01, J9 MEM2075-00-140-01-A, Q1 AO3400A, Q10 AO3400A, Q2 AO3400A, Q3 AO3401A, Q4 AO3400A, Q5 AO3401A, Q6 AO3400A, Q7 AO3401A, Q8 AO3400A, Q9 AO3401A, SW1 SW_Push, SW2 Switch_SW_Push, SW3 Switch_SW_Push, SW4 SW_Push, U1 TPS76801QDR, U2 SRV05-4, U4 ATGM336H-5N31, U5 SRV05-4, U6 SRV05-4, U7 BMI088, U8 MS5611-01BA

Commit message: update
Parts:
- removed C19: 100nF, Capacitor_SMD:C_0402_1005Metric
- J9: value MEM2075-00-140-01-A -> TFP09-2-12B; footprint Hardware:MEM20750014001A -> Hardware:TFP09212B
- moved SW4 52.3 mm to (56.5, 36.2), turned to 270 degrees
- moved R19 41.9 mm to (54.3, 41.2), turned to 90 degrees
- moved J9 7.99 mm to (38.5, 18.0), turned to 270 degrees
- moved R13 4.28 mm to (76.4, 74.5), turned to 90 degrees
- moved R16 2.45 mm to (70.9, 78.1), turned to 0 degrees
- moved R15 2.44 mm to (69.8, 75.1), turned to 270 degrees
- moved IC3 2.42 mm to (32.7, 55.8)
- moved Q5 2.32 mm to (73.8, 74.6)
- moved Q6 2.32 mm to (74.0, 78.9)
- moved R24 2.29 mm to (68.8, 72.0)
- moved R14 2.10 mm to (70.9, 75.1)
- moved U7 1.86 mm to (49.0, 72.5)
- moved J6 1.74 mm to (74.5, 66.7)
- moved C17 1.49 mm to (33.3, 37.6)
- moved R30 1.49 mm to (35.6, 36.1)
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Connections:
- IC2 pad 4: (no net) -> Net-(IC2-Pad4)
- IC3 pad 15: (no net) -> Net-(IC3-Pad15)
- IC3 pad 16: (no net) -> Net-(IC3-Pad16)
- IC3 pad 36: (no net) -> Net-(IC3-Pad36)
- IC3 pad 37: (no net) -> Net-(IC3-Pad37)
- IC3 pad 5: (no net) -> Net-(IC3-Pad5)
- J5 pad 10: (no net) -> Net-(J5-Pad10)
- J5 pad 7: (no net) -> Net-(J5-Pad7)
- J6 pad 4: (no net) -> Net-(J6-Pad4)
- R30 pad 2: Net-(J9-PadP1) -> Net-(J9-Pad1)
- R34 pad 2: Net-(J9-PadP8) -> Net-(J9-Pad8)
- R35 pad 2: Net-(J9-PadP5) -> Net-(J9-Pad5)
- U1 pad 8: (no net) -> Net-(U1-Pad8)
- U2 pad 4: (no net) -> Net-(U2-Pad4)
- U2 pad 6: (no net) -> Net-(U2-Pad6)
- U4 pad 13: (no net) -> Net-(U4-Pad13)
- U4 pad 15: (no net) -> Net-(U4-Pad15)
- U4 pad 16: (no net) -> Net-(U4-Pad16)
- U4 pad 17: (no net) -> Net-(U4-Pad17)
- U4 pad 18: (no net) -> Net-(U4-Pad18)
- U4 pad 7: (no net) -> Net-(U4-Pad7)
- U4 pad 9: (no net) -> Net-(U4-Pad9)
- U5 pad 3: Net-(J9-PadP1) -> Net-(J9-Pad1)
- U5 pad 6: Net-(J9-PadP5) -> Net-(J9-Pad5)
- U6 pad 3: Net-(J9-PadP8) -> Net-(J9-Pad8)
- U7 pad 1: (no net) -> Net-(U7-Pad1)
- U7 pad 13: (no net) -> Net-(U7-Pad13)
Routing:
- net USB_D-: track 26.1 -> 30.4 mm
- net USB_D+: track 24.8 -> 29.1 mm
Other:
- board outline added: 56.6 x 69.4 mm

Commit message: k
Parts:
- added C19: 100nF, Capacitor_SMD:C_0402_1005Metric, F.Cu at (52.5, 71.2)
- J3: footprint Connector_PinHeader_2.54mm:PinHeader_1x08_P2.54mm_Vertical -> Connector_PinHeader_2.54mm:PinHeader_1x09_P2.54mm_Vertical
- J7: value 5-1814832-1 -> 5-1814832-2; footprint Hardware:5-1814832-1 -> Hardware:518148322
- R40: value 4.7k -> 0k; footprint Resistor_SMD:R_0402_1005Metric -> Resistor_SMD:R_0805_2012Metric
- moved R19 26.4 mm to (28.0, 43.4), turned to 0 degrees
- moved SW4 24.0 mm to (33.1, 41.2), turned to 180 degrees
- moved R25 12.3 mm to (32.0, 71.7), turned to -90 degrees
- moved D5 11.7 mm to (34.1, 71.7)
- moved C20 7.31 mm to (45.5, 73.7)
- moved C18 6.77 mm to (31.9, 35.2), turned to 180 degrees
- moved R27 4.29 mm to (65.3, 36.7), turned to -90 degrees
- moved U5 3.66 mm to (52.0, 30.6), turned to 180 degrees
- moved R34 3.61 mm to (44.3, 39.6)
- moved C1 3.50 mm to (69.1, 65.2)
- moved R30 3.34 mm to (35.5, 39.4), turned to 90 degrees
- moved R1 3.30 mm to (59.1, 64.9)
- moved R35 3.27 mm to (40.7, 39.5)
- moved R38 3.27 mm to (46.6, 39.8)
- moved R33 3.01 mm to (42.6, 39.6)
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Connections:
- IC2 pad 4: Net-(IC2-Pad4) -> unconnected-(IC2-Pad4)
- IC3 pad 15: Net-(IC3-Pad15) -> unconnected-(IC3-Pad15)
- IC3 pad 16: Net-(IC3-Pad16) -> LCD_TCH_CS
- IC3 pad 23: LCD_DC -> LCD_RST
- IC3 pad 24: LCD_CS -> LCD_DC
- IC3 pad 25: LCD_RST -> LCD_CS
- IC3 pad 36: Net-(IC3-Pad36) -> unconnected-(IC3-Pad36)
- IC3 pad 37: Net-(IC3-Pad37) -> unconnected-(IC3-Pad37)
- IC3 pad 5: Net-(IC3-Pad5) -> unconnected-(IC3-Pad5)
- IC3 pad 7: IMU_ACC_CS -> GYR_INT
- IC3 pad 8: ACC_INT -> IMU_ACC_CS
- IC3 pad 9: GYR_INT -> ACC_INT
- J3 pad 3: LCD_RST -> LCD_TCH_CS
- J3 pad 4: LCD_DC -> LCD_RST
- J3 pad 5: LCD_CS -> LCD_DC
- J3 pad 6: SPI2_MOSI -> LCD_CS
- J3 pad 7: SPI2_SCK -> SPI2_MOSI
- J3 pad 8: SPI2_MISO -> SPI2_SCK
- J5 pad 10: Net-(J5-Pad10) -> unconnected-(J5-Pad10)
- J5 pad 7: Net-(J5-Pad7) -> unconnected-(J5-Pad7)
- J6 pad 4: Net-(J6-Pad4) -> unconnected-(J6-Pad4)
- J9 pad 11: Net-(J9-Pad11) -> unconnected-(J9-Pad11)
- J9 pad 12: Net-(J9-Pad12) -> unconnected-(J9-Pad12)
- J9 pad 13: Net-(J9-Pad13) -> unconnected-(J9-Pad13)
- U1 pad 8: Net-(U1-Pad8) -> unconnected-(U1-Pad8)
- U2 pad 4: Net-(U2-Pad4) -> unconnected-(U2-Pad4)
- U2 pad 6: Net-(U2-Pad6) -> unconnected-(U2-Pad6)
- U4 pad 13: Net-(U4-Pad13) -> unconnected-(U4-Pad13)
- U4 pad 15: Net-(U4-Pad15) -> unconnected-(U4-Pad15)
- U4 pad 16: Net-(U4-Pad16) -> unconnected-(U4-Pad16)
- U4 pad 17: Net-(U4-Pad17) -> unconnected-(U4-Pad17)
- U4 pad 18: Net-(U4-Pad18) -> unconnected-(U4-Pad18)
- U4 pad 7: Net-(U4-Pad7) -> unconnected-(U4-Pad7)
- U4 pad 9: Net-(U4-Pad9) -> unconnected-(U4-Pad9)
- U5 pad 6: Net-(J9-Pad5) -> 3.3V_SDCARD
- U6 pad 6: 3.3V_SDCARD -> Net-(J9-Pad5)
- U7 pad 1: Net-(U7-Pad1) -> unconnected-(U7-Pad1)
- U7 pad 13: Net-(U7-Pad13) -> unconnected-(U7-Pad13)
Routing:
- net GND: track 0.00 -> 137.6 mm, vias 0 -> 73
- net TIM1_CH1: track 0.00 -> 70.0 mm, vias 0 -> 3
- net SPI2_MOSI: track 0.00 -> 66.6 mm, vias 0 -> 2
- net EN: track 0.00 -> 54.2 mm, vias 0 -> 2
- net JTAG_TMS: track 0.00 -> 54.0 mm, vias 0 -> 2
- net LCD_TCH_CS: track 0.00 -> 53.9 mm, vias 0 -> 2
- net +3V3: track 0.00 -> 51.4 mm, vias 0 -> 28
- net TIM1_CH1N: track 0.00 -> 48.8 mm, vias 0 -> 2
- net JTAG_TCLK: track 0.00 -> 46.9 mm, vias 0 -> 2
- net JTAG_TDO: track 0.00 -> 46.8 mm, vias 0 -> 2
- net JTAG_TDI: track 0.00 -> 46.2 mm, vias 0 -> 2
- net +5V: track 0.00 -> 44.3 mm, vias 0 -> 1
- net LCD_RST: track 0.00 -> 41.7 mm
- net SPI2_SCK: track 0.00 -> 40.0 mm, vias 0 -> 3
- net LCD_DC: track 0.00 -> 39.7 mm
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- added copper zone on F.Cu, net +3V3
- added copper zone on In2.Cu, net +3V3
- added copper zone on F.Cu, net GND
- added copper zone on In1.Cu, net GND
Other:
- outline, holes or cut-outs redrawn
- net class Default removed

Commit message: fertig
Connections:
- Q1 pad 1: DW01A_OD -> DW01A_OC
- Q2 pad 1: DW01A_OC -> DW01A_OD
Routing:
- net DW01A_OD: track 6.13 -> 2.50 mm, vias 2 -> 0
- net EN: vias 2 -> 1
Other:
- outline, holes or cut-outs redrawn
- board text added: "+"
- board text added: "-"
- board text added: "3.3V"
- board text added: "BATTERY"
- board text added: "BOOT"
- board text added: "BUZZER"
- board text added: "DC"
- board text added: "GPS CONN"
- board text added: "GPS PPS"
- board text added: "INPUT BUTTON"
- board text added: "JLCJLCJLCJLC"
- board text added: "JTAG"
- board text added: "JUMPER"
- board text added: "LCD CONNECTOR"
- board text added: "LCD CS"
- board text added: "LED CHRG"
- board text added: "LED STBY"
- board text added: "MISO"
- board text added: "MOSI"
- board text added: "POWER"
- board text added: "POWER BUTTON"
- board text added: "RESET"
- board text added: "RST"
- board text added: "SCK"
- board text added: "SD CARD"
- board text added: "SW"
- board text added: "TCH CS"
- board text added: "TCLK"
- board text added: "TDI"
- board text added: "TDO"
- board text added: "TMS"
- board text added: "UNSW"
- board text added: "USB"
- board text added: "Variometer | V1.0"

Commit message: Variometer bestellt
Parts:
- added TP10: TP_SPI1_MISO, TestPoint:TestPoint_Pad_D1.0mm, B.Cu at (51.0, 68.6)
- added TP11: TP_PresSens_CS, TestPoint:TestPoint_Pad_D1.0mm, B.Cu at (53.4, 68.3)
- added TP2: TP_3.3V_SD-Card, TestPoint:TestPoint_Pad_D1.0mm, F.Cu at (28.2, 35.1)
- added TP3: TP_USB_D+, TestPoint:TestPoint_Pad_D1.0mm, F.Cu at (48.1, 64.2)
- added TP4: TP_USB_D-, TestPoint:TestPoint_Pad_D1.0mm, F.Cu at (45.7, 67.9)
- added TP5: TP_BATTERY, TestPoint:TestPoint_Pad_D1.0mm, F.Cu at (70.6, 80.8)
- added TP6: TP_TX, TestPoint:TestPoint_Pad_D1.0mm, F.Cu at (29.6, 72.1)
- added TP7: TP_RX, TestPoint:TestPoint_Pad_D1.0mm, F.Cu at (27.8, 73.7)
- added TP8: TP_SPI1_SCK, TestPoint:TestPoint_Pad_D1.0mm, B.Cu at (48.8, 68.7)
- added TP9: TP_SPI1_MOSI, TestPoint:TestPoint_Pad_D1.0mm, B.Cu at (45.3, 71.4)
- D4: value GREEN -> RED
- R39: value 4.7k -> 0k; footprint Resistor_SMD:R_0402_1005Metric -> Resistor_SMD:R_0805_2012Metric
- TP1: footprint Connector_Pin:Pin_D0.7mm_L6.5mm_W1.8mm_FlatFork -> TestPoint:TestPoint_Pad_D1.5mm
- moved TP1 2.08 mm to (57.5, 36.0)
- moved SW2 0.36 mm to (60.1, 80.7)
- moved R39 0.32 mm to (62.0, 78.1)
Routing:
- net USART2_RX: track 17.0 -> 29.4 mm, vias 2 -> 4
- net USART2_TX: track 19.3 -> 26.2 mm, vias 2 -> 3
- net BAT_ADC: track 37.4 -> 43.7 mm, vias 2 -> 3
- net 3.3V_SDCARD: track 28.5 -> 34.2 mm, vias 2 -> 3
- net USB_D+: track 34.2 -> 36.2 mm
- net +3V3: track 51.1 -> 52.6 mm, vias 28 -> 29
- net SPI1_MISO: track 35.0 -> 36.4 mm
- net USB_D-: track 35.2 -> 36.6 mm
- net PresSens_CS: track 21.0 -> 22.4 mm
- net SPI1_MOSI: track 31.8 -> 33.1 mm
- net SPI1_SCK: track 32.0 -> 33.1 mm
- net EN: track 54.2 -> 54.9 mm
Other:
- outline, holes or cut-outs redrawn
- board text added: "3.3V SD"
- board text added: "D-"
- board text added: "P_CS"
- board text added: "RX"
- board text added: "TX"
- board text added: "V+"
