File: Hardware/VariometerV2.kicad_sch (KiCad schematic)
At the start: 107 parts, among them IC1 TP4056, IC2 DW01A-G, IC3 ESP32-S3-WROOM-1, J1 LED_CHRG, J2 LED_STBY, J3 TFT_LCD_CONNECTOR, J4 Conn_01x02_Male, J5 SWD, J6 USB3135-30-A, J7 5-1814832-2, J8 Conn_02x01, J9 TFP09-2-12B, Q1 AO3400A, Q10 AO3400A, Q2 AO3400A, Q3 AO3401A, Q4 AO3400A, Q5 AO3401A, Q6 AO3400A, Q7 AO3401A, Q8 AO3400A, Q9 AO3401A, SW1 SW_Push, SW2 Switch_SW_Push, SW3 Switch_SW_Push, SW4 SW_Push, U1 TPS76801QDR, U2 SRV05-4, U4 ATGM336H-5N31, U5 SRV05-4, U6 SRV05-4, U7 BMI088, U8 MS5611-01BA

Commit message: fertig
Parts:
- C1, C10, C13, C18, C19, C2, C20, C21, C5, C7: JLCPCB Part # (none) -> C14663
- C11, C4: JLCPCB Part # (none) -> C52923
- C12, C15, C3, C6, C8, C9: JLCPCB Part # (none) -> C19702
- C16, C17: JLCPCB Part # (none) -> C12530
- D1, D2, D3: JLCPCB Part # (none) -> C8598
- D4: value GREEN -> RED; JLCPCB Part # (none) -> C2286
- D5: JLCPCB Part # (none) -> C72041
- F1: JLCPCB Part # (none) -> C516069
- FB1: JLCPCB Part # (none) -> C1002
- IC1: JLCPCB Part # (none) -> C16581
- IC2: JLCPCB Part # (none) -> C61503
- IC3: JLCPCB Part # (none) -> C2913198
- L1: JLCPCB Part # (none) -> C346317
- Q1, Q10, Q2, Q4, Q6, Q8: JLCPCB Part # (none) -> C20917
- Q3, Q5, Q7, Q9: JLCPCB Part # (none) -> AO3401A
- R1: JLCPCB Part # (none) -> C22765
- R10: JLCPCB Part # (none) -> C23196
- R11: JLCPCB Part # (none) -> C22967
- R12, R17: JLCPCB Part # (none) -> C22843
- R13, R38: JLCPCB Part # (none) -> C26083
- R14, R16, R24, R26, R27, R28, R29, R30, R31, R32, R33, R34, R36, R37: JLCPCB Part # (none) -> C25744
- R15: JLCPCB Part # (none) -> C25779
- R18, R6: JLCPCB Part # (none) -> C25804
- R19, R39: JLCPCB Part # (none) -> C25900
- R2, R25, R4, R5: JLCPCB Part # (none) -> C21190
- R20, R21, R22, R23, R35: JLCPCB Part # (none) -> C25092
- R3: JLCPCB Part # (none) -> C22775
- R7, R9: JLCPCB Part # (none) -> C25803
- R8: JLCPCB Part # (none) -> C23024
- U1: JLCPCB Part # (none) -> C20030
- U2, U5, U6: JLCPCB Part # (none) -> C85364
- U4: JLCPCB Part # (none) -> C90770
- U7: JLCPCB Part # (none) -> C194919
- U8: JLCPCB Part # (none) -> C37148
Connections:
- net DW01A_OC: now also Q1.1 (G); no longer Q2.1 (G)
- net DW01A_OD: now also Q2.1 (G); no longer Q1.1 (G)

Commit message: Variometer bestellt
Parts:
- added TP10: TP_SPI1_MISO, TestPoint:TestPoint_Pad_D1.0mm, symbol Connector:TestPoint
- added TP11: TP_PresSens_CS, TestPoint:TestPoint_Pad_D1.0mm, symbol Connector:TestPoint
- added TP2: TP_3.3V_SD-Card, TestPoint:TestPoint_Pad_D1.0mm, symbol Connector:TestPoint
- added TP3: TP_USB_D+, TestPoint:TestPoint_Pad_D1.0mm, symbol Connector:TestPoint
- added TP4: TP_USB_D-, TestPoint:TestPoint_Pad_D1.0mm, symbol Connector:TestPoint
- added TP5: TP_BATTERY, TestPoint:TestPoint_Pad_D1.0mm, symbol Connector:TestPoint
- added TP6: TP_TX, TestPoint:TestPoint_Pad_D1.0mm, symbol Connector:TestPoint
- added TP7: TP_RX, TestPoint:TestPoint_Pad_D1.0mm, symbol Connector:TestPoint
- added TP8: TP_SPI1_SCK, TestPoint:TestPoint_Pad_D1.0mm, symbol Connector:TestPoint
- added TP9: TP_SPI1_MOSI, TestPoint:TestPoint_Pad_D1.0mm, symbol Connector:TestPoint
- C1, C10, C13, C18, C19, C2, C20, C21, C5, C7: JLCPCB Part # C14663 -> C307331
- Q3, Q5, Q7, Q9: JLCPCB Part # AO3401A -> C15127
- R39: value 4.7k -> 0k; footprint Resistor_SMD:R_0402_1005Metric -> Resistor_SMD:R_0805_2012Metric; JLCPCB Part # C25900 -> (none)
- TP1: footprint Connector_Pin:Pin_D0.7mm_L6.5mm_W1.8mm_FlatFork -> TestPoint:TestPoint_Pad_D1.5mm
Connections:
- net 3.3V_SDCARD: now also TP2.1
- net BAT_ADC: now also TP5.1
- net PresSens_CS: now also TP11.1
- net SPI1_MISO: now also TP10.1
- net SPI1_MOSI: now also TP9.1
- net SPI1_SCK: now also TP8.1
- net USART2_RX: now also TP7.1
- net USART2_TX: now also TP6.1
- net USB_D+: now also TP3.1
- net USB_D-: now also TP4.1
