File: Hardware/GPS_Test/MAX_M10S_Breakout/MAX_M10S_Breakout.kicad_pcb (KiCad board)
At the start: 2 copper layers, 14 parts, among them J1 U.FL-R-SMT(01), J2 Conn_01x10, U1 MAX-M10S

Commit message: MAX-M10S continue
Parts:
- moved J2 32.6 mm to (84.5, 65.8), turned to 90 degrees
- moved D1 27.1 mm to (83.1, 46.4), turned to 180 degrees
- moved C1 26.0 mm to (100.1, 49.3), turned to 180 degrees
- moved JP1 26.0 mm to (103.8, 55.4), turned to 90 degrees
- moved L1 24.1 mm to (104.1, 51.8)
- moved R4 23.0 mm to (82.9, 50.9), turned to 180 degrees
- moved R2 21.9 mm to (105.0, 62.4), turned to 180 degrees
- moved J1 21.7 mm to (108.0, 55.4), turned to -90 degrees
- moved R1 21.0 mm to (100.1, 51.7)
- moved C4 20.0 mm to (83.2, 54.5), turned to 180 degrees
- moved R3 19.1 mm to (101.0, 62.4), turned to 180 degrees
- moved C3 12.5 mm to (86.6, 60.8), turned to -90 degrees
- moved C2 11.3 mm to (83.9, 57.8), turned to -90 degrees

Commit message: Weiter Max M10S
Parts:
- moved R2 11.1 mm to (94.0, 63.0), turned to -90 degrees
- moved D1 4.57 mm to (87.6, 46.2)
- moved R3 3.72 mm to (97.9, 64.5)
- moved J2 2.87 mm to (83.8, 68.6)
- moved JP1 0.77 mm to (103.6, 54.6)
Routing:
- net ~{RESET}: track 0.00 -> 33.0 mm
- net SCL: track 0.00 -> 25.3 mm, vias 0 -> 2
- net ~{SAFE}: track 0.00 -> 24.6 mm, vias 0 -> 2
- net INT: track 0.00 -> 24.4 mm, vias 0 -> 2
- net SDA: track 0.00 -> 21.1 mm
- net TX: track 0.00 -> 20.8 mm
- net +BATT: track 0.00 -> 19.9 mm, vias 0 -> 1
- net RX: track 0.00 -> 18.7 mm
- net +3.3V: track 0.00 -> 15.0 mm, vias 0 -> 4
- net GND: track 0.00 -> 14.6 mm, vias 0 -> 10
- net Net-(J1-SIG): track 0.00 -> 10.8 mm
- net Net-(D1-A): track 0.00 -> 6.64 mm
- net Net-(C1-Pad1): track 0.00 -> 4.57 mm
- net Net-(U1-VCC_RF): track 0.00 -> 3.66 mm
- net PPS: track 0.00 -> 3.39 mm
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- added copper zone on In2.Cu, net +3.3V
- added copper zone on In1.Cu, net GND
Other:
- board outline added: 32.1 x 28.6 mm
- copper layers 2 -> 4

Commit message: Continue GPS Hardware
Parts:
- added JP2: JMP, Jumper:SolderJumper-2_P1.3mm_Open_Pad1.0x1.5mm, F.Cu at (82.7, 50.5)
- C1, C3: footprint Capacitor_SMD:C_0805_2012Metric -> Capacitor_SMD:C_0603_1608Metric
- C2, C4: footprint Capacitor_SMD:C_0805_2012Metric -> Capacitor_SMD:C_0402_1005Metric
- D1: footprint LED_SMD:LED_0805_2012Metric -> LED_SMD:LED_0603_1608Metric
- L1: footprint Inductor_SMD:L_0805_2012Metric -> Inductor_SMD:L_0603_1608Metric
- R1, R2, R3: footprint Resistor_SMD:R_0805_2012Metric -> Resistor_SMD:R_0402_1005Metric
- R4: footprint Resistor_SMD:R_0805_2012Metric -> Resistor_SMD:R_0603_1608Metric
- moved C1 4.76 mm to (104.8, 48.8)
- moved C4 4.42 mm to (87.6, 54.5)
- moved C2 4.41 mm to (88.0, 56.2)
- moved R1 4.03 mm to (104.1, 51.5)
- moved R4 3.97 mm to (84.0, 47.1), turned to 0 degrees
- moved U1 3.41 mm to (94.8, 53.4)
- moved J1 1.64 mm to (108.4, 57.0)
- moved JP1 1.52 mm to (104.1, 56.0)
- moved L1 1.33 mm to (104.2, 53.1)
- moved C3 1.31 mm to (87.7, 60.1)
- moved D1 0.89 mm to (87.3, 47.0)
Connections:
- R4 pad 1: PPS -> Net-(JP2-A)
Routing:
- net ~{RESET}: track 33.0 -> 0.00 mm
- net SCL: track 25.3 -> 0.00 mm, vias 2 -> 0
- net ~{SAFE}: track 24.6 -> 0.00 mm, vias 2 -> 0
- net INT: track 24.4 -> 0.00 mm, vias 2 -> 0
- net SDA: track 21.1 -> 0.00 mm
- net TX: track 20.8 -> 0.00 mm
- net +BATT: track 19.9 -> 0.00 mm, vias 1 -> 0
- net RX: track 18.7 -> 0.00 mm
- net +3.3V: track 15.0 -> 0.00 mm, vias 4 -> 0
- net Net-(D1-A): track 6.64 -> 0.00 mm
- net GND: track 14.6 -> 8.87 mm, vias 10 -> 5
- net Net-(J1-SIG): track 10.8 -> 7.36 mm
- net PPS: track 3.39 -> 0.00 mm
- net Net-(U1-VCC_RF): track 3.66 -> 4.78 mm
- net Net-(C1-Pad1): track 4.57 -> 5.29 mm
Other:
- outline, holes or cut-outs redrawn

Commit message: Max-M10S finished
Parts:
- added C5: 4.7uF, Capacitor_SMD:C_0603_1608Metric, F.Cu at (84.2, 54.1)
- moved JP2 1.66 mm to (84.2, 49.8)
- moved J1 1.31 mm to (107.1, 57.0)
- moved J2 1.27 mm to (85.1, 68.4)
- moved JP1 0.82 mm to (103.3, 56.2)
- moved R4 0.70 mm to (84.0, 46.4)
- moved C4 0.66 mm to (87.5, 53.8), turned to 90 degrees
- moved D1 0.51 mm to (87.4, 46.5)
- moved C2 0.48 mm to (87.6, 56.0), turned to 180 degrees
Routing:
- net ~{SAFE}: track 0.00 -> 25.6 mm, vias 0 -> 2
- net TX: track 0.00 -> 23.3 mm, vias 0 -> 2
- net SDA: track 0.00 -> 22.2 mm, vias 0 -> 2
- net ~{RESET}: track 0.00 -> 21.2 mm
- net +BATT: track 0.00 -> 20.6 mm
- net INT: track 0.00 -> 20.4 mm, vias 0 -> 1
- net SCL: track 0.00 -> 20.2 mm, vias 0 -> 2
- net RX: track 0.00 -> 19.7 mm, vias 0 -> 1
- net +3.3V: track 0.00 -> 10.8 mm, vias 0 -> 3
- net GND: track 8.87 -> 18.7 mm, vias 5 -> 13
- net PPS: track 0.00 -> 6.67 mm
- net Net-(JP2-A): track 0.00 -> 3.20 mm
- net Net-(D1-A): track 0.00 -> 1.90 mm
- net Net-(J1-SIG): track 7.36 -> 6.05 mm
Other:
- board size 32.1 x 28.6 mm -> 30.5 x 27.9 mm
- board text added: "+"
- board text added: "-"
- board text added: "BATT"
- board text added: "INT"
- board text added: "Max-M10S Breakout Board"
- board text added: "RX"
- board text added: "SCL"
- board text added: "SDA"
- board text added: "TX"
- board text added: "~{RESET}"
- board text added: "~{SAFE}"
