File: Hardware/GPS_Test/MAX_M10S_Breakout/MAX_M10S_Breakout.kicad_sch (KiCad schematic)
At the start: 14 parts, among them J1 U.FL-R-SMT(01), J2 Conn_01x10, U1 MAX-M10S

Commit message: Continue GPS Hardware
Parts:
- added JP2: JMP, Jumper:SolderJumper-2_P1.3mm_Open_Pad1.0x1.5mm, symbol Jumper:SolderJumper_2_Open
- C1: footprint Capacitor_SMD:C_0805_2012Metric -> Capacitor_SMD:C_0603_1608Metric; LCSC Part C1710 -> C57112
- C2, C4: footprint Capacitor_SMD:C_0805_2012Metric -> Capacitor_SMD:C_0402_1005Metric; LCSC Part C28233 -> C307331
- C3: footprint Capacitor_SMD:C_0805_2012Metric -> Capacitor_SMD:C_0603_1608Metric; LCSC Part C15850 -> C19702
- D1: footprint LED_SMD:LED_0805_2012Metric -> LED_SMD:LED_0603_1608Metric; LCSC Part C2296 -> C72041
- L1: footprint Inductor_SMD:L_0805_2012Metric -> Inductor_SMD:L_0603_1608Metric; LCSC Part C98992 -> C148128
- R1: footprint Resistor_SMD:R_0805_2012Metric -> Resistor_SMD:R_0402_1005Metric; LCSC Part C17415 -> C25077
- R2, R3: footprint Resistor_SMD:R_0805_2012Metric -> Resistor_SMD:R_0402_1005Metric; LCSC Part C17673 -> C25900
- R4: footprint Resistor_SMD:R_0805_2012Metric -> Resistor_SMD:R_0603_1608Metric; LCSC Part C17513 -> C21190
Connections:
- net PPS: now also JP2.2 (B); no longer R4.1
- new net: JP2.1 (A), R4.1
Other:
- moved on the sheet: D1, R4
Changed lines of the file:
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@@
-    (stroke (width 0) (type default))
-  )
-  (wire (pts (xy 34.29 90.17) (xy 34.29 92.71))
     (stroke (width 0) (type default))
   )
@@
     (stroke (width 0) (type default))
   )
-  (wire (pts (xy 34.29 81.28) (xy 34.29 85.09))
+  (wire (pts (xy 34.29 91.44) (xy 34.29 92.71))
     (stroke (width 0) (type default))
   )
@@
     (stroke (width 0) (type default))
   )
-  (wire (pts (xy 34.29 100.33) (xy 34.29 102.87))
+  (wire (pts (xy 34.29 105.41) (xy 34.29 107.95))
     (stroke (width 0) (type default))
   )
@@
   )
   (wire (pts (xy 67.31 45.72) (xy 69.85 45.72))
+    (stroke (width 0) (type default))
+  )
+  (wire (pts (xy 34.29 80.01) (xy 34.29 83.82))
     (stroke (width 0) (type default))
   )
@@
     )
   )
-  (global_label "PPS" (shape input) (at 34.29 81.28 180) (fields_autoplaced)
-    (effects (font (size 1.27 1.27)) (justify right))
-    (property "Intersheetrefs" "${INTERSHEET_REFS}" (at 27.6347 81.28 0)
+  (global_label "PPS" (shape input) (at 34.29 80.01 180) (fields_autoplaced)
+    (effects (font (size 1.27 1.27)) (justify right))
+    (property "Intersheetrefs" "${INTERSHEET_REFS}" (at 27.6347 80.01 0)
       (effects (font (size 1.27 1.27)) (justify right) hide)
     )
@@
     )
   )
+  (symbol (lib_id "Jumper:SolderJumper_2_Open") (at 34.29 87.63 90) (unit 1)
+    (in_bom yes) (on_board yes) (dnp no) (fields_autoplaced)
+    (property "Reference" "JP2" (at 36.83 86.995 90)
+      (effects (font (size 1.27 1.27)) (justify right))
+    )
+    (property "Value" "JMP" (at 36.83 89.535 90)
+      (effects (font (size 1.27 1.27)) (justify right))
+    )
+    (property "Footprint" "Jumper:SolderJumper-2_P1.3mm_Open_Pad1.0x1.5mm" (at 34.29 87.63 0)
+      (effects (font (size 1.27 1.27)) hide)
+    )
+    (property "Datasheet" "~" (at 34.29 87.63 0)
+      (effects (font (size 1.27 1.27)) hide)
+    )
+    (property "LCSC Part" "" (at 34.29 87.63 0)
+      (effects (font (size 1.27 1.27)) hide)
+    )
+    (pin "1")
+    (pin "2")
+    (instances
+      (project "MAX_M10S_Breakout"
+        (path "/2b6017bd-63dd-43f9-96e5-8753c63bb938"
+          (reference "JP2") (unit 1)
+        )
+      )
+    )
+  )
   (symbol (lib_id "power:+3.3V") (at 39.37 48.26 0) (unit 1)
     (in_bom yes) (on_board yes) (dnp no) (fields_autoplaced)
@@
       (effects (font (size 1.27 1.27)) (justify left))
     )
-    (property "Footprint" "Resistor_SMD:R_0805_2012Metric" (at 87.63 57.15 0)
+    (property "Footprint" "Resistor_SMD:R_0402_1005Metric" (at 87.63 57.15 0)
       (effects (font (size 1.27 1.27)) hide)
     )
@@
       (effects (font (size 1.27 1.27)) hide)
     )
-    (property "LCSC Part" "C17415" (at 87.63 57.15 0)
+    (property "LCSC Part" "C25077" (at 87.63 57.15 0)
       (effects (font (size 1.27 1.27)) hide)
     )
@@
       (effects (font (size 1.27 1.27)) (justify left))
     )
-    (property "Footprint" "Capacitor_SMD:C_0805_2012Metric" (at 41.91 52.07 0)
+    (property "Footprint" "Capacitor_SMD:C_0603_1608Metric" (at 41.91 52.07 0)
       (effects (font (size 1.27 1.27)) hide)
     )
@@
       (effects (font (size 1.27 1.27)) hide)
     )
-    (property "LCSC Part" "C15850" (at 41.91 52.07 0)
+    (property "LCSC Part" "C19702" (at 41.91 52.07 0)
       (effects (font (size 1.27 1.27)) hide)
     )
@@
       (effects (font (size 1.27 1.27)) (justify left))
     )
-    (property "Footprint" "Resistor_SMD:R_0805_2012Metric" (at 30.48 66.04 0)
+    (property "Footprint" "Resistor_SMD:R_0402_1005Metric" (at 30.48 66.04 0)
       (effects (font (size 1.27 1.27)) hide)
     )
@@
       (effects (font (size 1.27 1.27)) hide)
     )
-    (property "LCSC Part" "C17673" (at 30.48 66.04 0)
+    (property "LCSC Part" "C25900" (at 30.48 66.04 0)
       (effects (font (size 1.27 1.27)) hide)
     )
@@
       (effects (font (size 1.27 1.27)) (justify left))
     )
-    (property "Footprint" "Capacitor_SMD:C_0805_2012Metric" (at 52.07 52.07 0)
+    (property "Footprint" "Capacitor_SMD:C_0402_1005Metric" (at 52.07 52.07 0)
       (effects (font (size 1.27 1.27)) hide)
     )
@@
       (effects (font (size 1.27 1.27)) hide)
     )
-    (property "LCSC Part" "C28233" (at 52.07 52.07 0)
+    (property "LCSC Part" "C307331" (at 52.07 52.07 0)
       (effects (font (size 1.27 1.27)) hide)
     )
@@
       (effects (font (size 1.27 1.27)) (justify left))
     )
-    (property "Footprint" "Capacitor_SMD:C_0805_2012Metric" (at 69.85 48.26 0)
+    (property "Footprint" "Capacitor_SMD:C_0402_1005Metric" (at 69.85 48.26 0)
       (effects (font (size 1.27 1.27)) hide)
     )
@@
       (effects (font (size 1.27 1.27)) hide)
     )
-    (property "LCSC Part" "C28233" (at 69.85 48.26 0)
+    (property "LCSC Part" "C307331" (at 69.85 48.26 0)
       (effects (font (size 1.27 1.27)) hide)
     )
@@
       (effects (font (size 1.27 1.27)) (justify left))
     )
-    (property "Footprint" "Capacitor_SMD:C_0805_2012Metric" (at 96.52 68.58 0)
+    (property "Footprint" "Capacitor_SMD:C_0603_1608Metric" (at 96.52 68.58 0)
       (effects (font (size 1.27 1.27)) hide)
     )
@@
       (effects (font (size 1.27 1.27)) hide)
     )
-    (property "LCSC Part" "C1710" (at 96.52 68.58 0)
+    (property "LCSC Part" "C57112" (at 96.52 68.58 0)
       (effects (font (size 1.27 1.27)) hide)
     )
@@
     )
   )
-  (symbol (lib_id "Device:R_Small") (at 34.29 87.63 0) (unit 1)
+  (symbol (lib_id "Device:R_Small") (at 34.29 95.25 0) (unit 1)
     (in_bom yes) (on_board yes) (dnp no)
-    (property "Reference" "R4" (at 36.83 86.995 0)
-      (effects (font (size 1.27 1.27)) (justify left))
-    )
-    (property "Value" "1k" (at 36.83 88.9 0)
-      (effects (font (size 1.27 1.27)) (justify left))
-    )
-    (property "Footprint" "Resistor_SMD:R_0805_2012Metric" (at 34.29 87.63 0)
-      (effects (font (size 1.27 1.27)) hide)
-    )
-    (property "Datasheet" "~" (at 34.29 87.63 0)
-      (effects (font (size 1.27 1.27)) hide)
-    )
-    (property "LCSC Part" "C17513" (at 34.29 87.63 0)
+    (property "Reference" "R4" (at 36.83 94.615 0)
+      (effects (font (size 1.27 1.27)) (justify left))
+    )
+    (property "Value" "1k" (at 36.83 96.52 0)
+      (effects (font (size 1.27 1.27)) (justify left))
+    )
+    (property "Footprint" "Resistor_SMD:R_0603_1608Metric" (at 34.29 95.25 0)
+      (effects (font (size 1.27 1.27)) hide)
+    )
+    (property "Datasheet" "~" (at 34.29 95.25 0)
+      (effects (font (size 1.27 1.27)) hide)
+    )
+    (property "LCSC Part" "C21190" (at 34.29 95.25 0)
       (effects (font (size 1.27 1.27)) hide)
     )
@@
       (effects (font (size 1.27 1.27)) (justify left))
     )
-    (property "Footprint" "Resistor_SMD:R_0805_2012Metric" (at 39.37 66.04 0)
+    (property "Footprint" "Resistor_SMD:R_0402_1005Metric" (at 39.37 66.04 0)
       (effects (font (size 1.27 1.27)) hide)
     )
@@
       (effects (font (size 1.27 1.27)) hide)
     )
-    (property "LCSC Part" "C17673" (at 39.37 66.04 0)
+    (property "LCSC Part" "C25900" (at 39.37 66.04 0)
       (effects (font (size 1.27 1.27)) hide)
     )
@@
     )
   )
-  (symbol (lib_id "Device:LED") (at 34.29 96.52 90) (unit 1)
-    (in_bom yes) (on_board yes) (dnp no) (fields_autoplaced)
-    (property "Reference" "D1" (at 38.1 97.4725 90)
+  (symbol (lib_id "Device:LED") (at 34.29 101.6 90) (unit 1)
+    (in_bom yes) (on_board yes) (dnp no) (fields_autoplaced)
+    (property "Reference" "D1" (at 38.1 102.5525 90)
       (effects (font (size 1.27 1.27)) (justify right))
     )
-    (property "Value" "BLUE" (at 38.1 100.0125 90)
+    (property "Value" "BLUE" (at 38.1 105.0925 90)
       (effects (font (size 1.27 1.27)) (justify right))
     )
-    (property "Footprint" "LED_SMD:LED_0805_2012Metric" (at 34.29 96.52 0)
-      (effects (font (size 1.27 1.27)) hide)
-    )
-    (property "Datasheet" "~" (at 34.29 96.52 0)
-      (effects (font (size 1.27 1.27)) hide)
-    )
-    (property "LCSC Part" "C2296" (at 34.29 96.52 0)
+    (property "Footprint" "LED_SMD:LED_0603_1608Metric" (at 34.29 101.6 0)
+      (effects (font (size 1.27 1.27)) hide)
+    )
+    (property "Datasheet" "~" (at 34.29 101.6 0)
+      (effects (font (size 1.27 1.27)) hide)
+    )
+    (property "LCSC Part" "C72041" (at 34.29 101.6 0)
       (effects (font (size 1.27 1.27)) hide)
     )
@@
       (effects (font (size 1.27 1.27)) (justify left))
     )
-    (property "Footprint" "Inductor_SMD:L_0805_2012Metric" (at 87.63 64.77 0)
+    (property "Footprint" "Inductor_SMD:L_0603_1608Metric" (at 87.63 64.77 0)
       (effects (font (size 1.27 1.27)) hide)
     )
@@
       (effects (font (size 1.27 1.27)) hide)
     )
-    (property "LCSC Part" "C98992" (at 87.63 64.77 0)
+    (property "LCSC Part" "C148128" (at 87.63 64.77 0)
       (effects (font (size 1.27 1.27)) hide)
     )
@@
     )
   )
-  (symbol (lib_id "power:GND") (at 34.29 102.87 0) (unit 1)
-    (in_bom yes) (on_board yes) (dnp no) (fields_autoplaced)
-    (property "Reference" "#PWR06" (at 34.29 109.22 0)
-      (effects (font (size 1.27 1.27)) hide)
-    )
-    (property "Value" "GND" (at 34.29 107.95 0)
-      (effects (font (size 1.27 1.27)))
-    )
-    (property "Footprint" "" (at 34.29 102.87 0)
-      (effects (font (size 1.27 1.27)) hide)
-    )
-    (property "Datasheet" "" (at 34.29 102.87 0)
-      (effects (font (size 1.27 1.27)) hide)
-    )
+  (symbol (lib_id "power:GND") (at 34.29 107.95 0) (unit 1)
+    (in_bom yes) (on_board yes) (dnp no) (fields_autoplaced)
+    (property "Reference" "#PWR06" (at 34.29 114.3 0)
+      (effects (font (size 1.27 1.27)) hide)
+    )
+    (property "Value" "GND" (at 34.29 113.03 0)
+      (effects (font (size 1.27 1.27)))
+    )
+    (property "Footprint" "" (at 34.29 107.95 0)
+      (effects (font (size 1.27 1.27)) hide)
+    )
+    (property "Datasheet" "" (at 34.29 107.95 0)
+      (effects (font (size 1.27 1.27)) hide)
+    )

Commit message: Max-M10S finished
Parts:
- added C5: 4.7uF, Capacitor_SMD:C_0603_1608Metric, symbol Device:C_Small
Connections:
- net +BATT: now also C5.1
- net GND: now also C5.2
Changed lines of the file:
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@@
   (junction (at 160.02 52.07) (diameter 0) (color 0 0 0 0)
+  )
+  (junction (at 69.85 52.07) (diameter 0) (color 0 0 0 0)
+  )
+  (junction (at 69.85 45.72) (diameter 0) (color 0 0 0 0)
   )
   (junction (at 48.26 57.15) (diameter 0) (color 0 0 0 0)
@@
     (stroke (width 0) (type default))
   )
+  (wire (pts (xy 69.85 52.07) (xy 81.28 52.07))
+    (stroke (width 0) (type default))
+  )
   (wire (pts (xy 39.37 73.66) (xy 39.37 68.58))
     (stroke (width 0) (type default))
@@
     (stroke (width 0) (type default))
   )
+  (wire (pts (xy 81.28 45.72) (xy 81.28 46.99))
+    (stroke (width 0) (type default))
+  )
   (wire (pts (xy 67.31 93.98) (xy 60.96 93.98))
     (stroke (width 0) (type default))
@@
     (stroke (width 0) (type default))
   )
+  (wire (pts (xy 69.85 45.72) (xy 81.28 45.72))
+    (stroke (width 0) (type default))
+  )
   (wire (pts (xy 69.85 50.8) (xy 69.85 52.07))
     (stroke (width 0) (type default))
@@
   )
   (text "Active Antenna: JP1 closed\nPassive Antenna: JP1 open"
-    (at 83.82 52.07 0)
+    (at 95.25 54.61 0)
     (effects (font (size 1.27 1.27)) (justify left bottom))
   )
@@
         )
       )
+    )
+  )
+  (symbol (lib_id "Device:C_Small") (at 81.28 49.53 0) (unit 1)
+    (in_bom yes) (on_board yes) (dnp no)
+    (property "Reference" "C5" (at 83.82 48.26 0)
+      (effects (font (size 1.27 1.27)) (justify left))
+    )
+    (property "Value" "4.7uF" (at 83.82 50.8 0)
+      (effects (font (size 1.27 1.27)) (justify left))
+    )
+    (property "Footprint" "Capacitor_SMD:C_0603_1608Metric" (at 81.28 49.53 0)
+      (effects (font (size 1.27 1.27)) hide)
+    )
+    (property "Datasheet" "~" (at 81.28 49.53 0)
+      (effects (font (size 1.27 1.27)) hide)
+    )
+    (property "LCSC Part" "C19666" (at 81.28 49.53 0)
+      (effects (font (size 1.27 1.27)) hide)
+    )
+    (pin "1")
+    (pin "2")
+    (instances
+      (project "MAX_M10S_Breakout"
+        (path "/2b6017bd-63dd-43f9-96e5-8753c63bb938"
+          (reference "C5") (unit 1)
+        )
+      )
