File: Hardware/GPS_Test/L96-M33_Breakout/L96-M33_Breakout.kicad_pcb (KiCad board)
At the start: 2 copper layers, 18 parts, among them IC1 L96-M33, J1 U.FL-R-SMT(01), J2 Conn_01x11

Commit message: Fertig GPS Test Platine
Parts:
- moved C5 77.4 mm to (141.0, 60.5), turned to 90 degrees
- moved D1 77.3 mm to (137.8, 48.5), turned to 180 degrees
- moved C4 63.8 mm to (132.5, 59.0), turned to 180 degrees
- moved C2 63.7 mm to (132.5, 57.5), turned to 180 degrees
- moved R4 60.2 mm to (137.8, 50.5), turned to 180 degrees
- moved J2 56.0 mm to (134.6, 74.5), turned to -90 degrees
- moved C3 54.6 mm to (138.7, 56.7), turned to 180 degrees
- moved R3 53.1 mm to (138.5, 70.0)
- moved JP4 53.1 mm to (137.8, 52.8), turned to 180 degrees
- moved IC1 52.2 mm to (123.8, 60.0)
- moved R2 52.0 mm to (137.0, 65.5)
- moved J1 41.1 mm to (105.5, 59.3), turned to 90 degrees
- moved L1 37.3 mm to (108.2, 63.6), turned to 180 degrees
- moved JP1 29.0 mm to (115.2, 56.4), turned to -90 degrees
- moved C1 26.4 mm to (109.0, 55.8)
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Routing:
- net GND: track 0.00 -> 55.2 mm, vias 0 -> 22
- net +BATT: track 0.00 -> 36.8 mm
- net SCL: track 0.00 -> 26.1 mm, vias 0 -> 1
- net PPS: track 0.00 -> 25.3 mm, vias 0 -> 2
- net SDA: track 0.00 -> 24.4 mm
- net JAM_DET: track 0.00 -> 19.9 mm, vias 0 -> 2
- net +3.3V: track 0.00 -> 19.7 mm, vias 0 -> 6
- net FORCE_ON: track 0.00 -> 15.9 mm, vias 0 -> 2
- net GEO_FENCE: track 0.00 -> 15.2 mm, vias 0 -> 1
- net 3D_FIX: track 0.00 -> 13.3 mm, vias 0 -> 2
- net TX: track 0.00 -> 12.1 mm, vias 0 -> 1
- net RX: track 0.00 -> 10.8 mm
- net RF_IN: track 0.00 -> 7.12 mm
- net Net-(J1-SIG): track 0.00 -> 7.11 mm
- net RF_OUT: track 0.00 -> 3.78 mm
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- added copper zone on In2.Cu, net +3.3V
- added copper zone on In1.Cu, net GND
Other:
- board outline added: 45 x 31 mm
- copper layers 2 -> 4
- board text added: "+"
- board text added: "-"
- board text added: "3d_F"
- board text added: "BATT+"
- board text added: "FOR_ON"
- board text added: "G_FE"
- board text added: "JAM_D"
- board text added: "L96-M33 Breakout Board"
- board text added: "RX"
- board text added: "SCL"
- board text added: "SDA"
- board text added: "TX"
