File: Hardware/GPS_Test/L96-M33_Breakout/L96-M33_Breakout.kicad_sch (KiCad schematic)
At the start: 14 parts, among them IC1 L96-M33, J1 U.FL-R-SMT(01), J2 Conn_01x12

Commit message: Continue GPS Hardware
Parts:
- removed J2: Conn_01x12, symbol Connector_Generic:Conn_01x12
- added C5: 4.7uF, Capacitor_SMD:C_0805_2012Metric, symbol Device:C_Small
- added D1: BLUE, LED_SMD:LED_0603_1608Metric, symbol Device:LED
- added J2: Conn_01x11, Connector_PinHeader_2.54mm:PinHeader_1x11_P2.54mm_Vertical, symbol Connector_Generic:Conn_01x11
- added JP2: JMP, Jumper:SolderJumper-2_P1.3mm_Open_Pad1.0x1.5mm, symbol Jumper:SolderJumper_2_Open
- added R4: 1k, Resistor_SMD:R_0603_1608Metric, symbol Device:R_Small
- C1: footprint (none) -> Capacitor_SMD:C_0603_1608Metric; LCSC Part (none) -> C14858
- C2, C4: footprint (none) -> Capacitor_SMD:C_0402_1005Metric; LCSC Part (none) -> C1525
- C3: footprint (none) -> Capacitor_SMD:C_0603_1608Metric; LCSC Part (none) -> C19702
- IC1: footprint L96 -> SamacSys_Parts:L96
- J1: footprint HRS_U.FL-R-SMT(01) -> SamacSys_Parts:HRS_U.FL-R-SMT(01)
- JP1, JP2, JP3: footprint (none) -> Jumper:SolderJumper-2_P1.3mm_Open_Pad1.0x1.5mm
- L1: footprint (none) -> Inductor_SMD:L_0805_2012Metric; LCSC Part (none) -> C162657
- R1: footprint (none) -> Resistor_SMD:R_0603_1608Metric; LCSC Part (none) -> C22859
- R2, R3: footprint (none) -> Resistor_SMD:R_0603_1608Metric; LCSC Part (none) -> C23162
Connections:
- net +3.3V: now also J2.1 (Pin_1)
- net +BATT: now also C5.2, J2.2 (Pin_2)
- net 3D_FIX: now also J2.3 (Pin_3)
- net FORCE_ON: now also J2.10 (Pin_10)
- net GEO_FENCE: now also J2.7 (Pin_7)
- net GND: now also C5.1, D1.1 (K), J2.11 (Pin_11)
- net JAM_DET: now also J2.6 (Pin_6)
- net PPS: now also JP2.2 (B)
- net RX: now also J2.9 (Pin_9)
- net SCL: now also J2.5 (Pin_5)
- net SDA: now also J2.4 (Pin_4)
- net TX: now also J2.8 (Pin_8)
- new net: D1.2 (A), R4.2
- new net: JP2.1 (A), R4.1
Other:
- moved on the sheet: C3, C4

Commit message: Fertig GPS Test Platine
Parts:
- R4: LCSC Part C17513 -> C21190
Changed lines of the file:
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@@
       (effects (font (size 1.27 1.27)) hide)
     )
-    (property "LCSC Part" "C17513" (at 77.47 104.14 0)
+    (property "LCSC Part" "C21190" (at 77.47 104.14 0)
       (effects (font (size 1.27 1.27)) hide)
     )

Commit message: GPS Test Files
Other:
- note added: "Active Antenna: JP2, JP3 closed, JP1 open Passiv Antenna: JP2 closed, JP1, JP3 open Internal Antenna: JP1 closed, JP2, JP3 open"
- note removed: "Active Antenna: JP2, JP3 closed, JP1 open Passiv Antenna: JP2 closed, JP1, JP3 open Internal Antenna: JP1 closed, JP2, JP3 closed"
Changed lines of the file:
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@@
     (stroke (width 0) (type default))
   )
-  (text "Active Antenna: JP2, JP3 closed, JP1 open\nPassiv Antenna: JP2 closed, JP1, JP3 open\nInternal Antenna: JP1 closed, JP2, JP3 closed"
+  (text "Active Antenna: JP2, JP3 closed, JP1 open\nPassiv Antenna: JP2 closed, JP1, JP3 open\nInternal Antenna: JP1 closed, JP2, JP3 open"
     (at 22.86 30.48 0)
     (effects (font (size 1.27 1.27)) (justify left bottom))
