File: Hardware/Version 2.1/VariometerV2.2.1/VariometerV2.2.1.kicad_sch (KiCad schematic)
At the start: 9 parts, among them IC1 ESP32-S3-WROOM, SW1 Switch_SW_Push, SW2 Switch_SW_Push

Commit message: Start Board Devlopment
Parts:
- added J1: USB_C_Receptacle_USB2.0, symbol Connector:USB_C_Receptacle_USB2.0
Connections:
- net BAT_ADC is gone; now on net SD_CD: IC1.12 (IO8)
- net BAT_MS is gone; now on net PrSen_INT: IC1.15 (IO3)
- net GPIO35 is gone; now on net LCD_CS: IC1.28 (IO35)
- net GPIO43 is gone; now on net BUTTON_4: IC1.37 (TXD0)
- net BUTTON_4: no longer IC1.25 (IO48)
- net I2C_SCL: now also IC1.34 (IO41); no longer IC1.29 (IO36)
- net I2C_SDA: now also IC1.33 (IO40); no longer IC1.30 (IO37)
- net LCD_BUSY: now also IC1.29 (IO36); no longer IC1.33 (IO40)
- net LCD_CLK: now also IC1.32 (IO39); no longer IC1.16 (IO46)
- net LCD_CS: no longer IC1.32 (IO39)
- net LCD_DC: now also IC1.31 (IO38); no longer IC1.35 (IO42)
- net LCD_DIN: now also IC1.30 (IO37); no longer IC1.34 (IO41)
- net PrSen_INT: no longer IC1.31 (IO38)
- net SD_CD: no longer IC1.22 (IO14)
- net AUDIO_EN renamed SPI_CLK
- net AUDIO_GAIN renamed CS_ACCEL
- net GPIO44: no longer names the net of IC1.36 (RXD0)
- net POSW_EN renamed SPI_MOSI
- new net: J1.A1 (GND), J1.A12 (GND), J1.B1 (GND), J1.B12 (GND)
- new net: J1.A4 (VBUS), J1.A9 (VBUS), J1.B4 (VBUS), J1.B9 (VBUS)
- new net CS_GYRO: IC1.25 (IO48)
- new net CS_PrSen: IC1.16 (IO46)
- new net POWS_EN: IC1.35 (IO42)
- new net SPI_MISO: IC1.22 (IO14)

Commit message: Start Vario PCB
Parts:
- removed J1: USB_C_Receptacle_USB2.0, symbol Connector:USB_C_Receptacle_USB2.0
Other:
- added sheet Peripherals (peripherals.kicad_sch)
- added sheet Power (Power.kicad_sch)
- moved on the sheet: C1, C2, C3, C4, C5, IC1, R1, SW1, SW2

Commit message: Develop Board
Connections:
- net SPI_MOSI is gone; now on net PrSen_INT: IC1.21 (IO13)
- net PrSen_INT: no longer IC1.15 (IO3)
- net CS_ACCEL: no longer names the net of IC1.24 (IO47)
- net CS_GYRO: no longer names the net of IC1.25 (IO48)
- net CS_PrSen renamed BAT_MS
- net I2C_SCL renamed I2C1_SCL
- net I2C_SDA renamed I2C1_SDA
- net SPI_CLK renamed I2C2_SDA
- net SPI_MISO renamed I2C2_SCL
- new net BAT_ADC: IC1.15 (IO3)
Other:
- added sheet Screen (Screen.kicad_sch)
- added sheet Sensors (Sesnors.kicad_sch)
Changed lines of the file:
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@@
     (effects (font (size 1.27 1.27)) (justify left bottom))
   )
-  (global_label "PrSen_INT" (shape input) (at 121.92 86.36 180) (fields_autoplaced)
-    (effects (font (size 1.27 1.27)) (justify right))
-    (property "Intersheetrefs" "${INTERSHEET_REFS}" (at 109.6404 86.36 0)
+  (global_label "PrSen_INT" (shape input) (at 121.92 101.6 180) (fields_autoplaced)
+    (effects (font (size 1.27 1.27)) (justify right))
+    (property "Intersheetrefs" "${INTERSHEET_REFS}" (at 109.6404 101.6 0)
       (effects (font (size 1.27 1.27)) (justify right) hide)
     )
@@
     )
   )
-  (global_label "I2C_SCL" (shape input) (at 154.94 71.12 0) (fields_autoplaced)
-    (effects (font (size 1.27 1.27)) (justify left))
-    (property "Intersheetrefs" "${INTERSHEET_REFS}" (at 165.4053 71.12 0)
+  (global_label "I2C1_SCL" (shape input) (at 154.94 71.12 0) (fields_autoplaced)
+    (effects (font (size 1.27 1.27)) (justify left))
+    (property "Intersheetrefs" "${INTERSHEET_REFS}" (at 166.6148 71.12 0)
       (effects (font (size 1.27 1.27)) (justify left) hide)
     )
@@
     )
   )
+  (global_label "BAT_MS" (shape input) (at 121.92 88.9 180) (fields_autoplaced)
+    (effects (font (size 1.27 1.27)) (justify right))
+    (property "Intersheetrefs" "${INTERSHEET_REFS}" (at 112.0595 88.9 0)
+      (effects (font (size 1.27 1.27)) (justify right) hide)
+    )
+  )
+  (global_label "I2C2_SCL" (shape input) (at 121.92 104.14 180) (fields_autoplaced)
+    (effects (font (size 1.27 1.27)) (justify right))
+    (property "Intersheetrefs" "${INTERSHEET_REFS}" (at 110.2452 104.14 0)
+      (effects (font (size 1.27 1.27)) (justify right) hide)
+    )
+  )
   (global_label "SD_CMD" (shape input) (at 121.92 60.96 180) (fields_autoplaced)
     (effects (font (size 1.27 1.27)) (justify right))
@@
     )
   )
-  (global_label "I2C_SDA" (shape input) (at 154.94 68.58 0) (fields_autoplaced)
-    (effects (font (size 1.27 1.27)) (justify left))
-    (property "Intersheetrefs" "${INTERSHEET_REFS}" (at 165.4658 68.58 0)
-      (effects (font (size 1.27 1.27)) (justify left) hide)
-    )
-  )
-  (global_label "CS_GYRO" (shape input) (at 121.92 111.76 180) (fields_autoplaced)
-    (effects (font (size 1.27 1.27)) (justify right))
-    (property "Intersheetrefs" "${INTERSHEET_REFS}" (at 110.608 111.76 0)
-      (effects (font (size 1.27 1.27)) (justify right) hide)
+  (global_label "I2C2_SDA" (shape input) (at 121.92 106.68 180) (fields_autoplaced)
+    (effects (font (size 1.27 1.27)) (justify right))
+    (property "Intersheetrefs" "${INTERSHEET_REFS}" (at 110.1847 106.68 0)
+      (effects (font (size 1.27 1.27)) (justify right) hide)
+    )
+  )
+  (global_label "I2C1_SDA" (shape input) (at 154.94 68.58 0) (fields_autoplaced)
+    (effects (font (size 1.27 1.27)) (justify left))
+    (property "Intersheetrefs" "${INTERSHEET_REFS}" (at 166.6753 68.58 0)
+      (effects (font (size 1.27 1.27)) (justify left) hide)
     )
   )
@@
     )
   )
-  (global_label "SPI_CLK" (shape input) (at 121.92 106.68 180) (fields_autoplaced)
-    (effects (font (size 1.27 1.27)) (justify right))
-    (property "Intersheetrefs" "${INTERSHEET_REFS}" (at 111.3942 106.68 0)
-      (effects (font (size 1.27 1.27)) (justify right) hide)
-    )
-  )
   (global_label "SD_CD" (shape input) (at 121.92 78.74 180) (fields_autoplaced)
     (effects (font (size 1.27 1.27)) (justify right))
@@
     )
   )
-  (global_label "SPI_MOSI" (shape input) (at 121.92 101.6 180) (fields_autoplaced)
-    (effects (font (size 1.27 1.27)) (justify right))
-    (property "Intersheetrefs" "${INTERSHEET_REFS}" (at 110.3661 101.6 0)
-      (effects (font (size 1.27 1.27)) (justify right) hide)
-    )
-  )
   (global_label "I2S_LRCLK" (shape input) (at 121.92 99.06 180) (fields_autoplaced)
     (effects (font (size 1.27 1.27)) (justify right))
@@
     )
   )
-  (global_label "SPI_MISO" (shape input) (at 121.92 104.14 180) (fields_autoplaced)
-    (effects (font (size 1.27 1.27)) (justify right))
-    (property "Intersheetrefs" "${INTERSHEET_REFS}" (at 110.3661 104.14 0)
-      (effects (font (size 1.27 1.27)) (justify right) hide)
-    )
-  )
   (global_label "LCD_BUSY" (shape input) (at 154.94 58.42 0) (fields_autoplaced)
     (effects (font (size 1.27 1.27)) (justify left))
@@
     )
   )
-  (global_label "CS_ACCEL" (shape input) (at 121.92 109.22 180) (fields_autoplaced)
-    (effects (font (size 1.27 1.27)) (justify right))
-    (property "Intersheetrefs" "${INTERSHEET_REFS}" (at 109.7614 109.22 0)
-      (effects (font (size 1.27 1.27)) (justify right) hide)
-    )
-  )
   (global_label "SD_DAT0" (shape input) (at 121.92 63.5 180) (fields_autoplaced)
     (effects (font (size 1.27 1.27)) (justify right))
@@
     )
   )
-  (global_label "CS_PrSen" (shape input) (at 121.92 88.9 180) (fields_autoplaced)
-    (effects (font (size 1.27 1.27)) (justify right))
-    (property "Intersheetrefs" "${INTERSHEET_REFS}" (at 110.0638 88.9 0)
+  (global_label "BAT_ADC" (shape input) (at 121.92 86.36 180) (fields_autoplaced)
+    (effects (font (size 1.27 1.27)) (justify right))
+    (property "Intersheetrefs" "${INTERSHEET_REFS}" (at 111.0918 86.36 0)
       (effects (font (size 1.27 1.27)) (justify right) hide)
     )
@@
       )
     )
+  )
+  (sheet (at 204.47 110.49) (size 20.32 12.7) (fields_autoplaced)
+    (stroke (width 0.1524) (type solid))
+    (fill (color 0 0 0 0.0000))
+    (property "Sheetname" "Sensors" (at 204.47 109.7784 0)
+      (effects (font (size 1.27 1.27)) (justify left bottom))
+    )
+    (property "Sheetfile" "Sesnors.kicad_sch" (at 204.47 123.7746 0)
+      (effects (font (size 1.27 1.27)) (justify left top))
+    )
+    (instances
+      (project "VariometerV2.2.1"
+        (path "/9d9a2a31-8397-4ba2-ad51-8bee2c0fd904" (page "5"))
+      )
+    )
+  )
+  (sheet (at 204.47 90.17) (size 20.32 12.7) (fields_autoplaced)
+    (stroke (width 0.1524) (type solid))
+    (fill (color 0 0 0 0.0000))
+    (property "Sheetname" "Screen" (at 204.47 89.4584 0)
+      (effects (font (size 1.27 1.27)) (justify left bottom))
+    )
+    (property "Sheetfile" "Screen.kicad_sch" (at 204.47 103.4546 0)
+      (effects (font (size 1.27 1.27)) (justify left top))
+    )
+    (instances
+      (project "VariometerV2.2.1"
+        (path "/9d9a2a31-8397-4ba2-ad51-8bee2c0fd904" (page "4"))
+      )
+    )

Commit message: Working on PCB
Parts:
- added H1, H2, H3, H4: MountingHole_Pad, MountingHole:MountingHole_2.2mm_M2_DIN965_Pad, symbol Mechanical:MountingHole_Pad
- added R37 (x2), R38 (x2): 10k, Resistor_SMD:R_0402_1005Metric, symbol Device:R_Small
- added TP3: TP_SDA2, TestPoint:TestPoint_Pad_D1.5mm, symbol Connector:TestPoint
- added TP3: TP_SDA1, TestPoint:TestPoint_Pad_D1.5mm, symbol Connector:TestPoint
- added TP4: TP_SCL2, TestPoint:TestPoint_Pad_D1.5mm, symbol Connector:TestPoint
- added TP4: TP_SCL1, TestPoint:TestPoint_Pad_D1.5mm, symbol Connector:TestPoint
- C1: footprint Capacitor_SMD:C_0603_1608Metric -> MainLibrary:TFP09212B
Connections:
- net GND: now also H1.1, H2.1, H3.1, H4.1
- net I2C1_SCL: now also R38.2, TP4.1
- net I2C1_SDA: now also R37.2, TP3.1
- net I2C2_SCL: now also R38.2, TP4.1
- net I2C2_SDA: now also R37.2, TP3.1
- net AUDIO_EN: now reaches IC1.24 (IO47)
- new net +3.1V_SW: R37.1, R37.1, R38.1, R38.1
Other:
- sheet Sensors renamed Devices
- note added: "I2C1 PULL-UPS"
- note added: "I2C2 PULL-UPS"
- moved on the sheet: C4, C5, SW1, SW2

Commit message: Update Schematics
Parts:
- C1: footprint MainLibrary:TFP09212B -> Capacitor_SMD:C_0603_1608Metric
- C4: footprint Capacitor_SMD:C_0603_1608Metric -> Capacitor_SMD:C_0402_1005Metric
- IC1: footprint SamacSys_Parts:ESP32S3WROOM1 -> MainLibrary:ESP32S3WROOM1
- R1, R37, R38: footprint Resistor_SMD:R_0402_1005Metric -> (none)
- SW1, SW2: footprint Button_Switch_THT:SW_PUSH_6mm -> (none)
- TP3, TP4: footprint TestPoint:TestPoint_Pad_D1.5mm -> (none)
Connections:
- net AUDIO_EN is gone; now on net I2C2_SCL: IC1.24 (IO47)
- net I2C2_SCL: no longer IC1.22 (IO14)
- net I2C2_SDA: now also IC1.25 (IO48); no longer IC1.23 (IO21)
- net PrSen_INT: now also IC1.23 (IO21); no longer IC1.21 (IO13)
- net CHARG_INT: now reaches IC1.36 (RXD0)
- new net USB_CC1: IC1.21 (IO13)
- new net USB_CC2: IC1.22 (IO14)
Other:
- note added: "CC-Voltage: 0V-0.2V: No Connection 0.2v-0.66V: Standard USB Current 0.66V-1.23V: 1.5A 1.23V+: 3A"
- moved on the sheet: C2, R1

Commit message: Working on PCB
Parts:
- R1: footprint (none) -> Resistor_SMD:R_0402_1005Metric
- R37, R38: footprint (none) -> Resistor_SMD:R_0603_1608Metric
- SW1, SW2: footprint (none) -> Button_Switch_THT:SW_PUSH_6mm
- TP3, TP4: footprint (none) -> TestPoint:TestPoint_Pad_D1.5mm
Changed lines of the file:
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@@
       (effects (font (size 1.27 1.27)) (justify left))
     )
-    (property "Footprint" "" (at 66.04 167.64 0)
+    (property "Footprint" "TestPoint:TestPoint_Pad_D1.5mm" (at 66.04 167.64 0)
       (effects (font (size 1.27 1.27)) hide)
     )
@@
       (effects (font (size 1.27 1.27)) (justify left))
     )
-    (property "Footprint" "" (at 160.02 142.24 0)
+    (property "Footprint" "Button_Switch_THT:SW_PUSH_6mm" (at 160.02 142.24 0)
       (effects (font (size 1.27 1.27)) hide)
     )
@@
       (effects (font (size 1.27 1.27)) (justify left))
     )
-    (property "Footprint" "" (at 35.56 163.83 0)
+    (property "Footprint" "TestPoint:TestPoint_Pad_D1.5mm" (at 35.56 163.83 0)
       (effects (font (size 1.27 1.27)) hide)
     )
@@
       (effects (font (size 1.27 1.27)) (justify left))
     )
-    (property "Footprint" "" (at 43.18 161.29 0)
+    (property "Footprint" "Resistor_SMD:R_0603_1608Metric" (at 43.18 161.29 0)
       (effects (font (size 1.27 1.27)) hide)
     )
@@
       (effects (font (size 1.27 1.27)) (justify left))
     )
-    (property "Footprint" "" (at 50.8 161.29 0)
+    (property "Footprint" "Resistor_SMD:R_0603_1608Metric" (at 50.8 161.29 0)
       (effects (font (size 1.27 1.27)) hide)
     )
@@
       (effects (font (size 1.27 1.27)) (justify left))
     )
-    (property "Footprint" "" (at 119.38 143.51 0)
+    (property "Footprint" "Button_Switch_THT:SW_PUSH_6mm" (at 119.38 143.51 0)
       (effects (font (size 1.27 1.27)) hide)
     )
@@
       (effects (font (size 1.27 1.27)) (justify left))
     )
-    (property "Footprint" "" (at 66.04 120.65 0)
+    (property "Footprint" "TestPoint:TestPoint_Pad_D1.5mm" (at 66.04 120.65 0)
       (effects (font (size 1.27 1.27)) hide)
     )
@@
       (effects (font (size 1.27 1.27)) (justify left))
     )
-    (property "Footprint" "" (at 43.18 114.3 0)
+    (property "Footprint" "Resistor_SMD:R_0603_1608Metric" (at 43.18 114.3 0)
       (effects (font (size 1.27 1.27)) hide)
     )
@@
       (effects (font (size 1.27 1.27)) (justify left))
     )
-    (property "Footprint" "" (at 35.56 116.84 0)
+    (property "Footprint" "TestPoint:TestPoint_Pad_D1.5mm" (at 35.56 116.84 0)
       (effects (font (size 1.27 1.27)) hide)
     )
@@
       (effects (font (size 1.27 1.27)) (justify left))
     )
-    (property "Footprint" "" (at 80.01 74.93 0)
+    (property "Footprint" "Resistor_SMD:R_0402_1005Metric" (at 80.01 74.93 0)
       (effects (font (size 1.27 1.27)) hide)
     )
@@
       (effects (font (size 1.27 1.27)) (justify left))
     )
-    (property "Footprint" "" (at 50.8 114.3 0)
-      (effects (font (size 1.27 1.27)) hide)
-    )
+    (property "Footprint" "Resistor_SMD:R_0603_1608Metric" (at 50.8 114.3 0)
+      (effects (font (size 1.27 1.27)) hide)
+    )

Commit message: PCB
Parts:
- C1: JLCPCB Part # C59461 -> (none); LCSC Part (none) -> C59461
- C2: JLCPCB Part # C52923 -> (none); LCSC Part (none) -> C52923; LCSC Part # C2345 -> (none)
- C3, C5: JLCPCB Part # C307331 -> (none); LCSC Part (none) -> C307331
- C4: JLCPCB Part # C14663 -> (none); LCSC Part (none) -> C307331
- IC1: JLCPCB Part # C2913198 -> (none); LCSC Part (none) -> C2913198
- R1: JLCPCB Part # C25744 -> (none); LCSC Part (none) -> C25744
- R37, R38: JLCPCB Part # C25744 -> (none); LCSC Part (none) -> C25804
Changed lines of the file:
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@@
+      (effects (font (size 1.27 1.27)) hide)
+    )
+    (property "LCSC Part" "" (at 60.96 167.64 0)
       (effects (font (size 1.27 1.27)) hide)
     )
@@
     )
     (property "Datasheet" "" (at 160.02 142.24 0)
+      (effects (font (size 1.27 1.27)) hide)
+    )
+    (property "LCSC Part" "" (at 154.94 142.24 0)
       (effects (font (size 1.27 1.27)) hide)
     )
@@
       (effects (font (size 1.27 1.27)) hide)
     )
+    (property "LCSC Part" "" (at 30.48 163.83 0)
+      (effects (font (size 1.27 1.27)) hide)
+    )
     (pin "1")
     (instances
@@
       (effects (font (size 1.27 1.27)) hide)
     )
-    (property "JLCPCB Part #" "C25744" (at 43.18 161.29 0)
+    (property "LCSC Part" "C25804" (at 43.18 161.29 0)
       (effects (font (size 1.27 1.27)) hide)
     )
@@
       (effects (font (size 1.27 1.27)) hide)
     )
-    (property "JLCPCB Part #" "C25744" (at 50.8 161.29 0)
+    (property "LCSC Part" "C25804" (at 50.8 161.29 0)
       (effects (font (size 1.27 1.27)) hide)
     )
@@
       (effects (font (size 1.27 1.27)) (justify left) hide)
     )
-    (property "JLCPCB Part #" "C2913198" (at 121.92 50.8 0)
+    (property "LCSC Part" "C2913198" (at 121.92 50.8 0)
       (effects (font (size 1.27 1.27)) hide)
     )
@@
       (effects (font (size 1.27 1.27)) hide)
     )
+    (property "LCSC Part" "" (at 114.3 143.51 0)
+      (effects (font (size 1.27 1.27)) hide)
+    )
     (pin "1")
     (pin "2")
@@
     )
     (property "Datasheet" "~" (at 33.02 41.91 0)
+      (effects (font (size 1.27 1.27)) hide)
+    )
+    (property "LCSC Part" "" (at 33.02 41.91 0)
       (effects (font (size 1.27 1.27)) hide)
     )
@@
       (effects (font (size 1.27 1.27)) hide)
     )
+    (property "LCSC Part" "" (at 60.96 120.65 0)
+      (effects (font (size 1.27 1.27)) hide)
+    )
     (pin "1")
     (instances
@@
     )
     (property "Datasheet" "~" (at 33.02 46.99 0)
+      (effects (font (size 1.27 1.27)) hide)
+    )
+    (property "LCSC Part" "" (at 33.02 46.99 0)
       (effects (font (size 1.27 1.27)) hide)
     )
@@
       (effects (font (size 1.27 1.27)) hide)
     )
-    (property "JLCPCB Part #" "C25744" (at 43.18 114.3 0)
+    (property "LCSC Part" "C25804" (at 43.18 114.3 0)
       (effects (font (size 1.27 1.27)) hide)
     )
@@
       (effects (font (size 1.27 1.27)) hide)
     )
-    (property "JLCPCB Part #" "C14663" (at 107.95 143.51 0)
+    (property "LCSC Part" "C307331" (at 107.95 143.51 0)
       (effects (font (size 1.27 1.27)) hide)
     )
@@
       (effects (font (size 1.27 1.27)) hide)
     )
+    (property "LCSC Part" "" (at 30.48 116.84 0)
+      (effects (font (size 1.27 1.27)) hide)
+    )
     (pin "1")
     (instances
@@
       (effects (font (size 1.27 1.27)) hide)
     )
-    (property "JLCPCB Part #" "C25744" (at 80.01 74.93 0)
+    (property "LCSC Part" "C25744" (at 80.01 74.93 0)
       (effects (font (size 1.27 1.27)) hide)
     )
@@
       (effects (font (size 1.27 1.27)) hide)
     )
+    (property "LCSC Part" "" (at 33.02 36.83 0)
+      (effects (font (size 1.27 1.27)) hide)
+    )
     (pin "1")
     (instances
@@
       (effects (font (size 1.27 1.27)) hide)
     )
-    (property "JLCPCB Part #" "C307331" (at 99.06 48.26 0)
+    (property "LCSC Part" "C307331" (at 99.06 48.26 0)
       (effects (font (size 1.27 1.27)) hide)
     )
@@
       (effects (font (size 1.27 1.27)) hide)
     )
-    (property "JLCPCB Part #" "C52923" (at 80.01 82.55 0)
-      (effects (font (size 1.27 1.27)) hide)
-    )
-    (property "LCSC Part #" "C2345" (at 80.01 82.55 0)
+    (property "LCSC Part" "C52923" (at 80.01 82.55 0)
       (effects (font (size 1.27 1.27)) hide)
     )
@@
       (effects (font (size 1.27 1.27)) hide)
     )
-    (property "JLCPCB Part #" "C25744" (at 50.8 114.3 0)
+    (property "LCSC Part" "C25804" (at 50.8 114.3 0)
       (effects (font (size 1.27 1.27)) hide)
     )
@@
       (effects (font (size 1.27 1.27)) hide)
     )
-    (property "JLCPCB Part #" "C59461" (at 88.9 48.26 0)
+    (property "LCSC Part" "C59461" (at 88.9 48.26 0)
       (effects (font (size 1.27 1.27)) hide)
     )
@@
       (effects (font (size 1.27 1.27)) hide)
     )
-    (property "JLCPCB Part #" "C307331" (at 148.59 142.24 0)
+    (property "LCSC Part" "C307331" (at 148.59 142.24 0)
       (effects (font (size 1.27 1.27)) hide)
     )
@@
       (effects (font (size 1.27 1.27)) hide)
     )
+    (property "LCSC Part" "" (at 33.02 52.07 0)
+      (effects (font (size 1.27 1.27)) hide)
+    )
