File: Hardware/Version 2.1/VariometerV2.2.1/VariometerV2.2.1.kicad_sch (KiCad schematic)
At the start: 21 parts, among them IC1 ESP32-S3-WROOM, SW1 Switch_SW_Push, SW2 Switch_SW_Push

Commit message: Start on pcb
Connections:
- net POWS_EN renamed POSW_EN
Changed lines of the file:
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@@
     )
   )
-  (global_label "POWS_EN" (shape input) (at 154.94 73.66 0) (fields_autoplaced)
+  (global_label "POSW_EN" (shape input) (at 154.94 73.66 0) (fields_autoplaced)
     (effects (font (size 1.27 1.27)) (justify left))
     (property "Intersheetrefs" "${INTERSHEET_REFS}" (at 166.5543 73.66 0)

Commit message: PCb Layout done
Parts:
- removed SW1, SW2: Switch_SW_Push, Button_Switch_THT:SW_PUSH_6mm, symbol VariometerV2-rescue:Switch_SW_Push-VariometerV2-cache
- added J6, J9: SW, MainLibrary:PTS636SM25FSMTRLFS, symbol Main_LibraryVario:PTS636_SM25F_SMTR_LFS
Connections:
- net EN: now also J6.1 (COM)
- net GND: now also J6.2 (NO), J9.2 (NO)
- net IO0: now also J9.1 (COM)
Changed lines of the file:
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@@
     (stroke (width 0) (type default))
   )
-  (wire (pts (xy 148.59 147.32) (xy 154.94 147.32))
+  (wire (pts (xy 148.59 147.32) (xy 156.21 147.32))
     (stroke (width 0) (type default))
   )
@@
     (stroke (width 0) (type default))
   )
-  (wire (pts (xy 114.3 138.43) (xy 107.95 138.43))
+  (wire (pts (xy 107.95 138.43) (xy 115.57 138.43))
     (stroke (width 0) (type default))
   )
@@
     (stroke (width 0) (type default))
   )
+  (wire (pts (xy 156.21 137.16) (xy 156.21 140.97))
+    (stroke (width 0) (type default))
+  )
   (wire (pts (xy 27.94 41.91) (xy 27.94 36.83))
     (stroke (width 0) (type default))
@@
     (stroke (width 0) (type default))
   )
+  (wire (pts (xy 115.57 148.59) (xy 115.57 144.78))
+    (stroke (width 0) (type default))
+  )
   (wire (pts (xy 148.59 137.16) (xy 148.59 139.7))
     (stroke (width 0) (type default))
@@
     (stroke (width 0) (type default))
   )
+  (wire (pts (xy 156.21 147.32) (xy 156.21 143.51))
+    (stroke (width 0) (type default))
+  )
   (wire (pts (xy 43.18 165.1) (xy 43.18 163.83))
     (stroke (width 0) (type default))
@@
     (stroke (width 0) (type default))
   )
-  (wire (pts (xy 154.94 137.16) (xy 148.59 137.16))
+  (wire (pts (xy 148.59 137.16) (xy 156.21 137.16))
     (stroke (width 0) (type default))
   )
@@
     (stroke (width 0) (type default))
   )
-  (wire (pts (xy 107.95 148.59) (xy 114.3 148.59))
+  (wire (pts (xy 107.95 148.59) (xy 115.57 148.59))
+    (stroke (width 0) (type default))
+  )
+  (wire (pts (xy 115.57 138.43) (xy 115.57 142.24))
     (stroke (width 0) (type default))
   )
@@
     )
   )
-  (symbol (lib_id "VariometerV2-rescue:Switch_SW_Push-VariometerV2-cache") (at 154.94 142.24 270) (unit 1)
-    (in_bom yes) (on_board yes) (dnp no)
-    (property "Reference" "SW2" (at 158.6992 141.0716 90)
-      (effects (font (size 1.27 1.27)) (justify left))
-    )
-    (property "Value" "Switch_SW_Push" (at 158.6992 143.383 90)
-      (effects (font (size 1.27 1.27)) (justify left))
-    )
-    (property "Footprint" "Button_Switch_THT:SW_PUSH_6mm" (at 160.02 142.24 0)
-      (effects (font (size 1.27 1.27)) hide)
-    )
-    (property "Datasheet" "" (at 160.02 142.24 0)
-      (effects (font (size 1.27 1.27)) hide)
-    )
-    (property "LCSC Part" "" (at 154.94 142.24 0)
-      (effects (font (size 1.27 1.27)) hide)
-    )
-    (pin "1")
-    (pin "2")
-    (instances
-      (project "VariometerV2.2.1"
-        (path "/9d9a2a31-8397-4ba2-ad51-8bee2c0fd904"
-          (reference "SW2") (unit 1)
-        )
-      )
-      (project "VariometerV2.2"
-        (path "/e63e39d7-6ac0-4ffd-8aa3-1841a4541b55"
-          (reference "SW2") (unit 1)
-        )
-      )
-    )
-  )
   (symbol (lib_id "VariometerV2:+3.1V_UNSW") (at 80.01 71.12 0) (unit 1)
     (in_bom yes) (on_board yes) (dnp no) (fields_autoplaced)
@@
         (path "/e63e39d7-6ac0-4ffd-8aa3-1841a4541b55"
           (reference "TP14") (unit 1)
+        )
+      )
+    )
+  )
+  (symbol (lib_id "Main_LibraryVario:PTS636_SM25F_SMTR_LFS") (at 115.57 142.24 0) (unit 1)
+    (in_bom yes) (on_board yes) (dnp no)
+    (property "Reference" "J6" (at 134.62 142.24 0)
+      (effects (font (size 1.27 1.27)) (justify left))
+    )
+    (property "Value" "SW" (at 134.62 144.78 0)
+      (effects (font (size 1.27 1.27)) (justify left))
+    )
+    (property "Footprint" "MainLibrary:PTS636SM25FSMTRLFS" (at 115.57 142.24 0)
+      (effects (font (size 1.27 1.27)) (justify bottom) hide)
+    )
+    (property "Datasheet" "" (at 115.57 142.24 0)
+      (effects (font (size 1.27 1.27)) hide)
+    )
+    (property "Manufacturer_Name" "C & K COMPONENTS" (at 115.57 142.24 0)
+      (effects (font (size 1.27 1.27)) (justify bottom) hide)
+    )
+    (property "Mouser_Price-Stock" "https://www.mouser.co.uk/ProductDetail/CK/PTS636-SM25F-SMTR-LFS?qs=vLWxofP3U2wcBTQSwfMFOw%3D%3D" (at 115.57 142.24 0)
+      (effects (font (size 1.27 1.27)) (justify bottom) hide)
+    )
+    (property "Description" "Tactile Switches Tact 50mA 12VDC, 6.0x3.5, 2.5mm H, 180gf, F leads, No ground pin, White Actuator" (at 115.57 142.24 0)
+      (effects (font (size 1.27 1.27)) (justify bottom) hide)
+    )
+    (property "Mouser_Part_Number" "611-PTS636SM25FSMTRL" (at 115.57 142.24 0)
+      (effects (font (size 1.27 1.27)) (justify bottom) hide)
+    )
+    (property "Height" "2.7mm" (at 115.57 142.24 0)
+      (effects (font (size 1.27 1.27)) (justify bottom) hide)
+    )
+    (property "Arrow_Price-Stock" "https://www.arrow.com/en/products/pts636-sm25f-smtr-lfs/ck" (at 115.57 142.24 0)
+      (effects (font (size 1.27 1.27)) (justify bottom) hide)
+    )
+    (property "Arrow_Part_Number" "PTS636 SM25F SMTR LFS" (at 115.57 142.24 0)
+      (effects (font (size 1.27 1.27)) (justify bottom) hide)
+    )
+    (property "Manufacturer_Part_Number" "PTS636 SM25F SMTR LFS" (at 115.57 142.24 0)
+      (effects (font (size 1.27 1.27)) (justify bottom) hide)
+    )
+    (pin "1")
+    (pin "2")
+    (instances
+      (project "VariometerV2.2.1"
+        (path "/9d9a2a31-8397-4ba2-ad51-8bee2c0fd904"
+          (reference "J6") (unit 1)
         )
       )
@@
     )
   )
-  (symbol (lib_id "VariometerV2-rescue:Switch_SW_Push-VariometerV2-cache") (at 114.3 143.51 270) (unit 1)
-    (in_bom yes) (on_board yes) (dnp no)
-    (property "Reference" "SW1" (at 118.0592 142.3416 90)
-      (effects (font (size 1.27 1.27)) (justify left))
-    )
-    (property "Value" "Switch_SW_Push" (at 118.0592 144.653 90)
-      (effects (font (size 1.27 1.27)) (justify left))
-    )
-    (property "Footprint" "Button_Switch_THT:SW_PUSH_6mm" (at 119.38 143.51 0)
-      (effects (font (size 1.27 1.27)) hide)
-    )
-    (property "Datasheet" "" (at 119.38 143.51 0)
-      (effects (font (size 1.27 1.27)) hide)
-    )
-    (property "LCSC Part" "" (at 114.3 143.51 0)
-      (effects (font (size 1.27 1.27)) hide)
-    )
-    (pin "1")
-    (pin "2")
-    (instances
-      (project "VariometerV2.2.1"
-        (path "/9d9a2a31-8397-4ba2-ad51-8bee2c0fd904"
-          (reference "SW1") (unit 1)
-        )
-      )
-      (project "VariometerV2.2"
-        (path "/e63e39d7-6ac0-4ffd-8aa3-1841a4541b55"
-          (reference "SW1") (unit 1)
-        )
-      )
-    )
-  )
   (symbol (lib_id "Mechanical:MountingHole_Pad") (at 33.02 41.91 270) (unit 1)
     (in_bom yes) (on_board yes) (dnp no)
@@
         )
       )
+    )
+  )
+  (symbol (lib_id "Main_LibraryVario:PTS636_SM25F_SMTR_LFS") (at 156.21 140.97 0) (unit 1)
+    (in_bom yes) (on_board yes) (dnp no)
+    (property "Reference" "J9" (at 175.26 140.97 0)
+      (effects (font (size 1.27 1.27)) (justify left))
+    )
+    (property "Value" "SW" (at 175.26 143.51 0)
+      (effects (font (size 1.27 1.27)) (justify left))
+    )
+    (property "Footprint" "MainLibrary:PTS636SM25FSMTRLFS" (at 156.21 140.97 0)
+      (effects (font (size 1.27 1.27)) (justify bottom) hide)
+    )
+    (property "Datasheet" "" (at 156.21 140.97 0)
+      (effects (font (size 1.27 1.27)) hide)
+    )
+    (property "Manufacturer_Name" "C & K COMPONENTS" (at 156.21 140.97 0)
+      (effects (font (size 1.27 1.27)) (justify bottom) hide)
+    )
+    (property "Mouser_Price-Stock" "https://www.mouser.co.uk/ProductDetail/CK/PTS636-SM25F-SMTR-LFS?qs=vLWxofP3U2wcBTQSwfMFOw%3D%3D" (at 156.21 140.97 0)
+      (effects (font (size 1.27 1.27)) (justify bottom) hide)
+    )
+    (property "Description" "Tactile Switches Tact 50mA 12VDC, 6.0x3.5, 2.5mm H, 180gf, F leads, No ground pin, White Actuator" (at 156.21 140.97 0)
+      (effects (font (size 1.27 1.27)) (justify bottom) hide)
+    )
+    (property "Mouser_Part_Number" "611-PTS636SM25FSMTRL" (at 156.21 140.97 0)
+      (effects (font (size 1.27 1.27)) (justify bottom) hide)
+    )
+    (property "Height" "2.7mm" (at 156.21 140.97 0)
+      (effects (font (size 1.27 1.27)) (justify bottom) hide)
+    )
+    (property "Arrow_Price-Stock" "https://www.arrow.com/en/products/pts636-sm25f-smtr-lfs/ck" (at 156.21 140.97 0)
+      (effects (font (size 1.27 1.27)) (justify bottom) hide)
+    )
+    (property "Arrow_Part_Number" "PTS636 SM25F SMTR LFS" (at 156.21 140.97 0)
+      (effects (font (size 1.27 1.27)) (justify bottom) hide)
+    )
+    (property "Manufacturer_Part_Number" "PTS636 SM25F SMTR LFS" (at 156.21 140.97 0)
+      (effects (font (size 1.27 1.27)) (justify bottom) hide)
+    )
+    (pin "1")
+    (pin "2")
+    (instances
+      (project "VariometerV2.2.1"
+        (path "/9d9a2a31-8397-4ba2-ad51-8bee2c0fd904"
+          (reference "J9") (unit 1)
+        )
+      )

Commit message: Finish PCB
Parts:
- H1, H2, H3, H4, J6, J9, TP3, TP4: LCSC Part (none) -> 0
Changed lines of the file:
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@@
       (effects (font (size 1.27 1.27)) hide)
     )
-    (property "LCSC Part" "" (at 60.96 167.64 0)
+    (property "LCSC Part" "0" (at 60.96 167.64 0)
       (effects (font (size 1.27 1.27)) hide)
     )
@@
       (effects (font (size 1.27 1.27)) hide)
     )
-    (property "LCSC Part" "" (at 30.48 163.83 0)
+    (property "LCSC Part" "0" (at 30.48 163.83 0)
       (effects (font (size 1.27 1.27)) hide)
     )
@@
     (property "Manufacturer_Part_Number" "PTS636 SM25F SMTR LFS" (at 115.57 142.24 0)
       (effects (font (size 1.27 1.27)) (justify bottom) hide)
+    )
+    (property "LCSC Part" "0" (at 115.57 142.24 0)
+      (effects (font (size 1.27 1.27)) hide)
     )
     (pin "1")
@@
       (effects (font (size 1.27 1.27)) hide)
     )
-    (property "LCSC Part" "" (at 33.02 41.91 0)
+    (property "LCSC Part" "0" (at 33.02 41.91 0)
       (effects (font (size 1.27 1.27)) hide)
     )
@@
       (effects (font (size 1.27 1.27)) hide)
     )
-    (property "LCSC Part" "" (at 60.96 120.65 0)
+    (property "LCSC Part" "0" (at 60.96 120.65 0)
       (effects (font (size 1.27 1.27)) hide)
     )
@@
       (effects (font (size 1.27 1.27)) (justify bottom) hide)
     )
+    (property "LCSC Part" "0" (at 156.21 140.97 0)
+      (effects (font (size 1.27 1.27)) hide)
+    )
     (pin "1")
     (pin "2")
@@
       (effects (font (size 1.27 1.27)) hide)
     )
-    (property "LCSC Part" "" (at 33.02 46.99 0)
+    (property "LCSC Part" "0" (at 33.02 46.99 0)
       (effects (font (size 1.27 1.27)) hide)
     )
@@
       (effects (font (size 1.27 1.27)) hide)
     )
-    (property "LCSC Part" "" (at 30.48 116.84 0)
+    (property "LCSC Part" "0" (at 30.48 116.84 0)
       (effects (font (size 1.27 1.27)) hide)
     )
@@
       (effects (font (size 1.27 1.27)) hide)
     )
-    (property "LCSC Part" "" (at 33.02 36.83 0)
+    (property "LCSC Part" "0" (at 33.02 36.83 0)
       (effects (font (size 1.27 1.27)) hide)
     )
@@
       (effects (font (size 1.27 1.27)) hide)
     )
-    (property "LCSC Part" "" (at 33.02 52.07 0)
-      (effects (font (size 1.27 1.27)) hide)
-    )
+    (property "LCSC Part" "0" (at 33.02 52.07 0)
+      (effects (font (size 1.27 1.27)) hide)
+    )
