File: Hardware/Version 2.1/VariometerV2.2.1/Sesnors.kicad_sch (KiCad schematic)
At the start: 0 parts

Commit message: Working on PCB
Parts:
- added C35, C36, C37, C38, C39, C43: 100nF, Capacitor_SMD:C_0402_1005Metric, symbol Device:C_Small
- added C40: 4.7uF, Capacitor_SMD:C_0603_1608Metric, symbol Device:C_Small
- added C41: 220nF, Capacitor_SMD:C_0402_1005Metric, symbol Device:C_Small
- added C42: 10uF, Capacitor_SMD:C_0603_1608Metric, symbol Device:C_Small
- added JP1: SolderJumper_3_Open, symbol Jumper:SolderJumper_3_Open
- added R36: 100k, Resistor_SMD:R_0402_1005Metric, symbol Device:R_Small
- added TP7: TP_BCLK, TestPoint:TestPoint_Pad_D1.5mm, symbol Connector:TestPoint
- added TP8: TP_LRCLK, TestPoint:TestPoint_Pad_D1.5mm, symbol Connector:TestPoint
- added TP9: TP_DIN, TestPoint:TestPoint_Pad_D1.5mm, symbol Connector:TestPoint
- added U4: DPS310, SamacSys_Parts:DPS310XTSA1, symbol VariometerV2:DPS310
- added U5: BMI088, Hardware:BMI088, symbol VariometerV2-rescue:BMI088-Vario2_Library
- added U6: QMC5883L, SamacSys_Parts:QMC5883L, symbol VariometerV2:QMC5883L
- added U7: MAX98357A, SamacSys_Parts:QFN50P300X300X80-17N, symbol VariometerV2:MAX98357A
Connections:
- new net: C40.1, U6.10 (C1)
- new net: C41.2, U6.12 (SETC)
- new net: C41.1, U6.8 (SETP)
- new net: JP1.2 (C), U7.2 (GAIN)
- new net +3.1V_SW: C35.1, C36.1, C37.1, C38.1, C39.1, JP1.1 (A), U4.6 (VDDIO), U4.8 (VDD), U5.11 (VDDIO), U5.14 (CSB1), U5.3 (VDD), U5.7 (PS), U6.13 (VDDIO), U6.2 (VDD), U6.4 (S1)
- new net AUDIO_EN: U7.4 (SD_MODE)
- new net AUDIO_OUTN: U7.10 (OUTN)
- new net AUDIO_OUTP: U7.9 (OUTP)
- new net GND: C35.2, C36.2, C37.2, C38.2, C39.2, C40.2, C42.2, C43.2, JP1.3 (B), R36.2, U4.1 (GND), U4.7 (GND), U5.10 (SDO2), U5.15 (SDO1), U5.2 (NC), U5.4 (GNDA), U5.6 (GNDIO), U6.11 (GND), U6.9 (GND), U7.11 (GND), U7.15 (GND), U7.17 (EP), U7.3 (GND)
- new net I2C1_SCL: U5.8 (SCK)
- new net I2C1_SDA: U5.9 (SDI)
- new net I2C2_SCL: U4.4 (SCK), U6.1 (SCL)
- new net I2C2_SDA: U4.3 (SDI), U6.16 (SDA)
- new net I2S_BCLK: TP7.1, U7.16 (BCLK)
- new net I2S_DIN: TP9.1, U7.1 (DIN)
- new net I2S_LRCLK: TP8.1, U7.14 (LRCLK)
- new net PrSen_INT: R36.1, U4.5 (SDO)
- new net VCC: C42.1, C43.1, U7.7 (VDD), U7.8 (VDD)
- no-connect marks 0 -> 15
Other:
- note added: "AUDIO DAC UND KLASSE D VERSTÄRKER"
- note added: "GAIN: GND = 12dB NC = 9dB VDD = 6dB"
- note added: "GPS!!"
- note added: "IMU Sensor"
- note added: "MAGNETIC SENSOR"
- note added: "PRESSURE SENSOR"
- note added: "SDMODE: HIGH: LEFT CHANNEL LOW: SHUTDOWN PULL-UP 248k: RIGHT PULL-UP 722.14k: (LEFT/2 + RIGHT/2)"

Commit message: Update Schematics
Parts:
- added R41: 10k B, symbol Device:R_Small
- JP1: footprint (none) -> Jumper:SolderJumper-3_P1.3mm_Open_Pad1.0x1.5mm_NumberLabels
- R36: footprint Resistor_SMD:R_0402_1005Metric -> (none)
- TP7, TP8, TP9: footprint TestPoint:TestPoint_Pad_D1.5mm -> (none)
- U4: footprint SamacSys_Parts:DPS310XTSA1 -> (none)
- U5: footprint Hardware:BMI088 -> (none)
- U6: footprint SamacSys_Parts:QMC5883L -> (none)
- U7: footprint SamacSys_Parts:QFN50P300X300X80-17N -> (none)
Connections:
- net AUDIO_EN is gone; now on net +3.1V_SW: U7.4 (SD_MODE)
- net +3.1V_SW: now also R41.1
- net GND: now also R41.2
- no-connect marks 15 -> 16
Changed lines of the file:
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@@
   (junction (at 38.1 168.91) (diameter 0) (color 0 0 0 0)
+  )
+  (junction (at 31.75 152.4) (diameter 0) (color 0 0 0 0)
   )
   (junction (at 134.62 33.02) (diameter 0) (color 0 0 0 0)
@@
   (no_connect (at 78.74 58.42))
   (no_connect (at 129.54 57.15))
+  (no_connect (at 78.74 46.99))
   (no_connect (at 90.17 170.18))
   (no_connect (at 90.17 165.1))
@@
     (stroke (width 0) (type default))
   )
+  (wire (pts (xy 31.75 160.02) (xy 31.75 162.56))
+    (stroke (width 0) (type default))
+  )
   (wire (pts (xy 242.57 44.45) (xy 256.54 44.45))
     (stroke (width 0) (type default))
   )
+  (wire (pts (xy 31.75 143.51) (xy 31.75 152.4))
+    (stroke (width 0) (type default))
+  )
   (wire (pts (xy 55.88 34.29) (xy 55.88 35.56))
     (stroke (width 0) (type default))
@@
     (stroke (width 0) (type default))
   )
-  (wire (pts (xy 53.34 152.4) (xy 68.58 152.4))
+  (wire (pts (xy 31.75 152.4) (xy 68.58 152.4))
     (stroke (width 0) (type default))
   )
@@
   )
   (wire (pts (xy 50.8 74.93) (xy 33.02 74.93))
+    (stroke (width 0) (type default))
+  )
+  (wire (pts (xy 31.75 152.4) (xy 31.75 154.94))
     (stroke (width 0) (type default))
   )
@@
   )
   (text "SDMODE:\nHIGH: 			LEFT CHANNEL\nLOW:  			SHUTDOWN\nPULL-UP 248k: 	RIGHT\nPULL-UP 722.14k:  (LEFT/2 + RIGHT/2)"
-    (at 38.1 129.54 0)
+    (at 15.24 130.81 0)
     (effects (font (size 1.27 1.27) italic) (justify left bottom))
   )
@@
     )
   )
-  (global_label "AUDIO_EN" (shape input) (at 53.34 152.4 180) (fields_autoplaced)
-    (effects (font (size 1.27 1.27)) (justify right))
-    (property "Intersheetrefs" "${INTERSHEET_REFS}" (at 41.8555 152.3206 0)
-      (effects (font (size 1.27 1.27)) (justify right) hide)
-    )
-  )
   (global_label "PrSen_INT" (shape input) (at 209.55 40.64 180) (fields_autoplaced)
     (effects (font (size 1.27 1.27)) (justify right))
@@
       (effects (font (size 1.27 1.27)) (justify left))
     )
-    (property "Footprint" "TestPoint:TestPoint_Pad_D1.5mm" (at 71.12 143.51 0)
+    (property "Footprint" "" (at 71.12 143.51 0)
       (effects (font (size 1.27 1.27)) hide)
     )
@@
     )
   )
+  (symbol (lib_id "power:GND") (at 31.75 162.56 0) (unit 1)
+    (in_bom yes) (on_board yes) (dnp no) (fields_autoplaced)
+    (property "Reference" "#PWR093" (at 31.75 168.91 0)
+      (effects (font (size 1.27 1.27)) hide)
+    )
+    (property "Value" "GND" (at 31.75 167.1225 0)
+      (effects (font (size 1.27 1.27)))
+    )
+    (property "Footprint" "" (at 31.75 162.56 0)
+      (effects (font (size 1.27 1.27)) hide)
+    )
+    (property "Datasheet" "" (at 31.75 162.56 0)
+      (effects (font (size 1.27 1.27)) hide)
+    )
+    (pin "1")
+    (instances
+      (project "VariometerV2.2.1"
+        (path "/9d9a2a31-8397-4ba2-ad51-8bee2c0fd904/056f5ab7-9063-4ff0-b10f-d2fc578ffe92"
+          (reference "#PWR093") (unit 1)
+        )
+      )
+      (project "VariometerV2.2"
+        (path "/e63e39d7-6ac0-4ffd-8aa3-1841a4541b55"
+          (reference "#PWR0162") (unit 1)
+        )
+      )
+    )
+  )
   (symbol (lib_id "VariometerV2:+3.1V_SW") (at 125.73 33.02 0) (unit 1)
     (in_bom yes) (on_board yes) (dnp no)
@@
       (effects (font (size 1.27 1.27)))
     )
-    (property "Footprint" "Hardware:BMI088" (at 60.96 52.07 0)
+    (property "Footprint" "" (at 60.96 52.07 0)
       (effects (font (size 1.27 1.27)) hide)
     )
@@
       (effects (font (size 1.27 1.27)) (justify left))
     )
-    (property "Footprint" "TestPoint:TestPoint_Pad_D1.5mm" (at 66.04 143.51 0)
+    (property "Footprint" "" (at 66.04 143.51 0)
       (effects (font (size 1.27 1.27)) hide)
     )
@@
       (effects (font (size 1.27 1.27)) (justify left))
     )
-    (property "Footprint" "SamacSys_Parts:QMC5883L" (at 137.16 49.53 0)
+    (property "Footprint" "" (at 137.16 49.53 0)
       (effects (font (size 1.27 1.27)) hide)
     )
@@
       (effects (font (size 1.27 1.27)))
     )
-    (property "Footprint" "SamacSys_Parts:DPS310XTSA1" (at 231.14 39.37 0)
+    (property "Footprint" "" (at 231.14 39.37 0)
       (effects (font (size 1.27 1.27)) hide)
     )
@@
       (effects (font (size 1.27 1.27)) (justify left))
     )
-    (property "Footprint" "" (at 110.49 158.75 0)
+    (property "Footprint" "Jumper:SolderJumper-3_P1.3mm_Open_Pad1.0x1.5mm_NumberLabels" (at 110.49 158.75 0)
       (effects (font (size 1.27 1.27)) hide)
     )
@@
       (effects (font (size 1.27 1.27)) (justify left))
     )
-    (property "Footprint" "TestPoint:TestPoint_Pad_D1.5mm" (at 62.23 143.51 0)
+    (property "Footprint" "" (at 62.23 143.51 0)
       (effects (font (size 1.27 1.27)) hide)
     )
@@
     )
   )
+  (symbol (lib_id "Device:R_Small") (at 31.75 157.48 0) (unit 1)
+    (in_bom yes) (on_board yes) (dnp no)
+    (property "Reference" "R41" (at 25.4 157.48 0)
+      (effects (font (size 1.27 1.27)) (justify left))
+    )
+    (property "Value" "10k B" (at 24.13 160.02 0)
+      (effects (font (size 1.27 1.27)) (justify left))
+    )
+    (property "Footprint" "" (at 31.75 157.48 0)
+      (effects (font (size 1.27 1.27)) hide)
+    )
+    (property "Datasheet" "~" (at 31.75 157.48 0)
+      (effects (font (size 1.27 1.27)) hide)
+    )
+    (pin "1")
+    (pin "2")
+    (instances
+      (project "VariometerV2.2.1"
+        (path "/9d9a2a31-8397-4ba2-ad51-8bee2c0fd904/056f5ab7-9063-4ff0-b10f-d2fc578ffe92"
+          (reference "R41") (unit 1)
+        )
+      )
+    )
+  )
   (symbol (lib_id "Device:R_Small") (at 214.63 44.45 0) (unit 1)
     (in_bom yes) (on_board yes) (dnp no)
@@
       (effects (font (size 1.27 1.27)) (justify left))
     )
-    (property "Footprint" "Resistor_SMD:R_0402_1005Metric" (at 214.63 44.45 0)
+    (property "Footprint" "" (at 214.63 44.45 0)
       (effects (font (size 1.27 1.27)) hide)
     )
@@
       (effects (font (size 1.27 1.27)))
     )
-    (property "Footprint" "SamacSys_Parts:QFN50P300X300X80-17N" (at 80.01 158.75 0)
+    (property "Footprint" "" (at 80.01 158.75 0)
       (effects (font (size 1.27 1.27)) hide)
     )
@@
         )
       )
+    )
+  )
+  (symbol (lib_id "VariometerV2:+3.1V_SW") (at 31.75 143.51 0) (unit 1)
+    (in_bom yes) (on_board yes) (dnp no)
+    (property "Reference" "#PWR092" (at 31.75 147.32 0)
+      (effects (font (size 1.27 1.27)) hide)
+    )
+    (property "Value" "+3.1V_SW" (at 31.75 139.7 0)
+      (effects (font (size 1.27 1.27)))
+    )
+    (property "Footprint" "" (at 31.75 143.51 0)
+      (effects (font (size 1.27 1.27)) hide)
+    )
+    (property "Datasheet" "" (at 31.75 143.51 0)
+      (effects (font (size 1.27 1.27)) hide)
+    )
+    (pin "1")
+    (instances
+      (project "VariometerV2.2.1"
+        (path "/9d9a2a31-8397-4ba2-ad51-8bee2c0fd904/056f5ab7-9063-4ff0-b10f-d2fc578ffe92"
+          (reference "#PWR092") (unit 1)
+        )
+      )
+      (project "VariometerV2.2"
+        (path "/e63e39d7-6ac0-4ffd-8aa3-1841a4541b55"
+          (reference "#PWR0152") (unit 1)
+        )
+      )

Commit message: Working on PCB
Parts:
- R36: footprint (none) -> Resistor_SMD:R_0603_1608Metric
- R41: footprint (none) -> Resistor_SMD:R_0805_2012Metric
- TP7, TP8, TP9: footprint (none) -> TestPoint:TestPoint_Pad_D1.5mm
- U4: footprint (none) -> MainLibrary:DPS310XTSA1
- U5: footprint (none) -> MainLibrary:BMI088
- U6: footprint (none) -> MainLibrary:QMC5883L
- U7: footprint (none) -> MainLibrary:QFN50P300X300X80-17N
Changed lines of the file:
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@@
       (effects (font (size 1.27 1.27)) (justify left))
     )
-    (property "Footprint" "" (at 71.12 143.51 0)
+    (property "Footprint" "TestPoint:TestPoint_Pad_D1.5mm" (at 71.12 143.51 0)
       (effects (font (size 1.27 1.27)) hide)
     )
@@
       (effects (font (size 1.27 1.27)))
     )
-    (property "Footprint" "" (at 60.96 52.07 0)
+    (property "Footprint" "MainLibrary:BMI088" (at 60.96 52.07 0)
       (effects (font (size 1.27 1.27)) hide)
     )
@@
       (effects (font (size 1.27 1.27)) (justify left))
     )
-    (property "Footprint" "" (at 66.04 143.51 0)
+    (property "Footprint" "TestPoint:TestPoint_Pad_D1.5mm" (at 66.04 143.51 0)
       (effects (font (size 1.27 1.27)) hide)
     )
@@
       (effects (font (size 1.27 1.27)) (justify left))
     )
-    (property "Footprint" "" (at 137.16 49.53 0)
+    (property "Footprint" "MainLibrary:QMC5883L" (at 137.16 49.53 0)
       (effects (font (size 1.27 1.27)) hide)
     )
@@
       (effects (font (size 1.27 1.27)))
     )
-    (property "Footprint" "" (at 231.14 39.37 0)
+    (property "Footprint" "MainLibrary:DPS310XTSA1" (at 231.14 39.37 0)
       (effects (font (size 1.27 1.27)) hide)
     )
@@
       (effects (font (size 1.27 1.27)) (justify left))
     )
-    (property "Footprint" "" (at 62.23 143.51 0)
+    (property "Footprint" "TestPoint:TestPoint_Pad_D1.5mm" (at 62.23 143.51 0)
       (effects (font (size 1.27 1.27)) hide)
     )
@@
       (effects (font (size 1.27 1.27)) (justify left))
     )
-    (property "Footprint" "" (at 31.75 157.48 0)
+    (property "Footprint" "Resistor_SMD:R_0805_2012Metric" (at 31.75 157.48 0)
       (effects (font (size 1.27 1.27)) hide)
     )
@@
       (effects (font (size 1.27 1.27)) (justify left))
     )
-    (property "Footprint" "" (at 214.63 44.45 0)
+    (property "Footprint" "Resistor_SMD:R_0603_1608Metric" (at 214.63 44.45 0)
       (effects (font (size 1.27 1.27)) hide)
     )
@@
       (effects (font (size 1.27 1.27)))
     )
-    (property "Footprint" "" (at 80.01 158.75 0)
-      (effects (font (size 1.27 1.27)) hide)
-    )
+    (property "Footprint" "MainLibrary:QFN50P300X300X80-17N" (at 80.01 158.75 0)
+      (effects (font (size 1.27 1.27)) hide)
+    )

Commit message: PCB
Parts:
- C35, C36, C37, C38, C39, C43: JLCPCB Part # C307331 -> (none); LCSC Part (none) -> C307331
- C40: JLCPCB Part # C19666 -> (none); LCSC Part (none) -> C19666
- C41: JLCPCB Part # C16772 -> (none); LCSC Part (none) -> C16772
- C42: JLCPCB Part # C96446 -> (none); LCSC Part (none) -> C19702
- R36: JLCPCB Part # C25741 -> (none); LCSC Part (none) -> C25803
- R41: LCSC Part (none) -> C17414
- U4: JLCPCB Part # C130156 -> (none); LCSC Part (none) -> C130156
- U5: JLCPCB Part # C194919 -> (none); LCSC Part (none) -> C194919
- U6: JLCPCB Part # C976032 -> (none); LCSC Part (none) -> C976032
- U7: JLCPCB Part # C910544 -> (none); LCSC Part (none) -> C910544
Changed lines of the file:
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@@
+      (effects (font (size 1.27 1.27)) hide)
+    )
+    (property "LCSC Part" "" (at 66.04 143.51 0)
       (effects (font (size 1.27 1.27)) hide)
     )
@@
       (effects (font (size 1.27 1.27)) hide)
     )
-    (property "JLCPCB Part #" "C194919" (at 60.96 52.07 0)
+    (property "LCSC Part" "C194919" (at 60.96 52.07 0)
       (effects (font (size 1.27 1.27)) hide)
     )
@@
       (effects (font (size 1.27 1.27)) hide)
     )
+    (property "LCSC Part" "" (at 60.96 143.51 0)
+      (effects (font (size 1.27 1.27)) hide)
+    )
     (pin "1")
     (instances
@@
       (effects (font (size 1.27 1.27)) hide)
     )
-    (property "JLCPCB Part #" "C976032" (at 137.16 49.53 0)
+    (property "LCSC Part" "C976032" (at 137.16 49.53 0)
       (effects (font (size 1.27 1.27)) hide)
     )
@@
       (effects (font (size 1.27 1.27)) hide)
     )
-    (property "JLCPCB Part #" "C96446" (at 38.1 171.45 0)
+    (property "LCSC Part" "C19702" (at 38.1 171.45 0)
       (effects (font (size 1.27 1.27)) hide)
     )
@@
       (effects (font (size 1.27 1.27)) hide)
     )
-    (property "JLCPCB Part #" "C307331" (at 49.53 171.45 0)
+    (property "LCSC Part" "C307331" (at 49.53 171.45 0)
       (effects (font (size 1.27 1.27)) hide)
     )
@@
       (effects (font (size 1.27 1.27)) hide)
     )
-    (property "JLCPCB Part #" "C307331" (at 256.54 46.99 0)
+    (property "LCSC Part" "C307331" (at 256.54 46.99 0)
       (effects (font (size 1.27 1.27)) hide)
     )
@@
       (effects (font (size 1.27 1.27)) hide)
     )
-    (property "JLCPCB Part #" "C307331" (at 55.88 31.75 0)
+    (property "LCSC Part" "C307331" (at 55.88 31.75 0)
       (effects (font (size 1.27 1.27)) hide)
     )
@@
       (effects (font (size 1.27 1.27)) hide)
     )
-    (property "JLCPCB Part #" "C19666" (at 134.62 76.2 0)
+    (property "LCSC Part" "C19666" (at 134.62 76.2 0)
       (effects (font (size 1.27 1.27)) hide)
     )
@@
       (effects (font (size 1.27 1.27)) hide)
     )
-    (property "JLCPCB Part #" "C130156" (at 231.14 39.37 0)
+    (property "LCSC Part" "C130156" (at 231.14 39.37 0)
       (effects (font (size 1.27 1.27)) hide)
     )
@@
       (effects (font (size 1.27 1.27)) hide)
     )
+    (property "LCSC Part" "" (at 110.49 158.75 0)
+      (effects (font (size 1.27 1.27)) hide)
+    )
     (pin "1")
     (pin "2")
@@
       (effects (font (size 1.27 1.27)) hide)
     )
-    (property "JLCPCB Part #" "C307331" (at 128.27 35.56 0)
+    (property "LCSC Part" "C307331" (at 128.27 35.56 0)
       (effects (font (size 1.27 1.27)) hide)
     )
@@
       (effects (font (size 1.27 1.27)) hide)
     )
+    (property "LCSC Part" "" (at 57.15 143.51 0)
+      (effects (font (size 1.27 1.27)) hide)
+    )
     (pin "1")
     (instances
@@
       (effects (font (size 1.27 1.27)) hide)
     )
-    (property "JLCPCB Part #" "C307331" (at 73.66 31.75 0)
+    (property "LCSC Part" "C307331" (at 73.66 31.75 0)
       (effects (font (size 1.27 1.27)) hide)
     )
@@
       (effects (font (size 1.27 1.27)) hide)
     )
-    (property "JLCPCB Part #" "C16772" (at 153.67 52.07 0)
+    (property "LCSC Part" "C16772" (at 153.67 52.07 0)
       (effects (font (size 1.27 1.27)) hide)
     )
@@
       (effects (font (size 1.27 1.27)) hide)
     )
+    (property "LCSC Part" "C17414" (at 31.75 157.48 0)
+      (effects (font (size 1.27 1.27)) hide)
+    )
     (pin "1")
     (pin "2")
@@
       (effects (font (size 1.27 1.27)) hide)
     )
-    (property "JLCPCB Part #" "C25741" (at 214.63 44.45 0)
+    (property "LCSC Part" "C25803" (at 214.63 44.45 0)
       (effects (font (size 1.27 1.27)) hide)
     )
@@
       (effects (font (size 1.27 1.27)) hide)
     )
-    (property "JLCPCB Part #" "C910544" (at 80.01 158.75 0)
+    (property "LCSC Part" "C910544" (at 80.01 158.75 0)
       (effects (font (size 1.27 1.27)) hide)
     )
@@
       (effects (font (size 1.27 1.27)) hide)
     )
-    (property "JLCPCB Part #" "C307331" (at 250.19 34.29 0)
-      (effects (font (size 1.27 1.27)) hide)
-    )
+    (property "LCSC Part" "C307331" (at 250.19 34.29 0)
+      (effects (font (size 1.27 1.27)) hide)
+    )

Commit message: Start on pcb
Parts:
- added C50, C8: 100nF, Capacitor_SMD:C_0402_1005Metric, symbol Device:C_Small
- added C7: 10uF, Capacitor_SMD:C_0402_1005Metric, symbol Device:C_Small
- added C9: 4.7uF, Capacitor_SMD:C_0402_1005Metric, symbol Device:C_Small
- added D1: BLUE, LED_SMD:LED_0603_1608Metric, symbol Device:LED
- added J1: U.FL-R-SMT(01), SamacSys_Parts:HRS_U.FL-R-SMT(01), symbol Main_Library:U.FL-R-SMT(01)
- added JP3: SJ, Jumper:SolderJumper-2_P1.3mm_Open_Pad1.0x1.5mm, symbol Jumper:SolderJumper_2_Open
- added JP5, JP7: ~, Jumper:SolderJumper-3_P1.3mm_Open_Pad1.0x1.5mm, symbol Jumper:SolderJumper_3_Open
- added L2: 47nH, Inductor_SMD:L_0805_2012Metric, symbol Device:L_Small
- added R10: 10R, Resistor_SMD:R_0603_1608Metric, symbol Device:R_Small
- added R4: 1k, Resistor_SMD:R_0603_1608Metric, symbol Device:R_Small
- added R7: 10k, Inductor_SMD:L_0603_1608Metric, symbol Device:R_Small
- added R8: 10k, Resistor_SMD:R_0603_1608Metric, symbol Device:R_Small
- added U8: L76-L, MainLibrary:XCVR_L76-L, symbol Main_LibraryVario:L76-L
Connections:
- net +3.1V_SW: now also C7.1, C8.1, R7.1, R8.1, U8.8 (VCC)
- net GND: now also C50.2, C7.2, C8.2, C9.2, D1.1 (K), J1.1 (GND), J1.2 (GND), U8.1 (GND), U8.10 (GND), U8.12 (GND)
- net I2C1_SCL: now also U6.1 (SCL)
- net I2C1_SDA: now also U6.16 (SDA)
- net I2C2_SCL: no longer U6.1 (SCL)
- net I2C2_SDA: no longer U6.16 (SDA)
- new net: JP3.2 (B), L2.1
- new net: L2.2, R10.1
- new net: D1.2 (A), R4.2
- new net: J1.3 (SIG), JP3.1 (A), U8.11 (RF_IN)
- new net: U8.15 (NC), U8.7 (NC)
- new net: R4.1, U8.4 (1PPS)
- new net +3.1V_UNSW: C50.1, C9.1, U8.6 (V_BCKP)
- new net GPS_RX: JP7.1 (A), U8.3 (RXD)
- new net GPS_SCL: JP5.3 (B), R8.2, U8.17 (I2C_SCL)
- new net GPS_SDA: JP7.3 (B), R7.2, U8.16 (I2C_SDA)
- new net GPS_TX: JP5.1 (A), U8.2 (TXD)
- new net GPS_VCCREF: R10.2, U8.14 (VCC_RF)
- new net USART2_RX: JP5.2 (C)
- new net USART2_TX: JP7.2 (C)
- no-connect marks 16 -> 20
Other:
- note added: "GPS"
- note removed: "GPS!!"
