File: Hardware/Version 2.1/VariometerV2.2.1/Sesnors.kicad_sch (KiCad schematic)
At the start: 34 parts, among them J1 U.FL-R-SMT(01), U4 DPS310, U5 BMI088, U6 QMC5883L, U7 MAX98357A, U8 L76-L

Commit message: PCb Layout done
Parts:
- removed TP7: TP_BCLK, TestPoint:TestPoint_Pad_D1.5mm, symbol Connector:TestPoint
- removed TP8: TP_LRCLK, TestPoint:TestPoint_Pad_D1.5mm, symbol Connector:TestPoint
- removed TP9: TP_DIN, TestPoint:TestPoint_Pad_D1.5mm, symbol Connector:TestPoint
Changed lines of the file:
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@@
   (junction (at 73.66 29.21) (diameter 0) (color 0 0 0 0)
   )
-  (junction (at 66.04 163.83) (diameter 0) (color 0 0 0 0)
-  )
   (junction (at 264.16 119.38) (diameter 0) (color 0 0 0 0)
   )
@@
   )
   (junction (at 269.24 90.17) (diameter 0) (color 0 0 0 0)
-  )
-  (junction (at 57.15 156.21) (diameter 0) (color 0 0 0 0)
-  )
-  (junction (at 60.96 160.02) (diameter 0) (color 0 0 0 0)
   )
   (junction (at 33.02 62.23) (diameter 0) (color 0 0 0 0)
@@
     (stroke (width 0) (type default))
   )
-  (wire (pts (xy 60.96 160.02) (xy 68.58 160.02))
+  (wire (pts (xy 54.61 160.02) (xy 68.58 160.02))
     (stroke (width 0) (type default))
   )
@@
     (stroke (width 0) (type default))
   )
-  (wire (pts (xy 60.96 143.51) (xy 60.96 160.02))
-    (stroke (width 0) (type default))
-  )
-  (wire (pts (xy 52.07 163.83) (xy 66.04 163.83))
+  (wire (pts (xy 52.07 163.83) (xy 68.58 163.83))
     (stroke (width 0) (type default))
   )
@@
     (stroke (width 0) (type default))
   )
-  (wire (pts (xy 66.04 143.51) (xy 66.04 163.83))
-    (stroke (width 0) (type default))
-  )
   (wire (pts (xy 246.38 33.02) (xy 246.38 31.75))
     (stroke (width 0) (type default))
@@
     (stroke (width 0) (type default))
   )
-  (wire (pts (xy 66.04 163.83) (xy 68.58 163.83))
-    (stroke (width 0) (type default))
-  )
   (wire (pts (xy 228.6 93.98) (xy 228.6 99.06))
     (stroke (width 0) (type default))
@@
     (stroke (width 0) (type default))
   )
-  (wire (pts (xy 53.34 156.21) (xy 57.15 156.21))
-    (stroke (width 0) (type default))
-  )
   (wire (pts (xy 266.7 113.03) (xy 266.7 111.76))
     (stroke (width 0) (type default))
   )
-  (wire (pts (xy 54.61 160.02) (xy 60.96 160.02))
-    (stroke (width 0) (type default))
-  )
   (wire (pts (xy 176.53 147.32) (xy 176.53 148.59))
     (stroke (width 0) (type default))
@@
     (stroke (width 0) (type default))
   )
-  (wire (pts (xy 57.15 143.51) (xy 57.15 156.21))
-    (stroke (width 0) (type default))
-  )
   (wire (pts (xy 138.43 33.02) (xy 134.62 33.02))
     (stroke (width 0) (type default))
@@
     (stroke (width 0) (type default))
   )
-  (wire (pts (xy 57.15 156.21) (xy 68.58 156.21))
+  (wire (pts (xy 53.34 156.21) (xy 68.58 156.21))
     (stroke (width 0) (type default))
   )
@@
         (path "/e63e39d7-6ac0-4ffd-8aa3-1841a4541b55"
           (reference "#PWR0151") (unit 1)
-        )
-      )
-    )
-  )
-  (symbol (lib_id "Connector:TestPoint") (at 66.04 143.51 0) (unit 1)
-    (in_bom yes) (on_board yes) (dnp no)
-    (property "Reference" "TP9" (at 67.437 139.2995 0)
-      (effects (font (size 1.27 1.27)) (justify left))
-    )
-    (property "Value" "TP_DIN" (at 67.31 142.24 0)
-      (effects (font (size 1.27 1.27)) (justify left))
-    )
-    (property "Footprint" "TestPoint:TestPoint_Pad_D1.5mm" (at 71.12 143.51 0)
-      (effects (font (size 1.27 1.27)) hide)
-    )
-    (property "Datasheet" "~" (at 71.12 143.51 0)
-      (effects (font (size 1.27 1.27)) hide)
-    )
-    (property "LCSC Part" "" (at 66.04 143.51 0)
-      (effects (font (size 1.27 1.27)) hide)
-    )
-    (pin "1")
-    (instances
-      (project "VariometerV2.2.1"
-        (path "/9d9a2a31-8397-4ba2-ad51-8bee2c0fd904/056f5ab7-9063-4ff0-b10f-d2fc578ffe92"
-          (reference "TP9") (unit 1)
-        )
-      )
-      (project "VariometerV2.2"
-        (path "/e63e39d7-6ac0-4ffd-8aa3-1841a4541b55"
-          (reference "TP13") (unit 1)
         )
       )
@@
         (path "/e63e39d7-6ac0-4ffd-8aa3-1841a4541b55"
           (reference "U6") (unit 1)
-        )
-      )
-    )
-  )
-  (symbol (lib_id "Connector:TestPoint") (at 60.96 143.51 0) (unit 1)
-    (in_bom yes) (on_board yes) (dnp no)
-    (property "Reference" "TP8" (at 59.69 134.62 0)
-      (effects (font (size 1.27 1.27)) (justify left))
-    )
-    (property "Value" "TP_LRCLK" (at 57.15 137.16 0)
-      (effects (font (size 1.27 1.27)) (justify left))
-    )
-    (property "Footprint" "TestPoint:TestPoint_Pad_D1.5mm" (at 66.04 143.51 0)
-      (effects (font (size 1.27 1.27)) hide)
-    )
-    (property "Datasheet" "~" (at 66.04 143.51 0)
-      (effects (font (size 1.27 1.27)) hide)
-    )
-    (property "LCSC Part" "" (at 60.96 143.51 0)
-      (effects (font (size 1.27 1.27)) hide)
-    )
-    (pin "1")
-    (instances
-      (project "VariometerV2.2.1"
-        (path "/9d9a2a31-8397-4ba2-ad51-8bee2c0fd904/056f5ab7-9063-4ff0-b10f-d2fc578ffe92"
-          (reference "TP8") (unit 1)
-        )
-      )
-      (project "VariometerV2.2"
-        (path "/e63e39d7-6ac0-4ffd-8aa3-1841a4541b55"
-          (reference "TP12") (unit 1)
         )
       )
@@
         )
       )
-    )
-  )
-  (symbol (lib_id "Connector:TestPoint") (at 57.15 143.51 0) (unit 1)
-    (in_bom yes) (on_board yes) (dnp no)
-    (property "Reference" "TP7" (at 50.8 139.7 0)
-      (effects (font (size 1.27 1.27)) (justify left))
-    )
-    (property "Value" "TP_BCLK" (at 48.26 142.24 0)
-      (effects (font (size 1.27 1.27)) (justify left))
-    )
-    (property "Footprint" "TestPoint:TestPoint_Pad_D1.5mm" (at 62.23 143.51 0)
-      (effects (font (size 1.27 1.27)) hide)
-    )
-    (property "Datasheet" "~" (at 62.23 143.51 0)
-      (effects (font (size 1.27 1.27)) hide)
-    )
-    (property "LCSC Part" "" (at 57.15 143.51 0)
-      (effects (font (size 1.27 1.27)) hide)
-    )
-    (pin "1")
-    (instances
-      (project "VariometerV2.2.1"
-        (path "/9d9a2a31-8397-4ba2-ad51-8bee2c0fd904/056f5ab7-9063-4ff0-b10f-d2fc578ffe92"
-          (reference "TP7") (unit 1)
-        )
-      )
-      (project "VariometerV2.2"
-        (path "/e63e39d7-6ac0-4ffd-8aa3-1841a4541b55"
-          (reference "TP11") (unit 1)
-        )
-      )

Commit message: Routing ..
Parts:
- added C52: 10uF, Capacitor_SMD:C_0603_1608Metric, symbol Device:C_Small
Connections:
- net +3.1V_SW: now also C52.1
- net GND: now also C52.2
Changed lines of the file:
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@@
   (junction (at 228.6 99.06) (diameter 0) (color 0 0 0 0)
+  )
+  (junction (at 256.54 52.07) (diameter 0) (color 0 0 0 0)
   )
   (junction (at 73.66 29.21) (diameter 0) (color 0 0 0 0)
@@
     (stroke (width 0) (type default))
   )
+  (wire (pts (xy 270.51 50.8) (xy 270.51 52.07))
+    (stroke (width 0) (type default))
+  )
   (wire (pts (xy 242.57 120.65) (xy 254 120.65))
     (stroke (width 0) (type default))
   )
+  (wire (pts (xy 270.51 45.72) (xy 270.51 44.45))
+    (stroke (width 0) (type default))
+  )
   (wire (pts (xy 31.75 152.4) (xy 68.58 152.4))
     (stroke (width 0) (type default))
@@
     (stroke (width 0) (type default))
   )
+  (wire (pts (xy 256.54 52.07) (xy 270.51 52.07))
+    (stroke (width 0) (type default))
+  )
   (wire (pts (xy 266.7 113.03) (xy 266.7 111.76))
     (stroke (width 0) (type default))
@@
   )
   (wire (pts (xy 134.62 71.12) (xy 134.62 73.66))
+    (stroke (width 0) (type default))
+  )
+  (wire (pts (xy 270.51 44.45) (xy 256.54 44.45))
     (stroke (width 0) (type default))
   )
@@
         )
       )
+    )
+  )
+  (symbol (lib_id "Device:C_Small") (at 270.51 48.26 0) (mirror y) (unit 1)
+    (in_bom yes) (on_board yes) (dnp no)
+    (property "Reference" "C52" (at 278.13 45.72 0)
+      (effects (font (size 1.27 1.27)) (justify left))
+    )
+    (property "Value" "10uF" (at 278.13 48.26 0)
+      (effects (font (size 1.27 1.27)) (justify left))
+    )
+    (property "Footprint" "Capacitor_SMD:C_0603_1608Metric" (at 270.51 48.26 0)
+      (effects (font (size 1.27 1.27)) hide)
+    )
+    (property "Datasheet" "~" (at 270.51 48.26 0)
+      (effects (font (size 1.27 1.27)) hide)
+    )
+    (property "LCSC Part" "C307331" (at 270.51 48.26 0)
+      (effects (font (size 1.27 1.27)) hide)
+    )
+    (pin "1")
+    (pin "2")
+    (instances
+      (project "VariometerV2.2.1"
+        (path "/9d9a2a31-8397-4ba2-ad51-8bee2c0fd904/056f5ab7-9063-4ff0-b10f-d2fc578ffe92"
+          (reference "C52") (unit 1)
+        )
+      )
+      (project "VariometerV2.2"
+        (path "/e63e39d7-6ac0-4ffd-8aa3-1841a4541b55"
+          (reference "C29") (unit 1)
+        )
+      )
