File: Hardware/Version 2.1/VariometerV2.2.1/Sesnors.kicad_sch (KiCad schematic)
At the start: 32 parts, among them J1 U.FL-R-SMT(01), U4 DPS310, U5 BMI088, U6 QMC5883L, U7 MAX98357A, U8 L76-L

Commit message: PCB Routing Done
Changed lines of the file:
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@@
   (symbol (lib_id "VariometerV2:MAX98357A") (at 80.01 158.75 0) (unit 1)
     (in_bom yes) (on_board yes) (dnp no) (fields_autoplaced)
-    (property "Reference" "U7" (at 79.375 145.9443 0)
+    (property "Reference" "U7" (at 79.375 144.78 0)
       (effects (font (size 1.27 1.27)))
     )
-    (property "Value" "MAX98357A" (at 79.375 148.7194 0)
+    (property "Value" "MAX98357A" (at 79.375 147.32 0)
       (effects (font (size 1.27 1.27)))
     )

Commit message: Finish PCB
Parts:
- C52: LCSC Part C307331 -> C19702
- C7: footprint Capacitor_SMD:C_0402_1005Metric -> Capacitor_SMD:C_0603_1608Metric; LCSC Part C307331 -> C19702
- C9: footprint Capacitor_SMD:C_0402_1005Metric -> Capacitor_SMD:C_0603_1608Metric; LCSC Part C307331 -> C19666
- J1, JP1, JP3, JP5, JP7, U8: LCSC Part (none) -> 0
- L2: LCSC Part (none) -> C162657
- R10: LCSC Part (none) -> C22859
- R7: footprint Inductor_SMD:L_0603_1608Metric -> Resistor_SMD:R_0603_1608Metric; LCSC Part (none) -> C25804
Changed lines of the file:
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@@
+      (effects (font (size 1.27 1.27)) hide)
+    )
+    (property "LCSC Part" "0" (at 228.6 88.9 0)
       (effects (font (size 1.27 1.27)) hide)
     )
@@
       (effects (font (size 1.27 1.27)) hide)
     )
+    (property "LCSC Part" "0" (at 186.69 88.9 0)
+      (effects (font (size 1.27 1.27)) hide)
+    )
     (pin "1")
     (pin "2")
@@
     )
     (property "Datasheet" "~" (at 176.53 144.78 0)
+      (effects (font (size 1.27 1.27)) hide)
+    )
+    (property "LCSC Part" "C162657" (at 176.53 144.78 0)
       (effects (font (size 1.27 1.27)) hide)
     )
@@
     (property "MANUFACTURER" "Quectel" (at 222.25 133.35 0)
       (effects (font (size 1.27 1.27)) (justify bottom) hide)
+    )
+    (property "LCSC Part" "0" (at 222.25 133.35 0)
+      (effects (font (size 1.27 1.27)) hide)
     )
     (pin "1")
@@
       (effects (font (size 1.27 1.27)) (justify left))
     )
-    (property "Footprint" "Inductor_SMD:L_0603_1608Metric" (at 213.36 95.25 0)
+    (property "Footprint" "Resistor_SMD:R_0603_1608Metric" (at 213.36 95.25 0)
       (effects (font (size 1.27 1.27)) hide)
     )
     (property "Datasheet" "~" (at 213.36 95.25 0)
+      (effects (font (size 1.27 1.27)) hide)
+    )
+    (property "LCSC Part" "C25804" (at 213.36 95.25 0)
       (effects (font (size 1.27 1.27)) hide)
     )
@@
       (effects (font (size 1.27 1.27)) hide)
     )
-    (property "LCSC Part" "" (at 110.49 158.75 0)
+    (property "LCSC Part" "0" (at 110.49 158.75 0)
       (effects (font (size 1.27 1.27)) hide)
     )
@@
       (effects (font (size 1.27 1.27)) (justify left))
     )
-    (property "Footprint" "Capacitor_SMD:C_0402_1005Metric" (at 261.62 115.57 0)
+    (property "Footprint" "Capacitor_SMD:C_0603_1608Metric" (at 261.62 115.57 0)
       (effects (font (size 1.27 1.27)) hide)
     )
@@
       (effects (font (size 1.27 1.27)) hide)
     )
-    (property "LCSC Part" "C307331" (at 261.62 115.57 0)
+    (property "LCSC Part" "C19702" (at 261.62 115.57 0)
       (effects (font (size 1.27 1.27)) hide)
     )
@@
       (effects (font (size 1.27 1.27)) hide)
     )
+    (property "LCSC Part" "0" (at 176.53 137.16 0)
+      (effects (font (size 1.27 1.27)) hide)
+    )
     (pin "1")
     (pin "2")
@@
       (effects (font (size 1.27 1.27)) (justify bottom) hide)
     )
+    (property "LCSC Part" "0" (at 173.99 118.11 0)
+      (effects (font (size 1.27 1.27)) hide)
+    )
     (pin "1")
     (pin "2")
@@
       (effects (font (size 1.27 1.27)) hide)
     )
+    (property "LCSC Part" "C22859" (at 176.53 151.13 0)
+      (effects (font (size 1.27 1.27)) hide)
+    )
     (pin "1")
     (pin "2")
@@
       (effects (font (size 1.27 1.27)) (justify left))
     )
-    (property "Footprint" "Capacitor_SMD:C_0402_1005Metric" (at 266.7 92.71 0)
+    (property "Footprint" "Capacitor_SMD:C_0603_1608Metric" (at 266.7 92.71 0)
       (effects (font (size 1.27 1.27)) hide)
     )
@@
       (effects (font (size 1.27 1.27)) hide)
     )
-    (property "LCSC Part" "C307331" (at 266.7 92.71 0)
+    (property "LCSC Part" "C19666" (at 266.7 92.71 0)
       (effects (font (size 1.27 1.27)) hide)
     )
@@
       (effects (font (size 1.27 1.27)) hide)
     )
-    (property "LCSC Part" "C307331" (at 270.51 48.26 0)
-      (effects (font (size 1.27 1.27)) hide)
-    )
+    (property "LCSC Part" "C19702" (at 270.51 48.26 0)
+      (effects (font (size 1.27 1.27)) hide)
+    )
