File: Hardware/Version 2.1/VariometerV2.2.1/peripherals.kicad_sch (KiCad schematic)
At the start: 23 parts, among them J1 USB_C_Receptacle_USB2.0, J2 Conn_01x02, J3 Conn_01x02, J4 Conn_01x02, J5 Conn_01x02, J6 Conn_01x02, J7 Conn_01x02, U1 SRV05-4

Commit message: Develop Board
Other:
- moved on the sheet: J2, J7
Changed lines of the file:
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@@
   (junction (at 109.22 147.32) (diameter 0) (color 0 0 0 0)
   )
-  (junction (at 170.18 60.96) (diameter 0) (color 0 0 0 0)
+  (junction (at 168.91 71.12) (diameter 0) (color 0 0 0 0)
   )
   (junction (at 59.69 50.8) (diameter 0) (color 0 0 0 0)
@@
     (stroke (width 0) (type default))
   )
-  (wire (pts (xy 165.1 60.96) (xy 170.18 60.96))
+  (wire (pts (xy 163.83 71.12) (xy 168.91 71.12))
     (stroke (width 0) (type default))
   )
@@
     (stroke (width 0) (type default))
   )
-  (wire (pts (xy 170.18 63.5) (xy 171.45 63.5))
+  (wire (pts (xy 168.91 73.66) (xy 170.18 73.66))
     (stroke (width 0) (type default))
   )
@@
     (stroke (width 0) (type default))
   )
-  (wire (pts (xy 165.1 59.69) (xy 165.1 60.96))
+  (wire (pts (xy 163.83 69.85) (xy 163.83 71.12))
     (stroke (width 0) (type default))
   )
@@
     (stroke (width 0) (type default))
   )
-  (wire (pts (xy 170.18 64.77) (xy 170.18 63.5))
+  (wire (pts (xy 168.91 74.93) (xy 168.91 73.66))
     (stroke (width 0) (type default))
   )
@@
     (stroke (width 0) (type default))
   )
-  (wire (pts (xy 170.18 60.96) (xy 171.45 60.96))
+  (wire (pts (xy 168.91 71.12) (xy 170.18 71.12))
     (stroke (width 0) (type default))
   )
@@
     (stroke (width 0) (type default))
   )
-  (wire (pts (xy 170.18 59.69) (xy 170.18 60.96))
+  (wire (pts (xy 168.91 69.85) (xy 168.91 71.12))
     (stroke (width 0) (type default))
   )
@@
     (effects (font (size 1.27 1.27)) (justify left bottom))
   )
-  (text "SPEAKER CONNECTOR" (at 165.1 41.91 0)
+  (text "SPEAKER CONNECTOR" (at 160.02 45.72 0)
     (effects (font (size 1.27 1.27)) (justify left bottom))
   )
-  (text "BATTERY CONNECTOR" (at 162.56 73.66 0)
+  (text "BATTERY CONNECTOR" (at 161.29 83.82 0)
     (effects (font (size 1.27 1.27)) (justify left bottom))
   )
@@
     (effects (font (size 1.27 1.27)) (justify left bottom))
   )
-  (global_label "AUDIO_OUTP" (shape input) (at 171.45 35.56 180) (fields_autoplaced)
+  (global_label "AUDIO_OUTP" (shape input) (at 166.37 39.37 180) (fields_autoplaced)
     (effects (font (size 1.27 1.27)) (justify right))
-    (property "Intersheetrefs" "${INTERSHEET_REFS}" (at 157.5464 35.6394 0)
+    (property "Intersheetrefs" "${INTERSHEET_REFS}" (at 152.4664 39.4494 0)
       (effects (font (size 1.27 1.27)) (justify right) hide)
     )
@@
     )
   )
-  (global_label "AUDIO_OUTN" (shape input) (at 171.45 33.02 180) (fields_autoplaced)
+  (global_label "AUDIO_OUTN" (shape input) (at 166.37 36.83 180) (fields_autoplaced)
     (effects (font (size 1.27 1.27)) (justify right))
-    (property "Intersheetrefs" "${INTERSHEET_REFS}" (at 157.4859 33.0994 0)
+    (property "Intersheetrefs" "${INTERSHEET_REFS}" (at 152.4059 36.9094 0)
       (effects (font (size 1.27 1.27)) (justify right) hide)
     )
@@
     )
   )
-  (symbol (lib_id "power:+BATT") (at 170.18 59.69 0) (unit 1)
-    (in_bom yes) (on_board yes) (dnp no)
-    (property "Reference" "#PWR018" (at 170.18 63.5 0)
-      (effects (font (size 1.27 1.27)) hide)
-    )
-    (property "Value" "+BATT" (at 171.45 55.88 0)
-      (effects (font (size 1.27 1.27)))
-    )
-    (property "Footprint" "" (at 170.18 59.69 0)
-      (effects (font (size 1.27 1.27)) hide)
-    )
-    (property "Datasheet" "" (at 170.18 59.69 0)
+  (symbol (lib_id "power:+BATT") (at 168.91 69.85 0) (unit 1)
+    (in_bom yes) (on_board yes) (dnp no)
+    (property "Reference" "#PWR018" (at 168.91 73.66 0)
+      (effects (font (size 1.27 1.27)) hide)
+    )
+    (property "Value" "+BATT" (at 170.18 66.04 0)
+      (effects (font (size 1.27 1.27)))
+    )
+    (property "Footprint" "" (at 168.91 69.85 0)
+      (effects (font (size 1.27 1.27)) hide)
+    )
+    (property "Datasheet" "" (at 168.91 69.85 0)
       (effects (font (size 1.27 1.27)) hide)
     )
@@
     )
   )
-  (symbol (lib_id "power:PWR_FLAG") (at 165.1 59.69 0) (unit 1)
-    (in_bom yes) (on_board yes) (dnp no)
-    (property "Reference" "#FLG01" (at 165.1 57.785 0)
-      (effects (font (size 1.27 1.27)) hide)
-    )
-    (property "Value" "PWR_FLAG" (at 158.75 57.15 0)
-      (effects (font (size 1.27 1.27)))
-    )
-    (property "Footprint" "" (at 165.1 59.69 0)
-      (effects (font (size 1.27 1.27)) hide)
-    )
-    (property "Datasheet" "~" (at 165.1 59.69 0)
+  (symbol (lib_id "power:PWR_FLAG") (at 163.83 69.85 0) (unit 1)
+    (in_bom yes) (on_board yes) (dnp no)
+    (property "Reference" "#FLG01" (at 163.83 67.945 0)
+      (effects (font (size 1.27 1.27)) hide)
+    )
+    (property "Value" "PWR_FLAG" (at 157.48 67.31 0)
+      (effects (font (size 1.27 1.27)))
+    )
+    (property "Footprint" "" (at 163.83 69.85 0)
+      (effects (font (size 1.27 1.27)) hide)
+    )
+    (property "Datasheet" "~" (at 163.83 69.85 0)
       (effects (font (size 1.27 1.27)) hide)
     )
@@
     )
   )
-  (symbol (lib_id "power:GND") (at 170.18 64.77 0) (unit 1)
-    (in_bom yes) (on_board yes) (dnp no)
-    (property "Reference" "#PWR023" (at 170.18 71.12 0)
-      (effects (font (size 1.27 1.27)) hide)
-    )
-    (property "Value" "GND" (at 170.307 69.1642 0)
-      (effects (font (size 1.27 1.27)))
-    )
-    (property "Footprint" "" (at 170.18 64.77 0)
-      (effects (font (size 1.27 1.27)) hide)
-    )
-    (property "Datasheet" "" (at 170.18 64.77 0)
+  (symbol (lib_id "power:GND") (at 168.91 74.93 0) (unit 1)
+    (in_bom yes) (on_board yes) (dnp no)
+    (property "Reference" "#PWR023" (at 168.91 81.28 0)
+      (effects (font (size 1.27 1.27)) hide)
+    )
+    (property "Value" "GND" (at 169.037 79.3242 0)
+      (effects (font (size 1.27 1.27)))
+    )
+    (property "Footprint" "" (at 168.91 74.93 0)
+      (effects (font (size 1.27 1.27)) hide)
+    )
+    (property "Datasheet" "" (at 168.91 74.93 0)
       (effects (font (size 1.27 1.27)) hide)
     )
@@
     )
   )
-  (symbol (lib_id "Connector_Generic:Conn_01x02") (at 176.53 33.02 0) (unit 1)
-    (in_bom yes) (on_board yes) (dnp no) (fields_autoplaced)
-    (property "Reference" "J2" (at 178.562 33.3815 0)
-      (effects (font (size 1.27 1.27)) (justify left))
-    )
-    (property "Value" "Conn_01x02" (at 178.562 36.1566 0)
-      (effects (font (size 1.27 1.27)) (justify left))
-    )
-    (property "Footprint" "Connector_PinHeader_2.54mm:PinHeader_1x02_P2.54mm_Vertical" (at 176.53 33.02 0)
-      (effects (font (size 1.27 1.27)) hide)
-    )
-    (property "Datasheet" "~" (at 176.53 33.02 0)
+  (symbol (lib_id "Connector_Generic:Conn_01x02") (at 171.45 36.83 0) (unit 1)
+    (in_bom yes) (on_board yes) (dnp no) (fields_autoplaced)
+    (property "Reference" "J2" (at 173.482 37.1915 0)
+      (effects (font (size 1.27 1.27)) (justify left))
+    )
+    (property "Value" "Conn_01x02" (at 173.482 39.9666 0)
+      (effects (font (size 1.27 1.27)) (justify left))
+    )
+    (property "Footprint" "Connector_PinHeader_2.54mm:PinHeader_1x02_P2.54mm_Vertical" (at 171.45 36.83 0)
+      (effects (font (size 1.27 1.27)) hide)
+    )
+    (property "Datasheet" "~" (at 171.45 36.83 0)
       (effects (font (size 1.27 1.27)) hide)
     )
@@
     )
   )
-  (symbol (lib_id "Connector_Generic:Conn_01x02") (at 176.53 60.96 0) (unit 1)
-    (in_bom yes) (on_board yes) (dnp no) (fields_autoplaced)
-    (property "Reference" "J7" (at 179.07 61.595 0)
-      (effects (font (size 1.27 1.27)) (justify left))
-    )
-    (property "Value" "Conn_01x02" (at 179.07 64.135 0)
-      (effects (font (size 1.27 1.27)) (justify left))
-    )
-    (property "Footprint" "" (at 176.53 60.96 0)
-      (effects (font (size 1.27 1.27)) hide)
-    )
-    (property "Datasheet" "~" (at 176.53 60.96 0)
-      (effects (font (size 1.27 1.27)) hide)
-    )
+  (symbol (lib_id "Connector_Generic:Conn_01x02") (at 175.26 71.12 0) (unit 1)
+    (in_bom yes) (on_board yes) (dnp no) (fields_autoplaced)
+    (property "Reference" "J7" (at 177.8 71.755 0)
+      (effects (font (size 1.27 1.27)) (justify left))
+    )
+    (property "Value" "Conn_01x02" (at 177.8 74.295 0)
+      (effects (font (size 1.27 1.27)) (justify left))
+    )
+    (property "Footprint" "" (at 175.26 71.12 0)
+      (effects (font (size 1.27 1.27)) hide)
+    )
+    (property "Datasheet" "~" (at 175.26 71.12 0)
+      (effects (font (size 1.27 1.27)) hide)
+    )

Commit message: Working on PCB
Parts:
- added C20: 100nF, Capacitor_SMD:C_0402_1005Metric, symbol Device:C_Small
- added C21, C22: 2.2uF, Capacitor_SMD:C_0603_1608Metric, symbol Device:C_Small
- added FB1: 600 @ 100 MHz, Inductor_SMD:L_0603_1608Metric, symbol Device:FerriteBead_Small
- added J10: ~, symbol Main_LibraryVario:Micro_SD_Card
- added R25, R26: 10k, symbol Device:R_Small
- added R27, R28, R29, R30, R31, R32: 10k, Resistor_SMD:R_0402_1005Metric, symbol Device:R_Small
- added R33: 22, Resistor_SMD:R_0402_1005Metric, symbol Device:R_Small
- added U2, U3: SRV05-4, Package_TO_SOT_SMD:SOT-23-6, symbol Power_Protection:SRV05-4
- R3: value 5.1 -> 5.1k
Connections:
- net GND: now also U1.2 (VN), C20.2, C21.2, C22.2, J10.6 (VSS), J10.G1 (GND), U2.2 (VN), U3.2 (VN)
- new net: J10.5 (CLK), R33.2, U3.6 (IO4)
- new net: R26.2, U3.5 (VP)
- new net: R25.2, U2.5 (VP)
- new net +3.1V_SW: C22.1, FB1.2, R25.1, R26.1, R27.1, R28.1, R29.1, R30.1, R31.1, R32.1
- new net 3.1V_SDCARD: C20.1, C21.1, FB1.1, J10.4 (VDD), U2.6 (IO4)
- new net SD_CD: J10.9 (DET), R32.2, U3.4 (IO3)
- new net SD_CLK: R33.1
- new net SD_CMD: J10.3 (CMD), R29.2, U2.4 (IO3)
- new net SD_DAT0: J10.7 (DAT0), R30.2, U3.1 (IO1)
- new net SD_DAT1: J10.8 (DAT1), R31.2, U3.3 (IO2)
- new net SD_DAT2: J10.1 (DAT2), R27.2, U2.3 (IO2)
- new net SD_DAT3: J10.2 (DAT3/CD), R28.2, U2.1 (IO1)
- no-connect marks 0 -> 5
Other:
- note added: "Micro SD-Card"
- moved on the sheet: C6, C7, C8, C9, J1, J2, J3, J4, J5, J6, J7, R10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

Commit message: Weiter PCB
Parts:
- R32: value 10k -> S10k
Changed lines of the file:
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@@
     (stroke (width 0) (type default))
   )
-  (wire (pts (xy 222.25 66.04) (xy 222.25 24.13))
+  (wire (pts (xy 223.52 66.04) (xy 223.52 24.13))
     (stroke (width 0) (type default))
   )
@@
     (stroke (width 0) (type default))
   )
-  (wire (pts (xy 222.25 66.04) (xy 229.87 66.04))
+  (wire (pts (xy 223.52 66.04) (xy 229.87 66.04))
     (stroke (width 0) (type default))
   )
@@
     (stroke (width 0) (type default))
   )
-  (wire (pts (xy 222.25 24.13) (xy 237.49 24.13))
+  (wire (pts (xy 223.52 24.13) (xy 237.49 24.13))
     (stroke (width 0) (type default))
   )
@@
       (effects (font (size 1.27 1.27)) (justify left))
     )
-    (property "Value" "10k" (at 217.3986 40.513 0)
-      (effects (font (size 1.27 1.27)) (justify left))
-    )
+    (property "Value" "S10k" (at 217.3986 40.513 0)
+      (effects (font (size 1.27 1.27)) (justify left))
+    )

Commit message: Update Schematics
Parts:
- removed C7, C8, C9: 1uF, Capacitor_SMD:C_0603_1608Metric, symbol Device:C_Small
- removed J10: ~, symbol Main_LibraryVario:Micro_SD_Card
- removed J3, J4, J5, J6: Conn_01x02, Connector_PinHeader_2.54mm:PinHeader_1x02_P2.54mm_Vertical, symbol Connector_Generic:Conn_01x02
- removed R10, R12, R8: 1k, Resistor_SMD:R_0603_1608Metric, symbol Device:R_Small
- removed R11, R7, R9: 10k, Resistor_SMD:R_0603_1608Metric, symbol Device:R_Small
- added C47, C48, C49: 1uF, Capacitor_SMD:C_0402_1005Metric, symbol Device:C_Small
- added J3: ~, MainLibrary:TFP09212B, symbol Main_LibraryVario:Micro_SD_Card
- added R44, R46, R48: 10k, symbol Device:R_Small
- added R45, R47, R49: 1k, symbol Device:R_Small
- added SW3, SW4, SW5, SW6: BTN1, Button_Switch_THT:SW_PUSH_6mm, symbol VariometerV2-rescue:Switch_SW_Push-VariometerV2-cache
- added TP11: CC1, symbol Connector:TestPoint
- added TP12: CC2, symbol Connector:TestPoint
- C6: footprint Capacitor_SMD:C_0603_1608Metric -> Capacitor_SMD:C_0402_1005Metric
- J1: footprint (none) -> Connector_USB:USB_C_Receptacle_HRO_TYPE-C-31-M-12
- J2: footprint Connector_PinHeader_2.54mm:PinHeader_1x02_P2.54mm_Vertical -> (none)
- R27, R28, R29, R30, R31, R33: footprint Resistor_SMD:R_0402_1005Metric -> (none)
- R32: value S10k -> 10k S; footprint Resistor_SMD:R_0402_1005Metric -> (none)
- R5, R6: footprint Resistor_SMD:R_0603_1608Metric -> (none)
- U1, U2, U3: footprint Package_TO_SOT_SMD:SOT-23-6 -> (none)
Connections:
- net +3.1V_UNSW: now also R44.1, R46.1, R48.1
- net 3.1V_SDCARD: now also J3.4 (VDD)
- net BUTTON_2: now also C47.1, R45.2
- net BUTTON_3: now also C48.1, R47.2
- net BUTTON_4: now also C49.1, R49.2
- net GND: now also C47.2, C48.2, C49.2, J3.6 (VSS), J3.G1 (GND), SW3.1, SW4.1, SW5.1, SW6.1
- net SD_CD: now also J3.CD1 (DET)
- net SD_CMD: now also J3.3 (CMD)
- net SD_DAT0: now also J3.7 (DAT0)
- net SD_DAT1: now also J3.8 (DAT1)
- net SD_DAT2: now also J3.1 (DAT2)
- net SD_DAT3: now also J3.2 (DAT3/CD)
- net at R33.2, U3.6 (IO4): now also J3.5 (CLK)
- net USB_CC1: now reaches J1.A5 (CC1), R3.1
- net USB_CC1: now also TP11.1
- net at R5.2, R6.1: now also SW3.2
- net USB_CC2: now reaches J1.B5 (CC2), R2.1
- net USB_CC2: now also TP12.1
- new net: R46.2, R47.1, SW5.2
- new net: R48.2, R49.1, SW6.2
- new net: R44.2, R45.1, SW4.2
- no-connect marks 5 -> 7
Other:
- moved on the sheet: C6, R3, R5, R6

Commit message: Working on PCB
Parts:
- R2, R3, R32: footprint (none) -> Resistor_SMD:R_0805_2012Metric
- R25, R26, R4: footprint (none) -> Resistor_SMD:R_0603_1608Metric
- R27, R28, R29, R30, R31, R33, R44, R45, R46, R47, R48, R49, R5, R6: footprint (none) -> Resistor_SMD:R_0402_1005Metric
- TP11, TP12: footprint (none) -> TestPoint:TestPoint_Pad_D1.5mm
- U1, U2, U3: footprint (none) -> Package_TO_SOT_SMD:SOT-23-6
Changed lines of the file:
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@@
       (effects (font (size 1.27 1.27)) (justify left))
     )
-    (property "Footprint" "" (at 189.23 40.64 0)
+    (property "Footprint" "Resistor_SMD:R_0402_1005Metric" (at 189.23 40.64 0)
       (effects (font (size 1.27 1.27)) hide)
     )
@@
       (effects (font (size 1.27 1.27)) (justify left))
     )
-    (property "Footprint" "" (at 170.18 68.58 0)
+    (property "Footprint" "Resistor_SMD:R_0402_1005Metric" (at 170.18 68.58 0)
       (effects (font (size 1.27 1.27)) hide)
     )
@@
       (effects (font (size 1.27 1.27)) (justify left))
     )
-    (property "Footprint" "" (at 162.56 39.37 0)
+    (property "Footprint" "Resistor_SMD:R_0402_1005Metric" (at 162.56 39.37 0)
       (effects (font (size 1.27 1.27)) hide)
     )
@@
       (effects (font (size 1.27 1.27)) (justify left))
     )
-    (property "Footprint" "" (at 105.41 31.75 0)
+    (property "Footprint" "TestPoint:TestPoint_Pad_D1.5mm" (at 105.41 31.75 0)
       (effects (font (size 1.27 1.27)) hide)
     )
@@
       (effects (font (size 1.27 1.27)) (justify left))
     )
-    (property "Footprint" "" (at 116.84 157.48 0)
+    (property "Footprint" "Resistor_SMD:R_0402_1005Metric" (at 116.84 157.48 0)
       (effects (font (size 1.27 1.27)) hide)
     )
@@
       (effects (font (size 1.27 1.27)) (justify left))
     )
-    (property "Footprint" "" (at 91.44 31.75 0)
+    (property "Footprint" "TestPoint:TestPoint_Pad_D1.5mm" (at 91.44 31.75 0)
       (effects (font (size 1.27 1.27)) hide)
     )
@@
       (effects (font (size 1.27 1.27)) (justify left))
     )
-    (property "Footprint" "" (at 153.67 157.48 0)
+    (property "Footprint" "Resistor_SMD:R_0402_1005Metric" (at 153.67 157.48 0)
       (effects (font (size 1.27 1.27)) hide)
     )
@@
       (effects (font (size 1.27 1.27)) (justify left))
     )
-    (property "Footprint" "" (at 210.82 97.79 0)
+    (property "Footprint" "Resistor_SMD:R_0603_1608Metric" (at 210.82 97.79 0)
       (effects (font (size 1.27 1.27)) hide)
     )
@@
       (effects (font (size 1.27 1.27)) (justify left))
     )
-    (property "Footprint" "" (at 146.05 153.67 0)
+    (property "Footprint" "Resistor_SMD:R_0402_1005Metric" (at 146.05 153.67 0)
       (effects (font (size 1.27 1.27)) hide)
     )
@@
       (effects (font (size 1.27 1.27)))
     )
-    (property "Footprint" "" (at 187.96 125.73 0)
+    (property "Footprint" "Package_TO_SOT_SMD:SOT-23-6" (at 187.96 125.73 0)
       (effects (font (size 1.27 1.27)) hide)
     )
@@
       (effects (font (size 1.27 1.27)) (justify left))
     )
-    (property "Footprint" "" (at 209.55 39.37 0)
+    (property "Footprint" "Resistor_SMD:R_0402_1005Metric" (at 209.55 39.37 0)
       (effects (font (size 1.27 1.27)) hide)
     )
@@
       (effects (font (size 1.27 1.27)) (justify left))
     )
-    (property "Footprint" "" (at 109.22 41.91 0)
+    (property "Footprint" "Resistor_SMD:R_0805_2012Metric" (at 109.22 41.91 0)
       (effects (font (size 1.27 1.27)) hide)
     )
@@
       (effects (font (size 1.27 1.27)) (justify left))
     )
-    (property "Footprint" "" (at 109.22 153.67 0)
+    (property "Footprint" "Resistor_SMD:R_0402_1005Metric" (at 109.22 153.67 0)
       (effects (font (size 1.27 1.27)) hide)
     )
@@
       (effects (font (size 1.27 1.27)) (justify left))
     )
-    (property "Footprint" "" (at 41.91 157.48 0)
+    (property "Footprint" "Resistor_SMD:R_0402_1005Metric" (at 41.91 157.48 0)
       (effects (font (size 1.27 1.27)) hide)
     )
@@
       (effects (font (size 1.27 1.27)) (justify left))
     )
-    (property "Footprint" "" (at 90.17 86.36 0)
+    (property "Footprint" "Package_TO_SOT_SMD:SOT-23-6" (at 90.17 86.36 0)
       (effects (font (size 1.27 1.27)) hide)
     )
@@
       (effects (font (size 1.27 1.27)) (justify left))
     )
-    (property "Footprint" "" (at 91.44 41.91 0)
+    (property "Footprint" "Resistor_SMD:R_0805_2012Metric" (at 91.44 41.91 0)
       (effects (font (size 1.27 1.27)) hide)
     )
@@
       (effects (font (size 1.27 1.27)) (justify left))
     )
-    (property "Footprint" "" (at 170.18 97.79 0)
+    (property "Footprint" "Resistor_SMD:R_0603_1608Metric" (at 170.18 97.79 0)
       (effects (font (size 1.27 1.27)) hide)
     )
@@
       (effects (font (size 1.27 1.27)) (justify left))
     )
-    (property "Footprint" "" (at 215.9 39.37 0)
+    (property "Footprint" "Resistor_SMD:R_0805_2012Metric" (at 215.9 39.37 0)
       (effects (font (size 1.27 1.27)) hide)
     )
@@
       (effects (font (size 1.27 1.27)) (justify left))
     )
-    (property "Footprint" "" (at 80.01 157.48 0)
+    (property "Footprint" "Resistor_SMD:R_0402_1005Metric" (at 80.01 157.48 0)
       (effects (font (size 1.27 1.27)) hide)
     )
@@
       (effects (font (size 1.27 1.27)))
     )
-    (property "Footprint" "" (at 228.6 125.73 0)
+    (property "Footprint" "Package_TO_SOT_SMD:SOT-23-6" (at 228.6 125.73 0)
       (effects (font (size 1.27 1.27)) hide)
     )
@@
       (effects (font (size 1.27 1.27)) (justify left))
     )
-    (property "Footprint" "" (at 34.29 153.67 0)
+    (property "Footprint" "Resistor_SMD:R_0402_1005Metric" (at 34.29 153.67 0)
       (effects (font (size 1.27 1.27)) hide)
     )
@@
       (effects (font (size 1.27 1.27)) (justify left))
     )
-    (property "Footprint" "" (at 200.66 39.37 0)
+    (property "Footprint" "Resistor_SMD:R_0402_1005Metric" (at 200.66 39.37 0)
       (effects (font (size 1.27 1.27)) hide)
     )
@@
       (effects (font (size 1.27 1.27)) (justify left))
     )
-    (property "Footprint" "" (at 168.91 39.37 0)
+    (property "Footprint" "Resistor_SMD:R_0402_1005Metric" (at 168.91 39.37 0)
       (effects (font (size 1.27 1.27)) hide)
     )
@@
       (effects (font (size 1.27 1.27)) (justify left))
     )
-    (property "Footprint" "" (at 72.39 57.15 0)
+    (property "Footprint" "Resistor_SMD:R_0603_1608Metric" (at 72.39 57.15 0)
       (effects (font (size 1.27 1.27)) hide)
     )
@@
       (effects (font (size 1.27 1.27)) (justify left))
     )
-    (property "Footprint" "" (at 72.39 153.67 0)
-      (effects (font (size 1.27 1.27)) hide)
-    )
+    (property "Footprint" "Resistor_SMD:R_0402_1005Metric" (at 72.39 153.67 0)
+      (effects (font (size 1.27 1.27)) hide)
+    )
