File: Hardware/Version 2.1/VariometerV2.2.1/peripherals.kicad_sch (KiCad schematic)
At the start: 41 parts, among them J1 USB_C_Receptacle_USB2.0, J2 Conn_01x02, J7 Conn_01x02, SW3 BTN1, SW4 BTN1, SW5 BTN1, SW6 BTN1, U1 SRV05-4, U2 SRV05-4, U3 SRV05-4

Commit message: PCB
Parts:
- C20: JLCPCB Part # C307331 -> (none); LCSC Part (none) -> C307331
- C21, C22: JLCPCB Part # C23630 -> (none); LCSC Part (none) -> C23630
- C47, C48, C49, C6: JLCPCB Part # C15849 -> (none); LCSC Part (none) -> C52923
- FB1: JLCPCB Part # C1002 -> (none); LCSC Part (none) -> C1002
- J1: LCSC Part (none) -> C165948
- R2, R3: LCSC Part (none) -> C27834
- R25, R26, R4: LCSC Part (none) -> C25804
- R27, R28, R29, R30, R31: JLCPCB Part # C25744 -> (none); LCSC Part (none) -> C25744
- R32: JLCPCB Part # C25744 -> (none); LCSC Part (none) -> C17414
- R33: JLCPCB Part # C25092 -> (none); LCSC Part (none) -> C25092
- R44, R46, R48, R5: JLCPCB Part # C25804 -> (none); LCSC Part (none) -> C25744
- R45, R47, R49, R6: JLCPCB Part # C21190 -> (none); LCSC Part (none) -> C11702
- U1: LCSC Part (none) -> C85364
- U2, U3: JLCPCB Part # C85364 -> (none); LCSC Part (none) -> C85364
Changed lines of the file:
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@@
       (effects (font (size 1.27 1.27)) hide)
     )
-    (property "JLCPCB Part #" "C25744" (at 189.23 40.64 0)
+    (property "LCSC Part" "C25744" (at 189.23 40.64 0)
       (effects (font (size 1.27 1.27)) hide)
     )
@@
       (effects (font (size 1.27 1.27)) hide)
     )
-    (property "JLCPCB Part #" "C25092" (at 170.18 68.58 0)
+    (property "LCSC Part" "C25092" (at 170.18 68.58 0)
       (effects (font (size 1.27 1.27)) hide)
     )
@@
       (effects (font (size 1.27 1.27)) hide)
     )
-    (property "JLCPCB Part #" "C15849" (at 82.55 172.72 0)
+    (property "LCSC Part" "C52923" (at 82.55 172.72 0)
       (effects (font (size 1.27 1.27)) hide)
     )
@@
       (effects (font (size 1.27 1.27)) hide)
     )
-    (property "JLCPCB Part #" "C1002" (at 256.54 24.13 0)
+    (property "LCSC Part" "C1002" (at 256.54 24.13 0)
       (effects (font (size 1.27 1.27)) hide)
     )
@@
       (effects (font (size 1.27 1.27)) hide)
     )
-    (property "JLCPCB Part #" "C25744" (at 162.56 39.37 0)
+    (property "LCSC Part" "C25744" (at 162.56 39.37 0)
       (effects (font (size 1.27 1.27)) hide)
     )
@@
       (effects (font (size 1.27 1.27)) hide)
     )
+    (property "LCSC Part" "" (at 100.33 31.75 0)
+      (effects (font (size 1.27 1.27)) hide)
+    )
     (pin "1")
     (instances
@@
       (effects (font (size 1.27 1.27)) hide)
     )
-    (property "JLCPCB Part #" "C21190" (at 116.84 157.48 0)
+    (property "LCSC Part" "C11702" (at 116.84 157.48 0)
       (effects (font (size 1.27 1.27)) hide)
     )
@@
       (effects (font (size 1.27 1.27)) hide)
     )
+    (property "LCSC Part" "" (at 86.36 31.75 0)
+      (effects (font (size 1.27 1.27)) hide)
+    )
     (pin "1")
     (instances
@@
       (effects (font (size 1.27 1.27)) hide)
     )
-    (property "JLCPCB Part #" "C21190" (at 153.67 157.48 0)
+    (property "LCSC Part" "C11702" (at 153.67 157.48 0)
       (effects (font (size 1.27 1.27)) hide)
     )
@@
       (effects (font (size 1.27 1.27)) hide)
     )
+    (property "LCSC Part" "C25804" (at 210.82 97.79 0)
+      (effects (font (size 1.27 1.27)) hide)
+    )
     (pin "1")
     (pin "2")
@@
     )
     (property "Datasheet" "" (at 248.92 46.99 0)
+      (effects (font (size 1.27 1.27)) hide)
+    )
+    (property "LCSC Part" "" (at 251.46 68.58 0)
       (effects (font (size 1.27 1.27)) hide)
     )
@@
       (effects (font (size 1.27 1.27)) hide)
     )
-    (property "JLCPCB Part #" "C25804" (at 146.05 153.67 0)
+    (property "LCSC Part" "C25744" (at 146.05 153.67 0)
       (effects (font (size 1.27 1.27)) hide)
     )
@@
       (effects (font (size 1.27 1.27)) hide)
     )
-    (property "JLCPCB Part #" "C85364" (at 170.18 114.3 0)
+    (property "LCSC Part" "C85364" (at 170.18 114.3 0)
       (effects (font (size 1.27 1.27)) hide)
     )
@@
       (effects (font (size 1.27 1.27)) hide)
     )
-    (property "JLCPCB Part #" "C307331" (at 237.49 30.48 0)
+    (property "LCSC Part" "C307331" (at 237.49 30.48 0)
       (effects (font (size 1.27 1.27)) hide)
     )
@@
       (effects (font (size 1.27 1.27)) hide)
     )
-    (property "JLCPCB Part #" "C25744" (at 209.55 39.37 0)
+    (property "LCSC Part" "C25744" (at 209.55 39.37 0)
       (effects (font (size 1.27 1.27)) hide)
     )
@@
       (effects (font (size 1.27 1.27)) hide)
     )
+    (property "LCSC Part" "C27834" (at 109.22 41.91 0)
+      (effects (font (size 1.27 1.27)) hide)
+    )
     (pin "1")
     (pin "2")
@@
       (effects (font (size 1.27 1.27)) hide)
     )
-    (property "JLCPCB Part #" "C25804" (at 109.22 153.67 0)
+    (property "LCSC Part" "C25744" (at 109.22 153.67 0)
       (effects (font (size 1.27 1.27)) hide)
     )
@@
       (effects (font (size 1.27 1.27)) hide)
     )
-    (property "JLCPCB Part #" "C21190" (at 41.91 157.48 0)
+    (property "LCSC Part" "C11702" (at 41.91 157.48 0)
       (effects (font (size 1.27 1.27)) hide)
     )
@@
       (effects (font (size 1.27 1.27)) hide)
     )
-    (property "JLCPCB Part #" "C15849" (at 156.21 172.72 0)
+    (property "LCSC Part" "C52923" (at 156.21 172.72 0)
       (effects (font (size 1.27 1.27)) hide)
     )
@@
     )
     (property "Datasheet" "https://www.usb.org/sites/default/files/documents/usb_type-c.zip" (at 40.64 45.72 0)
+      (effects (font (size 1.27 1.27)) hide)
+    )
+    (property "LCSC Part" "C165948" (at 36.83 45.72 0)
       (effects (font (size 1.27 1.27)) hide)
     )
@@
       (effects (font (size 1.27 1.27)) hide)
     )
+    (property "LCSC Part" "C85364" (at 72.39 74.93 0)
+      (effects (font (size 1.27 1.27)) hide)
+    )
     (pin "1")
     (pin "2")
@@
       (effects (font (size 1.27 1.27)) hide)
     )
+    (property "LCSC Part" "C27834" (at 91.44 41.91 0)
+      (effects (font (size 1.27 1.27)) hide)
+    )
     (pin "1")
     (pin "2")
@@
       (effects (font (size 1.27 1.27)) hide)
     )
+    (property "LCSC Part" "" (at 72.39 168.91 0)
+      (effects (font (size 1.27 1.27)) hide)
+    )
     (pin "1")
     (pin "2")
@@
       (effects (font (size 1.27 1.27)) hide)
     )
+    (property "LCSC Part" "C25804" (at 170.18 97.79 0)
+      (effects (font (size 1.27 1.27)) hide)
+    )
     (pin "1")
     (pin "2")
@@
       (effects (font (size 1.27 1.27)) hide)
     )
-    (property "JLCPCB Part #" "C15849" (at 119.38 172.72 0)
+    (property "LCSC Part" "C52923" (at 119.38 172.72 0)
       (effects (font (size 1.27 1.27)) hide)
     )
@@
       (effects (font (size 1.27 1.27)) hide)
     )
+    (property "LCSC Part" "" (at 34.29 168.91 0)
+      (effects (font (size 1.27 1.27)) hide)
+    )
     (pin "1")
     (pin "2")
@@
       (effects (font (size 1.27 1.27)) hide)
     )
-    (property "JLCPCB Part #" "C25744" (at 215.9 39.37 0)
+    (property "LCSC Part" "C17414" (at 215.9 39.37 0)
       (effects (font (size 1.27 1.27)) hide)
     )
@@
       (effects (font (size 1.27 1.27)) hide)
     )
-    (property "JLCPCB Part #" "C21190" (at 80.01 157.48 0)
+    (property "LCSC Part" "C11702" (at 80.01 157.48 0)
       (effects (font (size 1.27 1.27)) hide)
     )
@@
       (effects (font (size 1.27 1.27)) hide)
     )
-    (property "JLCPCB Part #" "C85364" (at 210.82 114.3 0)
+    (property "LCSC Part" "C85364" (at 210.82 114.3 0)
       (effects (font (size 1.27 1.27)) hide)
     )
@@
       (effects (font (size 1.27 1.27)) hide)
     )
-    (property "JLCPCB Part #" "C25804" (at 34.29 153.67 0)
+    (property "LCSC Part" "C25744" (at 34.29 153.67 0)
       (effects (font (size 1.27 1.27)) hide)
     )
@@
       (effects (font (size 1.27 1.27)) hide)
     )
+    (property "LCSC Part" "" (at 109.22 168.91 0)
+      (effects (font (size 1.27 1.27)) hide)
+    )
     (pin "1")
     (pin "2")
@@
       (effects (font (size 1.27 1.27)) hide)
     )
-    (property "JLCPCB Part #" "C25744" (at 200.66 39.37 0)
+    (property "LCSC Part" "C25744" (at 200.66 39.37 0)
       (effects (font (size 1.27 1.27)) hide)
     )
@@
       (effects (font (size 1.27 1.27)) hide)
     )
-    (property "JLCPCB Part #" "C23630" (at 248.92 30.48 0)
+    (property "LCSC Part" "C23630" (at 248.92 30.48 0)
       (effects (font (size 1.27 1.27)) hide)
     )
@@
       (effects (font (size 1.27 1.27)) hide)
     )
-    (property "JLCPCB Part #" "C25744" (at 168.91 39.37 0)
+    (property "LCSC Part" "C25744" (at 168.91 39.37 0)
       (effects (font (size 1.27 1.27)) hide)
     )
@@
       (effects (font (size 1.27 1.27)) hide)
     )
-    (property "JLCPCB Part #" "C23630" (at 266.7 29.21 0)
+    (property "LCSC Part" "C23630" (at 266.7 29.21 0)
       (effects (font (size 1.27 1.27)) hide)
     )
@@
       (effects (font (size 1.27 1.27)) hide)
     )
+    (property "LCSC Part" "" (at 146.05 168.91 0)
+      (effects (font (size 1.27 1.27)) hide)
+    )
     (pin "1")
     (pin "2")
@@
       (effects (font (size 1.27 1.27)) hide)
     )
+    (property "LCSC Part" "" (at 48.26 113.03 0)
+      (effects (font (size 1.27 1.27)) hide)
+    )
     (pin "1")
     (pin "2")
@@
       (effects (font (size 1.27 1.27)) hide)
     )
+    (property "LCSC Part" "C25804" (at 72.39 57.15 0)
+      (effects (font (size 1.27 1.27)) hide)
+    )
     (pin "1")
     (pin "2")
@@
       (effects (font (size 1.27 1.27)) hide)
     )
-    (property "JLCPCB Part #" "C15849" (at 44.45 172.72 0)
+    (property "LCSC Part" "C52923" (at 44.45 172.72 0)
       (effects (font (size 1.27 1.27)) hide)
     )
@@
       (effects (font (size 1.27 1.27)) hide)
     )
+    (property "LCSC Part" "" (at 106.68 114.3 0)
+      (effects (font (size 1.27 1.27)) hide)
+    )
     (pin "1")
     (pin "2")
@@
       (effects (font (size 1.27 1.27)) hide)
     )
-    (property "JLCPCB Part #" "C25804" (at 72.39 153.67 0)
-      (effects (font (size 1.27 1.27)) hide)
-    )
+    (property "LCSC Part" "C25744" (at 72.39 153.67 0)
+      (effects (font (size 1.27 1.27)) hide)
+    )

Commit message: Start on pcb
Parts:
- J2: footprint (none) -> Connector_PinHeader_2.54mm:PinHeader_1x02_P2.54mm_Vertical
- J7: footprint (none) -> Connector_JST:JST_PH_B2B-PH-K_1x02_P2.00mm_Vertical
Connections:
- net +3.1V_SW: no longer C22.1, FB1.2
- new net +3.3V: C22.1, FB1.2
Changed lines of the file:
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@@
   (junction (at 156.21 165.1) (diameter 0) (color 0 0 0 0)
   )
+  (junction (at 100.33 114.3) (diameter 0) (color 0 0 0 0)
+  )
   (junction (at 72.39 30.48) (diameter 0) (color 0 0 0 0)
   )
   (junction (at 226.06 68.58) (diameter 0) (color 0 0 0 0)
-  )
-  (junction (at 100.33 114.3) (diameter 0) (color 0 0 0 0)
   )
   (junction (at 248.92 24.13) (diameter 0) (color 0 0 0 0)
@@
     (stroke (width 0) (type default))
   )
-  (wire (pts (xy 95.25 114.3) (xy 100.33 114.3))
-    (stroke (width 0) (type default))
-  )
   (wire (pts (xy 226.06 116.84) (xy 226.06 68.58))
     (stroke (width 0) (type default))
@@
     (stroke (width 0) (type default))
   )
+  (wire (pts (xy 90.17 114.3) (xy 100.33 114.3))
+    (stroke (width 0) (type default))
+  )
   (wire (pts (xy 200.66 36.83) (xy 200.66 31.75))
     (stroke (width 0) (type default))
@@
     (stroke (width 0) (type default))
   )
-  (wire (pts (xy 95.25 113.03) (xy 95.25 114.3))
-    (stroke (width 0) (type default))
-  )
   (wire (pts (xy 59.69 49.53) (xy 54.61 49.53))
     (stroke (width 0) (type default))
@@
   )
   (wire (pts (xy 182.88 111.76) (xy 184.15 111.76))
+    (stroke (width 0) (type default))
+  )
+  (wire (pts (xy 90.17 113.03) (xy 90.17 114.3))
     (stroke (width 0) (type default))
   )
@@
         (path "/9d9a2a31-8397-4ba2-ad51-8bee2c0fd904/844bac58-4296-4d6f-b6fa-b18911d535fb"
           (reference "R26") (unit 1)
+        )
+      )
+    )
+  )
+  (symbol (lib_id "Main_LibraryVario:+3.1V_SW") (at 266.7 21.59 0) (unit 1)
+    (in_bom yes) (on_board yes) (dnp no) (fields_autoplaced)
+    (property "Reference" "#PWR055" (at 266.7 25.4 0)
+      (effects (font (size 1.27 1.27)) hide)
+    )
+    (property "Value" "+3.1V_SW" (at 266.7 17.78 0)
+      (effects (font (size 1.27 1.27)))
+    )
+    (property "Footprint" "" (at 266.7 21.59 0)
+      (effects (font (size 1.27 1.27)) hide)
+    )
+    (property "Datasheet" "" (at 266.7 21.59 0)
+      (effects (font (size 1.27 1.27)) hide)
+    )
+    (pin "1")
+    (instances
+      (project "VariometerV2.2.1"
+        (path "/9d9a2a31-8397-4ba2-ad51-8bee2c0fd904/844bac58-4296-4d6f-b6fa-b18911d535fb"
+          (reference "#PWR055") (unit 1)
         )
       )
@@
     )
   )
-  (symbol (lib_id "power:PWR_FLAG") (at 95.25 113.03 0) (unit 1)
-    (in_bom yes) (on_board yes) (dnp no)
-    (property "Reference" "#FLG01" (at 95.25 111.125 0)
-      (effects (font (size 1.27 1.27)) hide)
-    )
-    (property "Value" "PWR_FLAG" (at 88.9 110.49 0)
-      (effects (font (size 1.27 1.27)))
-    )
-    (property "Footprint" "" (at 95.25 113.03 0)
-      (effects (font (size 1.27 1.27)) hide)
-    )
-    (property "Datasheet" "~" (at 95.25 113.03 0)
-      (effects (font (size 1.27 1.27)) hide)
-    )
-    (pin "1")
-    (instances
-      (project "VariometerV2.2.1"
-        (path "/9d9a2a31-8397-4ba2-ad51-8bee2c0fd904/844bac58-4296-4d6f-b6fa-b18911d535fb"
-          (reference "#FLG01") (unit 1)
-        )
-      )
-      (project "VariometerV2.2"
-        (path "/e63e39d7-6ac0-4ffd-8aa3-1841a4541b55"
-          (reference "#FLG0101") (unit 1)
-        )
-      )
-    )
-  )
   (symbol (lib_id "Device:R_Small") (at 91.44 41.91 0) (unit 1)
     (in_bom yes) (on_board yes) (dnp no) (fields_autoplaced)
@@
     )
   )
+  (symbol (lib_id "power:PWR_FLAG") (at 90.17 113.03 0) (unit 1)
+    (in_bom yes) (on_board yes) (dnp no) (fields_autoplaced)
+    (property "Reference" "#FLG01" (at 90.17 111.125 0)
+      (effects (font (size 1.27 1.27)) hide)
+    )
+    (property "Value" "PWR_FLAG" (at 90.17 109.22 0)
+      (effects (font (size 1.27 1.27)))
+    )
+    (property "Footprint" "" (at 90.17 113.03 0)
+      (effects (font (size 1.27 1.27)) hide)
+    )
+    (property "Datasheet" "~" (at 90.17 113.03 0)
+      (effects (font (size 1.27 1.27)) hide)
+    )
+    (pin "1")
+    (instances
+      (project "VariometerV2.2.1"
+        (path "/9d9a2a31-8397-4ba2-ad51-8bee2c0fd904/844bac58-4296-4d6f-b6fa-b18911d535fb"
+          (reference "#FLG01") (unit 1)
+        )
+      )
+    )
+  )
   (symbol (lib_id "power:PWR_FLAG") (at 72.39 27.94 0) (unit 1)
     (in_bom yes) (on_board yes) (dnp no)
@@
     )
   )
-  (symbol (lib_id "VariometerV2:+3.1V_SW") (at 266.7 21.59 0) (unit 1)
-    (in_bom yes) (on_board yes) (dnp no)
-    (property "Reference" "#PWR055" (at 266.7 25.4 0)
-      (effects (font (size 1.27 1.27)) hide)
-    )
-    (property "Value" "+3.1V_SW" (at 266.7 17.78 0)
-      (effects (font (size 1.27 1.27)))
-    )
-    (property "Footprint" "" (at 266.7 21.59 0)
-      (effects (font (size 1.27 1.27)) hide)
-    )
-    (property "Datasheet" "" (at 266.7 21.59 0)
-      (effects (font (size 1.27 1.27)) hide)
-    )
-    (pin "1")
-    (instances
-      (project "VariometerV2.2.1"
-        (path "/9d9a2a31-8397-4ba2-ad51-8bee2c0fd904/844bac58-4296-4d6f-b6fa-b18911d535fb"
-          (reference "#PWR055") (unit 1)
-        )
-      )
-      (project "VariometerV2.2"
-        (path "/e63e39d7-6ac0-4ffd-8aa3-1841a4541b55"
-          (reference "#PWR0102") (unit 1)
-        )
-      )
-    )
-  )
   (symbol (lib_id "Device:R_Small") (at 168.91 39.37 0) (unit 1)
     (in_bom yes) (on_board yes) (dnp no)
@@
       (effects (font (size 1.27 1.27)) (justify left))
     )
-    (property "Footprint" "" (at 48.26 113.03 0)
+    (property "Footprint" "Connector_PinHeader_2.54mm:PinHeader_1x02_P2.54mm_Vertical" (at 48.26 113.03 0)
       (effects (font (size 1.27 1.27)) hide)
     )
@@
       (effects (font (size 1.27 1.27)) (justify left))
     )
-    (property "Footprint" "" (at 106.68 114.3 0)
-      (effects (font (size 1.27 1.27)) hide)
-    )
+    (property "Footprint" "Connector_JST:JST_PH_B2B-PH-K_1x02_P2.00mm_Vertical" (at 106.68 114.3 0)
+      (effects (font (size 1.27 1.27)) hide)
+    )

Commit message: Routing ..
Parts:
- J7: footprint Connector_JST:JST_PH_B2B-PH-K_1x02_P2.00mm_Vertical -> Connector_JST:JST_PH_S2B-PH-K_1x02_P2.00mm_Horizontal
Changed lines of the file:
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@@
       (effects (font (size 1.27 1.27)) (justify left))
     )
-    (property "Footprint" "Connector_JST:JST_PH_B2B-PH-K_1x02_P2.00mm_Vertical" (at 106.68 114.3 0)
+    (property "Footprint" "Connector_JST:JST_PH_S2B-PH-K_1x02_P2.00mm_Horizontal" (at 106.68 114.3 0)
       (effects (font (size 1.27 1.27)) hide)
     )
