File: Hardware/Version 2.1/VariometerV2.2.1/peripherals.kicad_sch (KiCad schematic)
At the start: 41 parts, among them J1 USB_C_Receptacle_USB2.0, J2 Conn_01x02, J7 Conn_01x02, SW3 BTN1, SW4 BTN1, SW5 BTN1, SW6 BTN1, U1 SRV05-4, U2 SRV05-4, U3 SRV05-4

Commit message: New 3D File
Parts:
- SW3, SW4, SW5, SW6: footprint Button_Switch_THT:SW_PUSH_6mm -> Button_Switch_THT:SW_PUSH_6mm_H4.3mm
Changed lines of the file:
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@@
       (effects (font (size 1.27 1.27)) (justify left))
     )
-    (property "Footprint" "Button_Switch_THT:SW_PUSH_6mm" (at 67.31 168.91 0)
+    (property "Footprint" "Button_Switch_THT:SW_PUSH_6mm_H4.3mm" (at 67.31 168.91 0)
       (effects (font (size 1.27 1.27)) hide)
     )
@@
       (effects (font (size 1.27 1.27)) (justify left))
     )
-    (property "Footprint" "Button_Switch_THT:SW_PUSH_6mm" (at 29.21 168.91 0)
+    (property "Footprint" "Button_Switch_THT:SW_PUSH_6mm_H4.3mm" (at 29.21 168.91 0)
       (effects (font (size 1.27 1.27)) hide)
     )
@@
       (effects (font (size 1.27 1.27)) (justify left))
     )
-    (property "Footprint" "Button_Switch_THT:SW_PUSH_6mm" (at 104.14 168.91 0)
+    (property "Footprint" "Button_Switch_THT:SW_PUSH_6mm_H4.3mm" (at 104.14 168.91 0)
       (effects (font (size 1.27 1.27)) hide)
     )
@@
       (effects (font (size 1.27 1.27)) (justify left))
     )
-    (property "Footprint" "Button_Switch_THT:SW_PUSH_6mm" (at 140.97 168.91 0)
-      (effects (font (size 1.27 1.27)) hide)
-    )
+    (property "Footprint" "Button_Switch_THT:SW_PUSH_6mm_H4.3mm" (at 140.97 168.91 0)
+      (effects (font (size 1.27 1.27)) hide)
+    )

Commit message: Finish PCB
Parts:
- J2, J3, J7, SW3, SW4, SW5, SW6, TP11, TP12: LCSC Part (none) -> 0
Changed lines of the file:
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@@
       (effects (font (size 1.27 1.27)) hide)
     )
-    (property "LCSC Part" "" (at 100.33 31.75 0)
+    (property "LCSC Part" "0" (at 100.33 31.75 0)
       (effects (font (size 1.27 1.27)) hide)
     )
@@
       (effects (font (size 1.27 1.27)) hide)
     )
-    (property "LCSC Part" "" (at 86.36 31.75 0)
+    (property "LCSC Part" "0" (at 86.36 31.75 0)
       (effects (font (size 1.27 1.27)) hide)
     )
@@
       (effects (font (size 1.27 1.27)) hide)
     )
-    (property "LCSC Part" "" (at 251.46 68.58 0)
+    (property "LCSC Part" "0" (at 251.46 68.58 0)
       (effects (font (size 1.27 1.27)) hide)
     )
@@
       (effects (font (size 1.27 1.27)) hide)
     )
-    (property "LCSC Part" "" (at 72.39 168.91 0)
+    (property "LCSC Part" "0" (at 72.39 168.91 0)
       (effects (font (size 1.27 1.27)) hide)
     )
@@
       (effects (font (size 1.27 1.27)) hide)
     )
-    (property "LCSC Part" "" (at 34.29 168.91 0)
+    (property "LCSC Part" "0" (at 34.29 168.91 0)
       (effects (font (size 1.27 1.27)) hide)
     )
@@
       (effects (font (size 1.27 1.27)) hide)
     )
-    (property "LCSC Part" "" (at 109.22 168.91 0)
+    (property "LCSC Part" "0" (at 109.22 168.91 0)
       (effects (font (size 1.27 1.27)) hide)
     )
@@
       (effects (font (size 1.27 1.27)) hide)
     )
-    (property "LCSC Part" "" (at 146.05 168.91 0)
+    (property "LCSC Part" "0" (at 146.05 168.91 0)
       (effects (font (size 1.27 1.27)) hide)
     )
@@
       (effects (font (size 1.27 1.27)) hide)
     )
-    (property "LCSC Part" "" (at 48.26 113.03 0)
+    (property "LCSC Part" "0" (at 48.26 113.03 0)
       (effects (font (size 1.27 1.27)) hide)
     )
@@
       (effects (font (size 1.27 1.27)) hide)
     )
-    (property "LCSC Part" "" (at 106.68 114.3 0)
-      (effects (font (size 1.27 1.27)) hide)
-    )
+    (property "LCSC Part" "0" (at 106.68 114.3 0)
+      (effects (font (size 1.27 1.27)) hide)
+    )
