File: Hardware/Version 2.1/VariometerV2.2.1/Power.kicad_sch (KiCad schematic)
At the start: 0 parts

Commit message: Working on PCB
Parts:
- added C10, C12: 2.2uF, symbol Device:C_Small
- added C11, C14: 10uF, symbol Device:C_Small
- added C13: 47nF, symbol Device:C_Small
- added C15, C16, C19: 1uF, Capacitor_SMD:C_0402_1005Metric, symbol Device:C_Small
- added C17: 100nF, Capacitor_SMD:C_0402_1005Metric, symbol Device:C_Small
- added C18: 10nF, Capacitor_SMD:C_0402_1005Metric, symbol Device:C_Small
- added D1: B5819W SL, Diode_SMD:D_SOD-123, symbol Device:D_Schottky_Small
- added D2: RED, LED_SMD:LED_0603_1608Metric, symbol Device:LED_Small
- added IC2: BQ25303JRTER, QFN50P300X300X80-17N-D, symbol Main_LibraryVario:BQ25303JRTER
- added IC4: TPS22916CNYFPR, SamacSys_Parts:BGA4C40P2X2_78X78X50, symbol VariometerV2:TPS22916CNYFPR
- added IC5: TPS73701DCQR, SamacSys_Parts:SOT127P706X180-6N, symbol VariometerV2:TPS73701DCQR
- added J8: LED_CHRG, Connector_PinHeader_2.00mm:PinHeader_2x01_P2.00mm_Vertical, symbol Connector_Generic:Conn_02x01
- added L1: 1uH PW, symbol Device:L_Small
- added Q1, Q2: AO3401A, Package_TO_SOT_SMD:SOT-23, symbol Transistor_FET:AO3401A
- added Q3: AO3400A, Package_TO_SOT_SMD:SOT-23, symbol Transistor_FET:AO3400A
- added R13: 43k, symbol Device:R_Small
- added R14: 1k, symbol Device:R_Small
- added R15, R16: 10k, symbol Device:R_Small
- added R17, R20: 10k, Resistor_SMD:R_0402_1005Metric, symbol Device:R_Small
- added R18: 33k, Resistor_SMD:R_0402_1005Metric, symbol Device:R_Small
- added R19: 1M, Resistor_SMD:R_0402_1005Metric, symbol Device:R_Small
- added R21: 47k, Resistor_SMD:R_0603_1608Metric, symbol Device:R_Small
- added R22: 20k, Resistor_SMD:R_0603_1608Metric, symbol Device:R_Small
- added R23: 9.1k, Resistor_SMD:R_0603_1608Metric, symbol Device:R_Small
- added R24: 1.5k, Resistor_SMD:R_0603_1608Metric, symbol Device:R_Small
- added TP1: TP_BATTERY, TestPoint:TestPoint_Pad_D1.5mm, symbol Connector:TestPoint
- added TP2: 3.1V TP, TestPoint:TestPoint_Pad_D1.5mm, symbol Connector:TestPoint
Connections:
- new net: D2.1 (K), R24.1
- new net: Q3.1 (G), R20.2
- new net: Q2.1 (G), Q3.3 (D), R19.1
- new net: C18.2, IC5.4 (FB), R21.2, R22.1
- new net: C13.1, IC2.13 (SW1), IC2.14 (SW2), L1.1
- new net: C13.2, IC2.15 (BTST)
- new net: C11.1, IC2.16 (PMID)
- new net: Q2.3 (D), R17.2
- new net: J8.2 (Pin_2), R14.1
- new net: R22.2, R23.1
- new net +3.1V_SW: C17.1, D2.2 (A), IC4.A1 (VOUT)
- new net +3.1V_UNSW: C15.1, C18.1, C19.1, IC4.A2 (VIN), IC5.2 (Vout), R21.1, TP2.1
- new net +5V: C10.1, D1.2 (A), IC2.1 (VBUS)
- new net +BATT: C14.1, IC2.10 (BAT), L1.2, Q1.3 (D), Q2.2 (S), R19.2
- new net BAT_ADC: R17.1, R18.2, TP1.1
- new net BAT_MS: R20.1
- new net CHRG_STAT: IC2.3 (STAT), R14.2
- new net GND: C10.2, C11.2, C12.2, C14.2, C15.2, C16.2, C17.2, C19.2, IC2.11 (GND), IC2.12 (GND), IC2.17 (EP), IC2.9 (VSET), IC4.B1 (GND), IC5.3 (GND_1), IC5.6 (GND_2), Q1.1 (G), Q3.2 (S), R13.2, R16.1, R18.1, R23.2, R24.2
- new net ICHG: IC2.4 (ICHG), R13.1
- new net POSW_EN: IC4.B2 (ON)
- new net REGN: C12.1, IC2.2 (REGN), J8.1 (Pin_1), R15.2
- new net TS: IC2.7 (TS), R15.1, R16.2
- new net VCC: C16.1, D1.1 (K), IC5.1 (Vin), IC5.5 (EN), Q1.2 (S)
- no-connect marks 0 -> 3
Other:
- note added: "Battery Charger"
- note added: "Battery Voltage Measure"
- note added: "CHANGE!!!"
- note added: "Charge LED"
- note added: "End Voltage 4.1V"
- note added: "I(A) = 40000 / R = 0.93A"
- note added: "LDO (3.1V OUTPUT)"
- note added: "LOAD SWITCH FÜR ALLE SENSOREN"
- note added: "Power LED"
- note added: "REVERSE POLARITY PROTECTION"
- note added: "Vout = (R1+R2)/R2 * 1.204"

Commit message: Weiter PCB
Other:
- note added: "USE bq24196 ??"
Changed lines of the file:
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@@
     (effects (font (size 1.27 1.27)) (justify left bottom))
+  )
+  (text "USE bq24196 ??" (at 97.79 25.4 0)
+    (effects (font (size 3 3)) (justify left bottom))
   )
   (text "Vout = (R1+R2)/R2 * 1.204" (at 234.95 114.3 0)

Commit message: Update Schematics
Parts:
- removed IC2: BQ25303JRTER, QFN50P300X300X80-17N-D, symbol Main_LibraryVario:BQ25303JRTER
- added C44, C45: 10uF, Capacitor_SMD:C_0603_1608Metric, symbol Device:C_Small
- added C46: 4.7Uf, Capacitor_SMD:C_0603_1608Metric, symbol Device:C_Small
- added D6: B5819W SL, Diode_SMD:D_SOD-123, symbol Device:D_Schottky_Small
- added IC2: BQ24196RGER, MainLibrary:QFN50P400X400X100-25N-D, symbol Main_LibraryVario:BQ24196RGER
- added J11: LED_CHRG, Connector_PinHeader_2.54mm:PinHeader_2x01_P2.54mm_Vertical, symbol Connector_Generic:Conn_02x01
- added JP2, JP4: JMP, Jumper:SolderJumper-2_P1.3mm_Open_Pad1.0x1.5mm, symbol Jumper:SolderJumper_2_Open
- added JP3: SJMP, Jumper:SolderJumper-3_P1.3mm_Bridged12_Pad1.0x1.5mm_NumberLabels, symbol Jumper:SolderJumper_3_Bridged12
- added R42, R43: 10k, symbol Device:R_Small
- added TP10: TP_SYS_LOAD, symbol Connector:TestPoint
- C10: value 2.2uF -> 6.8uF; footprint (none) -> Capacitor_SMD:C_0603_1608Metric; JLCPCB Part # (none) -> C52923; LCSC Part # (none) -> C2345
- C11: value 10uF -> 1uF; footprint (none) -> Capacitor_SMD:C_0402_1005Metric; JLCPCB Part # (none) -> C52923; LCSC Part # (none) -> C2345
- C12: value 2.2uF -> 47nF; footprint (none) -> Capacitor_SMD:C_0603_1608Metric; JLCPCB Part # (none) -> C52923; LCSC Part # (none) -> C2345
- C13: value 47nF -> 10uF; footprint (none) -> Capacitor_SMD:C_0603_1608Metric; JLCPCB Part # (none) -> C52923; LCSC Part # (none) -> C2345
- C14: footprint (none) -> Capacitor_SMD:C_0603_1608Metric; JLCPCB Part # (none) -> C52923; LCSC Part # (none) -> C2345
- IC4: footprint SamacSys_Parts:BGA4C40P2X2_78X78X50 -> MainLibrary:BGA4C40P2X2_78X78X50
- IC5: footprint SamacSys_Parts:SOT127P706X180-6N -> MainLibrary:SOT127P706X180-6N
- J8: footprint Connector_PinHeader_2.00mm:PinHeader_2x01_P2.00mm_Vertical -> Connector_PinHeader_2.54mm:PinHeader_2x01_P2.54mm_Vertical
- L1: value 1uH PW -> 1uH P
- Q1, Q2, Q3: footprint Package_TO_SOT_SMD:SOT-23 -> (none)
- R13: value 43k -> 1k; JLCPCB Part # (none) -> C21190
- R14: JLCPCB Part # (none) -> C21190
- R15: JLCPCB Part # (none) -> C25819
- R16: value 10k -> 360R
- R17, R18, R19, R20: footprint Resistor_SMD:R_0402_1005Metric -> (none)
- R21, R22, R23, R24: footprint Resistor_SMD:R_0603_1608Metric -> (none)
- TP1, TP2: footprint TestPoint:TestPoint_Pad_D1.5mm -> (none)
Connections:
- net ICHG is gone; now on an unnamed net: R13.1
- net +3.1V_UNSW: now also R15.1
- net +5V: now also C11.1, IC2.1 (VBUS1), IC2.24 (VBUS2), JP2.2 (B), JP3.3 (B); no longer C10.1, D1.2 (A)
- net +BATT: now also C13.1, IC2.13 (BAT1), IC2.14 (BAT2), JP4.2 (B); no longer C14.1, L1.2, Q1.3 (D)
- net GND: now also C13.2, R16.2, C44.2, C45.2, C46.2, IC2.17 (PGND), IC2.18 (PGND), IC2.25 (EP), IC2.9 (~{CE}), JP3.1 (A), R43.2; no longer C12.2, R13.2, R16.1
- net REGN: now also C46.1, IC2.22 (REGN), R42.1; no longer C12.1, J8.1 (Pin_1), R15.2
- net TS: now also IC2.11 (TS1), IC2.12 (TS2), R42.2, R43.1; no longer R15.1, R16.2
- net VCC: now also D6.1 (K)
- net at L1.1: now also C12.1, IC2.19 (SW1), IC2.20 (SW2); no longer C13.1
- net at J8.2 (Pin_2): no longer R14.1
- net CHRG_STAT renamed ~{PG}
- net ~{PG}: now also IC2.3 (~{PG})
- new net: D1.2 (A), JP2.1 (A)
- new net: J11.2 (Pin_2), R14.1
- new net: IC2.2 (PSEL), IC2.8 (OTG), JP3.2 (C)
- new net: IC2.10 (ILIM), R16.1
- new net: D6.2 (A), JP4.1 (A)
- new net: C10.1, IC2.23 (PMID)
- new net: C12.2, IC2.21 (BTST)
- new net CHARG_INT: IC2.7 (INT), R15.2
- new net I2C2_SCL: IC2.5 (SCL)
- new net I2C2_SDA: IC2.6 (SDA)
- new net STAT: IC2.4 (STAT), R13.2
- new net SYS: C14.1, C44.1, C45.1, IC2.15 (SYS1), IC2.16 (SYS2), J11.1 (Pin_1), J8.1 (Pin_1), L1.2, Q1.3 (D), TP10.1
- no-connect marks 3 -> 0
Other:
- note added: "CHARGE LED"
- note added: "GND: Custom power Source with custom Input current 5V: USB Power with 500mA"
- note added: "Imax = 1V/R * 530 1.47A"
- note added: "POWER GOOD LED"
- note removed: "Battery Charger"
- note removed: "Charge LED"
- note removed: "End Voltage 4.1V"
- note removed: "I(A) = 40000 / R = 0.93A"
- note removed: "USE bq24196 ??"
- moved on the sheet: C15, C17, D1, IC4, Q1, Q2, Q3, R17, R18, R19, R20, TP1

Commit message: Working on PCB
Parts:
- Q1, Q2, Q3: footprint (none) -> Package_TO_SOT_SMD:SOT-23
- R13, R14, R15, R16, R21, R22, R23, R24, R42, R43: footprint (none) -> Resistor_SMD:R_0603_1608Metric
- R17, R18, R19, R20: footprint (none) -> Resistor_SMD:R_0402_1005Metric
- TP1, TP10, TP2: footprint (none) -> TestPoint:TestPoint_Pad_D1.5mm
Changed lines of the file:
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@@
       (effects (font (size 1.27 1.27)) (justify left))
     )
-    (property "Footprint" "" (at 49.53 175.895 0)
+    (property "Footprint" "Package_TO_SOT_SMD:SOT-23" (at 49.53 175.895 0)
       (effects (font (size 1.27 1.27) italic) (justify left) hide)
     )
@@
       (effects (font (size 1.27 1.27)))
     )
-    (property "Footprint" "" (at 62.23 173.99 0)
+    (property "Footprint" "Resistor_SMD:R_0402_1005Metric" (at 62.23 173.99 0)
       (effects (font (size 1.27 1.27)) hide)
     )
@@
       (effects (font (size 1.27 1.27)) (justify left))
     )
-    (property "Footprint" "" (at 80.01 71.12 0)
+    (property "Footprint" "Resistor_SMD:R_0603_1608Metric" (at 80.01 71.12 0)
       (effects (font (size 1.27 1.27)) hide)
     )
@@
       (effects (font (size 1.27 1.27)))
     )
-    (property "Footprint" "" (at 41.91 168.91 0)
+    (property "Footprint" "Resistor_SMD:R_0402_1005Metric" (at 41.91 168.91 0)
       (effects (font (size 1.27 1.27)) hide)
     )
@@
       (effects (font (size 1.27 1.27)) (justify right))
     )
-    (property "Footprint" "" (at 209.55 149.86 0)
+    (property "Footprint" "TestPoint:TestPoint_Pad_D1.5mm" (at 209.55 149.86 0)
       (effects (font (size 1.27 1.27)) hide)
     )
@@
       (effects (font (size 1.27 1.27)) (justify left))
     )
-    (property "Footprint" "" (at 26.67 106.68 0)
+    (property "Footprint" "Resistor_SMD:R_0603_1608Metric" (at 26.67 106.68 0)
       (effects (font (size 1.27 1.27)) hide)
     )
@@
       (effects (font (size 1.27 1.27)) (justify right))
     )
-    (property "Footprint" "" (at 45.72 72.39 0)
+    (property "Footprint" "Resistor_SMD:R_0603_1608Metric" (at 45.72 72.39 0)
       (effects (font (size 1.27 1.27)) hide)
     )
@@
       (effects (font (size 1.27 1.27)) (justify left))
     )
-    (property "Footprint" "" (at 241.3 102.87 0)
+    (property "Footprint" "Resistor_SMD:R_0603_1608Metric" (at 241.3 102.87 0)
       (effects (font (size 1.27 1.27)) hide)
     )
@@
       (effects (font (size 1.27 1.27)))
     )
-    (property "Footprint" "" (at 41.91 177.8 0)
+    (property "Footprint" "Resistor_SMD:R_0402_1005Metric" (at 41.91 177.8 0)
       (effects (font (size 1.27 1.27)) hide)
     )
@@
       (effects (font (size 1.27 1.27)) (justify left))
     )
-    (property "Footprint" "" (at 26.67 116.84 0)
+    (property "Footprint" "Resistor_SMD:R_0603_1608Metric" (at 26.67 116.84 0)
       (effects (font (size 1.27 1.27)) hide)
     )
@@
       (effects (font (size 1.27 1.27)) (justify right))
     )
-    (property "Footprint" "" (at 45.72 53.34 0)
+    (property "Footprint" "Resistor_SMD:R_0603_1608Metric" (at 45.72 53.34 0)
       (effects (font (size 1.27 1.27)) hide)
     )
@@
       (effects (font (size 1.27 1.27)))
     )
-    (property "Footprint" "" (at 152.4 87.63 0)
+    (property "Footprint" "Resistor_SMD:R_0603_1608Metric" (at 152.4 87.63 0)
       (effects (font (size 1.27 1.27)) hide)
     )
@@
       (effects (font (size 1.27 1.27)) (justify left))
     )
-    (property "Footprint" "" (at 241.3 109.22 0)
+    (property "Footprint" "Resistor_SMD:R_0603_1608Metric" (at 241.3 109.22 0)
       (effects (font (size 1.27 1.27)) hide)
     )
@@
       (effects (font (size 1.27 1.27)) (justify left))
     )
-    (property "Footprint" "" (at 39.37 156.845 0)
+    (property "Footprint" "Package_TO_SOT_SMD:SOT-23" (at 39.37 156.845 0)
       (effects (font (size 1.27 1.27) italic) (justify left) hide)
     )
@@
       (effects (font (size 1.27 1.27)) (justify right))
     )
-    (property "Footprint" "" (at 22.86 179.07 0)
+    (property "Footprint" "TestPoint:TestPoint_Pad_D1.5mm" (at 22.86 179.07 0)
       (effects (font (size 1.27 1.27)) hide)
     )
@@
       (effects (font (size 1.27 1.27)) (justify left))
     )
-    (property "Footprint" "" (at 240.03 147.32 0)
+    (property "Footprint" "Resistor_SMD:R_0603_1608Metric" (at 240.03 147.32 0)
       (effects (font (size 1.27 1.27)) hide)
     )
@@
       (effects (font (size 1.27 1.27)) (justify left))
     )
-    (property "Footprint" "" (at 241.3 96.52 0)
+    (property "Footprint" "Resistor_SMD:R_0603_1608Metric" (at 241.3 96.52 0)
       (effects (font (size 1.27 1.27)) hide)
     )
@@
       (effects (font (size 1.27 1.27)))
     )
-    (property "Footprint" "" (at 230.505 43.18 0)
+    (property "Footprint" "Package_TO_SOT_SMD:SOT-23" (at 230.505 43.18 0)
       (effects (font (size 1.27 1.27) italic) (justify left) hide)
     )
@@
       (effects (font (size 1.27 1.27)) (justify left))
     )
-    (property "Footprint" "" (at 201.93 31.75 0)
+    (property "Footprint" "TestPoint:TestPoint_Pad_D1.5mm" (at 201.93 31.75 0)
       (effects (font (size 1.27 1.27)) hide)
     )
@@
       (effects (font (size 1.27 1.27)))
     )
-    (property "Footprint" "" (at 52.07 153.67 0)
-      (effects (font (size 1.27 1.27)) hide)
-    )
+    (property "Footprint" "Resistor_SMD:R_0402_1005Metric" (at 52.07 153.67 0)
+      (effects (font (size 1.27 1.27)) hide)
+    )

Commit message: PCB
Parts:
- C10: footprint Capacitor_SMD:C_0603_1608Metric -> Capacitor_SMD:C_0805_2012Metric; JLCPCB Part # C52923 -> (none); LCSC Part # C2345 -> (none)
- C11, C15, C16, C19: JLCPCB Part # C52923 -> (none); LCSC Part (none) -> C52923; LCSC Part # C2345 -> (none)
- C12: JLCPCB Part # C52923 -> (none); LCSC Part (none) -> C1622; LCSC Part # C2345 -> (none)
- C13, C14, C44, C45: JLCPCB Part # C52923 -> (none); LCSC Part (none) -> C19702; LCSC Part # C2345 -> (none)
- C17: JLCPCB Part # C307331 -> (none); LCSC Part (none) -> C307331
- C18: JLCPCB Part # C15195 -> (none); LCSC Part (none) -> C15195
- C46: value 4.7Uf -> 4.7uF; JLCPCB Part # C52923 -> (none); LCSC Part (none) -> C19666; LCSC Part # C2345 -> (none)
- D1, D6: JLCPCB Part # C8598 -> (none); LCSC Part (none) -> C8598
- D2: JLCPCB Part # C2286 -> (none); LCSC Part (none) -> C2286
- IC2: LCSC Part (none) -> C117006; Mouser Part Number 595-BQ24196RGER -> (none); Mouser Price/Stock https://www.mouser.co.uk/ProductDetail/Texas-Instruments/BQ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 -> (none)
- IC4: JLCPCB Part # C2655476 -> (none); LCSC Part (none) -> C2655476
- IC5: JLCPCB Part # C56848 -> (none); LCSC Part (none) -> C56848
- L1: footprint (none) -> Inductor_SMD:L_0603_1608Metric
- Q1, Q2: JLCPCB Part # C15127 -> (none); LCSC Part (none) -> C15127
- Q3: JLCPCB Part # C20917 -> (none); LCSC Part (none) -> C20917
- R13, R14: JLCPCB Part # C21190 -> (none); LCSC Part (none) -> C21190
- R15, R42, R43: JLCPCB Part # C25819 -> (none); LCSC Part (none) -> C25804
- R16: LCSC Part (none) -> C25194
- R17, R20: JLCPCB Part # C25744 -> (none); LCSC Part (none) -> C25744
- R18: JLCPCB Part # C25779 -> (none); LCSC Part (none) -> C25779
- R19: JLCPCB Part # C26083 -> (none); LCSC Part (none) -> C26083
- R21: JLCPCB Part # C25819 -> (none); LCSC Part (none) -> C25819
- R22: JLCPCB Part # C4184 -> (none); LCSC Part (none) -> C4184
- R23: JLCPCB Part # C23260 -> (none); LCSC Part (none) -> C23260
- R24: JLCPCB Part # C22843 -> (none); LCSC Part (none) -> C22843

Commit message: Start on pcb
Parts:
- removed IC2: BQ24196RGER, MainLibrary:QFN50P400X400X100-25N-D, symbol Main_LibraryVario:BQ24196RGER
- removed JP3: SJMP, Jumper:SolderJumper-3_P1.3mm_Bridged12_Pad1.0x1.5mm_NumberLabels, symbol Jumper:SolderJumper_3_Bridged12
- added IC3: BQ24196RGER, MainLibrary:QFN50P400X400X100-25N-D, symbol Main_LibraryVario:BQ24196RGER
- added JP8: SJMP, Jumper:SolderJumper-3_P1.3mm_Open_Pad1.0x1.5mm, symbol Jumper:SolderJumper_3_Open
- R17: footprint Resistor_SMD:R_0402_1005Metric -> Resistor_SMD:R_0805_2012Metric
- R18: value 33k -> 15k; footprint Resistor_SMD:R_0402_1005Metric -> Resistor_SMD:R_0805_2012Metric; LCSC Part C25779 -> C22809
Connections:
- net +5V: now also IC3.1 (VBUS1), IC3.24 (VBUS2), JP8.3 (B)
- net +BATT: now also IC3.13 (BAT1), IC3.14 (BAT2)
- net CHARG_INT: now also IC3.7 (INT)
- net GND: now also IC3.17 (PGND), IC3.18 (PGND), IC3.25 (EP), IC3.9 (~{CE}), JP8.1 (A)
- net I2C2_SCL: now also IC3.5 (SCL)
- net I2C2_SDA: now also IC3.6 (SDA)
- net REGN: now also IC3.22 (REGN)
- net STAT: now also IC3.4 (STAT)
- net SYS: now also IC3.15 (SYS1), IC3.16 (SYS2)
- net TS: now also IC3.11 (TS1), IC3.12 (TS2)
- net ~{PG}: now also IC3.3 (~{PG})
- net at R16.1: now also IC3.10 (ILIM)
- net at C10.1: now also IC3.23 (PMID)
- net at C12.1, L1.1: now also IC3.19 (SW1), IC3.20 (SW2)
- net at C12.2: now also IC3.21 (BTST)
- new net: IC3.2 (PSEL), IC3.8 (OTG), JP8.2 (C)
Other:
- note added: "4.4V -> 2.64V"
- note removed: "CHANGE!!!"
- moved on the sheet: C15, C17, IC4, Q2, Q3, R17, R18, R19, R20, TP1
