File: Hardware/Version 2.1/VariometerV2.2.1/Power.kicad_sch (KiCad schematic)
At the start: 45 parts, among them IC3 BQ24196RGER, IC4 TPS22916CNYFPR, IC5 TPS73701DCQR, J11 LED_CHRG, J8 LED_CHRG, Q1 AO3401A, Q2 AO3401A, Q3 AO3400A

Commit message: PCb Layout done
Parts:
- removed J11: LED_CHRG, Connector_PinHeader_2.54mm:PinHeader_2x01_P2.54mm_Vertical, symbol Connector_Generic:Conn_02x01
- removed R14: 1k, Resistor_SMD:R_0603_1608Metric, symbol Device:R_Small
- added C51: 1uF, Capacitor_SMD:C_0603_1608Metric, symbol Device:C_Small
Connections:
- net BAT_ADC: now also C51.1
- net GND: now also C51.2
- net ~{PG}: no longer names the net of IC3.3 (~{PG})
- no-connect marks 0 -> 1
Other:
- note removed: "POWER GOOD LED"
Changed lines of the file:
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@@
   (junction (at 241.3 93.98) (diameter 0) (color 0 0 0 0)
   )
+  (junction (at 26.67 171.45) (diameter 0) (color 0 0 0 0)
+  )
   (junction (at 127 115.57) (diameter 0) (color 0 0 0 0)
   )
@@
   (junction (at 148.59 77.47) (diameter 0) (color 0 0 0 0)
   )
+  (no_connect (at 105.41 54.61))
   (wire (pts (xy 152.4 50.8) (xy 152.4 52.07))
     (stroke (width 0) (type default))
@@
     (stroke (width 0) (type default))
   )
-  (wire (pts (xy 48.26 53.34) (xy 54.61 53.34))
+  (wire (pts (xy 26.67 177.8) (xy 26.67 179.07))
     (stroke (width 0) (type default))
   )
@@
     (stroke (width 0) (type default))
   )
+  (wire (pts (xy 26.67 171.45) (xy 52.07 171.45))
+    (stroke (width 0) (type default))
+  )
   (wire (pts (xy 241.3 99.06) (xy 255.27 99.06))
     (stroke (width 0) (type default))
@@
     (stroke (width 0) (type default))
   )
+  (wire (pts (xy 26.67 171.45) (xy 26.67 172.72))
+    (stroke (width 0) (type default))
+  )
   (wire (pts (xy 152.4 35.56) (xy 156.21 35.56))
     (stroke (width 0) (type default))
@@
     (stroke (width 0) (type default))
   )
-  (wire (pts (xy 24.13 49.53) (xy 24.13 53.34))
-    (stroke (width 0) (type default))
-  )
   (wire (pts (xy 214.63 93.98) (xy 217.17 93.98))
     (stroke (width 0) (type default))
@@
     (stroke (width 0) (type default))
   )
-  (wire (pts (xy 101.6 54.61) (xy 105.41 54.61))
-    (stroke (width 0) (type default))
-  )
   (wire (pts (xy 52.07 149.86) (xy 62.23 149.86))
     (stroke (width 0) (type default))
@@
     (stroke (width 0) (type default))
   )
-  (wire (pts (xy 24.13 53.34) (xy 30.48 53.34))
-    (stroke (width 0) (type default))
-  )
   (wire (pts (xy 106.68 101.6) (xy 95.25 101.6))
     (stroke (width 0) (type default))
@@
     (stroke (width 0) (type default))
   )
-  (wire (pts (xy 48.26 171.45) (xy 52.07 171.45))
+  (wire (pts (xy 24.13 171.45) (xy 26.67 171.45))
     (stroke (width 0) (type default))
   )
@@
     (stroke (width 0) (type default))
   )
-  (text "4.4V -> 2.64V" (at 31.75 167.64 0)
+  (text "4.4V -> 2.64V" (at 15.24 158.75 0)
     (effects (font (size 1.27 1.27)) (justify left bottom))
   )
@@
   )
   (text "Power LED" (at 236.22 158.75 0)
-    (effects (font (size 1.27 1.27)) (justify left bottom))
-  )
-  (text "POWER GOOD LED" (at 33.02 57.15 0)
     (effects (font (size 1.27 1.27)) (justify left bottom))
   )
@@
     (effects (font (size 1.27 1.27)) (justify left bottom))
   )
-  (label "SYS" (at 24.13 49.53 0) (fields_autoplaced)
-    (effects (font (size 1.27 1.27)) (justify left bottom))
-  )
   (label "REGN" (at 152.4 50.8 180) (fields_autoplaced)
     (effects (font (size 1.27 1.27)) (justify right bottom))
@@
     (effects (font (size 1.27 1.27)) (justify right bottom))
   )
-  (label "~{PG}" (at 54.61 53.34 180) (fields_autoplaced)
-    (effects (font (size 1.27 1.27)) (justify right bottom))
-  )
   (label "SYS_LOAD" (at 210.82 45.72 0) (fields_autoplaced)
     (effects (font (size 1.27 1.27)) (justify left bottom))
@@
   (label "SYS_LOAD" (at 210.82 35.56 180) (fields_autoplaced)
     (effects (font (size 1.27 1.27)) (justify right bottom))
-  )
-  (label "~{PG}" (at 101.6 54.61 0) (fields_autoplaced)
-    (effects (font (size 1.27 1.27)) (justify left bottom))
   )
   (global_label "I2C2_SCL" (shape input) (at 100.33 74.93 180) (fields_autoplaced)
@@
     )
   )
-  (global_label "BAT_ADC" (shape input) (at 48.26 171.45 180) (fields_autoplaced)
+  (global_label "BAT_ADC" (shape input) (at 24.13 171.45 180) (fields_autoplaced)
     (effects (font (size 1.27 1.27)) (justify right))
-    (property "Intersheetrefs" "${INTERSHEET_REFS}" (at 37.9245 171.3706 0)
+    (property "Intersheetrefs" "${INTERSHEET_REFS}" (at 13.7945 171.3706 0)
       (effects (font (size 1.27 1.27)) (justify right) hide)
     )
@@
     )
   )
+  (symbol (lib_id "Device:C_Small") (at 26.67 175.26 0) (unit 1)
+    (in_bom yes) (on_board yes) (dnp no)
+    (property "Reference" "C51" (at 29.0068 174.0916 0)
+      (effects (font (size 1.27 1.27)) (justify left))
+    )
+    (property "Value" "1uF" (at 29.0068 176.403 0)
+      (effects (font (size 1.27 1.27)) (justify left))
+    )
+    (property "Footprint" "Capacitor_SMD:C_0603_1608Metric" (at 26.67 175.26 0)
+      (effects (font (size 1.27 1.27)) hide)
+    )
+    (property "Datasheet" "~" (at 26.67 175.26 0)
+      (effects (font (size 1.27 1.27)) hide)
+    )
+    (property "LCSC Part" "C52923" (at 26.67 175.26 0)
+      (effects (font (size 1.27 1.27)) hide)
+    )
+    (pin "1")
+    (pin "2")
+    (instances
+      (project "VariometerV2.2.1"
+        (path "/9d9a2a31-8397-4ba2-ad51-8bee2c0fd904/6f171705-fa97-4c0f-bbde-f97e718855cc"
+          (reference "C51") (unit 1)
+        )
+      )
+      (project "VariometerV2.2"
+        (path "/e63e39d7-6ac0-4ffd-8aa3-1841a4541b55"
+          (reference "C6") (unit 1)
+        )
+      )
+    )
+  )
   (symbol (lib_id "power:VCC") (at 201.93 93.98 0) (unit 1)
     (in_bom yes) (on_board yes) (dnp no) (fields_autoplaced)
@@
     )
   )
-  (symbol (lib_id "Connector_Generic:Conn_02x01") (at 35.56 53.34 0) (unit 1)
-    (in_bom yes) (on_board yes) (dnp no)
-    (property "Reference" "J11" (at 36.83 47.8282 0)
-      (effects (font (size 1.27 1.27)))
-    )
-    (property "Value" "LED_CHRG" (at 36.83 50.1396 0)
-      (effects (font (size 1.27 1.27)))
-    )
-    (property "Footprint" "Connector_PinHeader_2.54mm:PinHeader_2x01_P2.54mm_Vertical" (at 35.56 53.34 0)
-      (effects (font (size 1.27 1.27)) hide)
-    )
-    (property "Datasheet" "~" (at 35.56 53.34 0)
-      (effects (font (size 1.27 1.27)) hide)
-    )
-    (property "LCSC Part" "" (at 35.56 53.34 0)
-      (effects (font (size 1.27 1.27)) hide)
-    )
-    (pin "1")
-    (pin "2")
-    (instances
-      (project "VariometerV2.2.1"
-        (path "/9d9a2a31-8397-4ba2-ad51-8bee2c0fd904/6f171705-fa97-4c0f-bbde-f97e718855cc"
-          (reference "J11") (unit 1)
-        )
-      )
-      (project "VariometerV2.2"
-        (path "/e63e39d7-6ac0-4ffd-8aa3-1841a4541b55"
-          (reference "J1") (unit 1)
-        )
-      )
-    )
-  )
   (symbol (lib_id "Device:R_Small") (at 52.07 176.53 180) (unit 1)
     (in_bom yes) (on_board yes) (dnp no)
@@
     )
   )
-  (symbol (lib_id "Device:R_Small") (at 45.72 53.34 90) (unit 1)
-    (in_bom yes) (on_board yes) (dnp no)
-    (property "Reference" "R14" (at 44.45 48.26 90)
-      (effects (font (size 1.27 1.27)) (justify right))
-    )
-    (property "Value" "1k" (at 44.45 50.8 90)
-      (effects (font (size 1.27 1.27)) (justify right))
-    )
-    (property "Footprint" "Resistor_SMD:R_0603_1608Metric" (at 45.72 53.34 0)
-      (effects (font (size 1.27 1.27)) hide)
-    )
-    (property "Datasheet" "~" (at 45.72 53.34 0)
-      (effects (font (size 1.27 1.27)) hide)
-    )
-    (property "LCSC Part" "C21190" (at 45.72 53.34 0)
-      (effects (font (size 1.27 1.27)) hide)
-    )
-    (pin "1")
-    (pin "2")
-    (instances
-      (project "VariometerV2.2.1"
-        (path "/9d9a2a31-8397-4ba2-ad51-8bee2c0fd904/6f171705-fa97-4c0f-bbde-f97e718855cc"
-          (reference "R14") (unit 1)
-        )
-      )
-      (project "VariometerV2.2"
-        (path "/e63e39d7-6ac0-4ffd-8aa3-1841a4541b55"
-          (reference "R2") (unit 1)
-        )
-      )
-    )
-  )
   (symbol (lib_id "Device:C_Small") (at 170.18 39.37 0) (unit 1)
     (in_bom yes) (on_board yes) (dnp no)
@@
   (symbol (lib_name "BQ24196RGER_1") (lib_id "Main_LibraryVario:BQ24196RGER") (at 135.89 63.5 0) (unit 1)
     (in_bom yes) (on_board yes) (dnp no) (fields_autoplaced)
-    (property "Reference" "IC3" (at 125.73 26.67 0)
-      (effects (font (size 1.27 1.27)))
-    )
-    (property "Value" "BQ24196RGER" (at 125.73 29.21 0)
+    (property "Reference" "IC3" (at 125.73 25.4 0)
+      (effects (font (size 1.27 1.27)))
+    )
+    (property "Value" "BQ24196RGER" (at 125.73 27.94 0)
       (effects (font (size 1.27 1.27)))
     )
@@
         )
       )
+    )
+  )
+  (symbol (lib_id "power:GND") (at 26.67 179.07 0) (unit 1)
+    (in_bom yes) (on_board yes) (dnp no)
+    (property "Reference" "#PWR0110" (at 26.67 185.42 0)
+      (effects (font (size 1.27 1.27)) hide)
+    )
+    (property "Value" "GND" (at 26.797 183.4642 0)
+      (effects (font (size 1.27 1.27)))
+    )
+    (property "Footprint" "" (at 26.67 179.07 0)
+      (effects (font (size 1.27 1.27)) hide)
+    )
+    (property "Datasheet" "" (at 26.67 179.07 0)
+      (effects (font (size 1.27 1.27)) hide)
+    )
+    (pin "1")
+    (instances
+      (project "VariometerV2.2.1"
+        (path "/9d9a2a31-8397-4ba2-ad51-8bee2c0fd904/6f171705-fa97-4c0f-bbde-f97e718855cc"
+          (reference "#PWR0110") (unit 1)
+        )
+      )
+      (project "VariometerV2.2"
+        (path "/e63e39d7-6ac0-4ffd-8aa3-1841a4541b55"
+          (reference "#PWR0146") (unit 1)
+        )
+      )

Commit message: Finish PCB
Parts:
- C10, J8, JP2, JP4, JP8, L1, TP1, TP10, TP2: LCSC Part (none) -> 0
- C51: LCSC Part C52923 -> C15849
- IC3: LCSC Part (none) -> C117006
- R17: footprint Resistor_SMD:R_0805_2012Metric -> Resistor_SMD:R_0603_1608Metric; LCSC Part C25744 -> C25804
- R18: footprint Resistor_SMD:R_0805_2012Metric -> Resistor_SMD:R_0603_1608Metric
Changed lines of the file:
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@@
       (effects (font (size 1.27 1.27)) hide)
     )
-    (property "LCSC Part" "" (at 35.56 72.39 0)
+    (property "LCSC Part" "0" (at 35.56 72.39 0)
       (effects (font (size 1.27 1.27)) hide)
     )
@@
       (effects (font (size 1.27 1.27)))
     )
-    (property "Footprint" "Resistor_SMD:R_0805_2012Metric" (at 52.07 167.64 0)
+    (property "Footprint" "Resistor_SMD:R_0603_1608Metric" (at 52.07 167.64 0)
       (effects (font (size 1.27 1.27)) hide)
     )
@@
       (effects (font (size 1.27 1.27)) hide)
     )
-    (property "LCSC Part" "C25744" (at 52.07 167.64 0)
+    (property "LCSC Part" "C25804" (at 52.07 167.64 0)
       (effects (font (size 1.27 1.27)) hide)
     )
@@
       (effects (font (size 1.27 1.27)) hide)
     )
-    (property "LCSC Part" "" (at 214.63 149.86 0)
+    (property "LCSC Part" "0" (at 214.63 149.86 0)
       (effects (font (size 1.27 1.27)) hide)
     )
@@
       (effects (font (size 1.27 1.27)) hide)
     )
-    (property "LCSC Part" "" (at 238.76 31.75 0)
+    (property "LCSC Part" "0" (at 238.76 31.75 0)
       (effects (font (size 1.27 1.27)) hide)
     )
@@
       (effects (font (size 1.27 1.27)) hide)
     )
+    (property "LCSC Part" "0" (at 85.09 93.98 0)
+      (effects (font (size 1.27 1.27)) hide)
+    )
     (pin "1")
     (pin "2")
@@
       (effects (font (size 1.27 1.27)) hide)
     )
-    (property "LCSC Part" "C52923" (at 26.67 175.26 0)
+    (property "LCSC Part" "C15849" (at 26.67 175.26 0)
       (effects (font (size 1.27 1.27)) hide)
     )
@@
       (effects (font (size 1.27 1.27)))
     )
-    (property "Footprint" "Resistor_SMD:R_0805_2012Metric" (at 52.07 176.53 0)
+    (property "Footprint" "Resistor_SMD:R_0603_1608Metric" (at 52.07 176.53 0)
       (effects (font (size 1.27 1.27)) hide)
     )
@@
       (effects (font (size 1.27 1.27)) hide)
     )
-    (property "LCSC Part" "" (at 93.98 45.72 0)
+    (property "LCSC Part" "0" (at 93.98 45.72 0)
       (effects (font (size 1.27 1.27)) hide)
     )
@@
     (property "Arrow Price/Stock" "https://www.arrow.com/en/products/bq24196rger/texas-instruments?region=nac" (at 167.64 1048.26 0)
       (effects (font (size 1.27 1.27)) (justify left top) hide)
+    )
+    (property "LCSC Part" "C117006" (at 135.89 63.5 0)
+      (effects (font (size 1.27 1.27)) hide)
     )
     (pin "1")
@@
       (effects (font (size 1.27 1.27)) hide)
     )
-    (property "LCSC Part" "" (at 38.1 177.8 0)
+    (property "LCSC Part" "0" (at 38.1 177.8 0)
       (effects (font (size 1.27 1.27)) hide)
     )
@@
       (effects (font (size 1.27 1.27)) hide)
     )
-    (property "LCSC Part" "" (at 158.75 35.56 0)
+    (property "LCSC Part" "0" (at 158.75 35.56 0)
       (effects (font (size 1.27 1.27)) hide)
     )
@@
       (effects (font (size 1.27 1.27)) hide)
     )
-    (property "LCSC Part" "" (at 255.27 31.75 0)
+    (property "LCSC Part" "0" (at 255.27 31.75 0)
       (effects (font (size 1.27 1.27)) hide)
     )
@@
       (effects (font (size 1.27 1.27)) hide)
     )
-    (property "LCSC Part" "" (at 196.85 31.75 0)
-      (effects (font (size 1.27 1.27)) hide)
-    )
+    (property "LCSC Part" "0" (at 196.85 31.75 0)
+      (effects (font (size 1.27 1.27)) hide)
+    )
