File: Hardware/Version 2.1/VariometerV2.2.1/Power.kicad_sch (KiCad schematic)
At the start: 44 parts, among them IC3 BQ24196RGER, IC4 TPS22916CNYFPR, IC5 TPS73701DCQR, J8 LED_CHRG, Q1 AO3401A, Q2 AO3401A, Q3 AO3400A

Commit message: PCB Work
Parts:
- R16: value 360R -> 270R; LCSC Part C25194 -> C22966
Other:
- note added: "Imax = 1V/R * 530 2A"
- note removed: "Imax = 1V/R * 530 1.47A"
Changed lines of the file:
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@@
     (effects (font (size 1.27 1.27)) (justify left bottom))
   )
-  (text "Imax = 1V/R * 530\n1.47A" (at 168.91 88.9 0)
+  (text "Imax = 1V/R * 530\n2A" (at 168.91 88.9 0)
     (effects (font (size 1.27 1.27)) (justify left bottom))
   )
@@
       (effects (font (size 1.27 1.27)))
     )
-    (property "Value" "360R" (at 152.4 85.09 90)
+    (property "Value" "270R" (at 152.4 85.09 90)
       (effects (font (size 1.27 1.27)))
     )
@@
       (effects (font (size 1.27 1.27)) hide)
     )
-    (property "LCSC Part" "C25194" (at 152.4 87.63 0)
-      (effects (font (size 1.27 1.27)) hide)
-    )
+    (property "LCSC Part" "C22966" (at 152.4 87.63 0)
+      (effects (font (size 1.27 1.27)) hide)
+    )
