File: Hardware/Version 2.1/VariometerV2.2.1/VariometerV2.2.1.kicad_pcb (KiCad board)
At the start: 4 copper layers, 91 x 70.5 mm, 161 parts, among them IC1 ESP32-S3-WROOM, IC3 BQ24196RGER, IC4 TPS22916CNYFPR, IC5 TPS73701DCQR, J1 USB_C_Receptacle_USB2.0, J11 LED_CHRG, J2 Conn_01x02, J4 FFC24/0.5MM, J5 U.FL-R-SMT(01), J7 Conn_01x02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

Commit message: PCb Layout done
Parts:
- removed J11: LED_CHRG, Connector_PinHeader_2.54mm:PinHeader_2x01_P2.54mm_Vertical
- removed R14: 1k, Resistor_SMD:R_0603_1608Metric
- removed SW1, SW2: Switch_SW_Push, Button_Switch_THT:SW_PUSH_6mm
- removed TP7: TP_BCLK, TestPoint:TestPoint_Pad_D1.5mm
- removed TP8: TP_LRCLK, TestPoint:TestPoint_Pad_D1.5mm
- removed TP9: TP_DIN, TestPoint:TestPoint_Pad_D1.5mm
- added C51: 1uF, Capacitor_SMD:C_0603_1608Metric, F.Cu at (148.1, 76.8)
- added J6: SW, MainLibrary:PTS636SM25FSMTRLFS, F.Cu at (165.5, 97.2)
- added J9: SW, MainLibrary:PTS636SM25FSMTRLFS, F.Cu at (177.0, 97.4)
- moved H2 183.1 mm to (192.1, 118.3)
- moved C38 174.6 mm to (170.2, 53.1), turned to 180 degrees
- moved C37 174.6 mm to (172.5, 53.1), turned to 0 degrees
- moved U6 173.0 mm to (179.3, 55.9)
- moved U5 173.0 mm to (171.0, 56.0), turned to 180 degrees
- moved C41 172.0 mm to (182.7, 57.8)
- moved C40 171.7 mm to (183.1, 55.1), turned to 90 degrees
- moved C39 168.3 mm to (176.1, 56.3), turned to -90 degrees
- moved TP4 163.6 mm to (187.1, 54.7)
- moved H3 160.0 mm to (192.2, 54.6)
- moved C35 158.7 mm to (178.4, 88.3), turned to -90 degrees
- moved TP3 158.2 mm to (187.1, 58.1)
- moved R36 156.3 mm to (175.9, 85.3), turned to 180 degrees
- moved U4 154.3 mm to (176.1, 88.1), turned to -90 degrees
- moved C36 153.5 mm to (176.1, 90.6), turned to 180 degrees
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Connections:
- IC3 pad 3: /Power/~{PG} -> unconnected-(IC3-~{PG}-Pad3)

Commit message: PCb Work...
Parts:
- moved TP3 10.7 mm to (197.1, 62.1)
- moved TP4 10.7 mm to (197.1, 58.6)
- moved C40 10.6 mm to (193.0, 58.8)
- moved C41 10.6 mm to (192.6, 61.5)
- moved U6 10.6 mm to (189.2, 59.6)
- moved C39 10.6 mm to (185.9, 60.0)
- moved R38 10.1 mm to (180.5, 69.2)
- moved U5 10.1 mm to (176.9, 64.3)
- moved C37 10.1 mm to (178.4, 61.4)
- moved C38 10.1 mm to (176.1, 61.4)
- moved R37 10.1 mm to (178.2, 69.2)
- moved C33 9.01 mm to (186.1, 68.1)
- moved R35 8.30 mm to (197.5, 75.2)
- moved D3 7.80 mm to (196.9, 66.9)
- moved L3 7.80 mm to (190.9, 67.1)
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Other:
- board size 91 x 70.5 mm -> 95.9 x 70.5 mm

Commit message: WRL File
Parts:
- moved JP1 42.4 mm to (131.3, 105.9)
- moved R41 42.2 mm to (126.4, 105.7)
- moved C42 39.5 mm to (129.7, 114.3)
- moved C43 39.5 mm to (130.0, 111.4)
- moved J2 39.5 mm to (134.4, 119.1)
- moved U7 39.5 mm to (133.3, 112.2)
- moved D3 38.8 mm to (196.3, 105.6)
- moved L3 36.2 mm to (189.6, 103.3)
- moved D4 30.3 mm to (182.5, 103.3)
- moved C33 30.2 mm to (180.4, 97.9)
- moved D5 29.1 mm to (179.8, 103.1)
- moved R35 25.3 mm to (196.2, 100.5)
- moved C34 24.2 mm to (183.8, 97.5)
- moved Q4 23.8 mm to (188.6, 97.1)
- moved R34 23.7 mm to (193.1, 97.0)
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Other:
- board size 95.9 x 70.5 mm -> 94.7 x 69.1 mm

Commit message: Routing ..
Parts:
- added C52: 10uF, Capacitor_SMD:C_0603_1608Metric, F.Cu at (181.8, 92.1)
- J7: footprint Connector_JST:JST_PH_B2B-PH-K_1x02_P2.00mm_Vertical -> Connector_JST:JST_PH_S2B-PH-K_1x02_P2.00mm_Horizontal
- moved R13 17.8 mm to (122.0, 71.7)
- moved J8 17.5 mm to (123.4, 74.5)
- moved R43 15.4 mm to (131.8, 63.6), turned to 0 degrees
- moved TP3 15.2 mm to (181.8, 65.8)
- moved R42 13.3 mm to (131.9, 65.6), turned to 180 degrees
- moved R19 12.3 mm to (166.0, 86.0), turned to 90 degrees
- moved L1 12.2 mm to (120.7, 58.9)
- moved R44 11.2 mm to (141.3, 119.5), turned to 90 degrees
- moved R45 10.8 mm to (143.1, 119.5)
- moved C47 10.8 mm to (144.4, 119.5)
- moved TP1 9.40 mm to (156.1, 89.7), turned to 180 degrees
- moved R18 8.36 mm to (157.9, 83.3), turned to 0 degrees
- moved J7 8.36 mm to (130.4, 55.1)
- moved Q3 8.24 mm to (162.9, 89.8), turned to 0 degrees
- moved C39 6.72 mm to (189.0, 65.7), turned to 0 degrees
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Routing:
- net +3.1V_UNSW: track 0.00 -> 132.1 mm, vias 0 -> 8
- net +BATT: track 0.00 -> 109.3 mm, vias 0 -> 4
- net BUTTON_1: track 0.00 -> 89.1 mm, vias 0 -> 4
- net BUTTON_2: track 0.00 -> 82.0 mm, vias 0 -> 6
- net I2C2_SDA: track 0.00 -> 75.1 mm, vias 0 -> 6
- net I2C2_SCL: track 0.00 -> 70.4 mm, vias 0 -> 4
- net USB_CC1: track 0.00 -> 69.6 mm, vias 0 -> 2
- net +5V: track 0.00 -> 66.6 mm, vias 0 -> 4
- net USB_CC2: track 0.00 -> 63.0 mm, vias 0 -> 3
- net SD_CMD: track 0.00 -> 62.8 mm
- net SD_DAT3: track 0.00 -> 62.3 mm, vias 0 -> 3
- net SD_DAT2: track 0.00 -> 61.7 mm, vias 0 -> 2
- net SD_DAT0: track 0.00 -> 55.3 mm, vias 0 -> 3
- net SD_DAT1: track 0.00 -> 55.2 mm, vias 0 -> 3
- net BUTTON_4: track 0.00 -> 53.7 mm, vias 0 -> 2
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- added copper zone on F.Cu, net +3.1V_SW
- added copper zone on In2.Cu, net +3.1V_SW
- added copper zone on F.Cu, net +3.1V_UNSW
- added copper zone on F.Cu, net +5V
- added copper zone on F.Cu, net +BATT
- added copper zone on F.Cu, net /Power/SYS
- added copper zone on F.Cu, net GND
- added copper zone on In1.Cu, net GND
- added copper zone on F.Cu, net VCC

Commit message: PCB Routing Done
Parts:
- moved TP2 19.0 mm to (174.3, 113.8)
- moved C44 15.1 mm to (119.4, 59.1), turned to -90 degrees
- moved C14 10.9 mm to (121.3, 60.3)
- moved C30 10.4 mm to (188.7, 75.9), turned to 0 degrees
- moved C31 9.49 mm to (187.9, 82.9)
- moved C32 9.26 mm to (189.4, 83.0)
- moved C29 6.09 mm to (186.3, 73.8), turned to 0 degrees
- moved R43 5.87 mm to (137.0, 60.8)
- moved R42 5.87 mm to (137.1, 62.8)
- moved C33 5.57 mm to (184.7, 101.5)
- moved C28 4.12 mm to (186.3, 72.6), turned to 0 degrees
- moved L1 4.11 mm to (119.0, 62.6), turned to 90 degrees
- moved C27 2.33 mm to (186.4, 71.3), turned to 0 degrees
- moved R26 2.31 mm to (114.3, 83.6)
- moved C12 2.03 mm to (116.5, 62.6)
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Routing:
- net GND: track 12.9 -> 186.8 mm, vias 21 -> 146
- net EN: track 0.00 -> 67.1 mm, vias 0 -> 2
- net +3.1V_UNSW: track 132.1 -> 185.5 mm, vias 8 -> 12
- net POSW_EN: track 0.00 -> 49.4 mm, vias 0 -> 2
- net +3.1V_SW: track 14.0 -> 61.6 mm, vias 5 -> 35
- net CHARG_INT: track 3.82 -> 49.2 mm, vias 0 -> 4
- net IO0: track 0.00 -> 27.3 mm, vias 0 -> 2
- net /Power/REGN: track 9.36 -> 36.1 mm, vias 2 -> 5
- net VCC: track 34.0 -> 56.1 mm, vias 2 -> 3
- net Net-(IC5-FB): track 1.86 -> 19.3 mm, vias 0 -> 2
- net Net-(U8-1PPS): track 0.00 -> 13.7 mm, vias 0 -> 2
- net Net-(J4-VGL): track 11.2 -> 2.86 mm
- net Net-(J4-VGH): track 12.4 -> 4.48 mm
- net /Power/SYS: track 32.1 -> 39.7 mm
- net Net-(R44-Pad2): track 10.9 -> 17.4 mm
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Other:
- board text added: "3.1V"
- board text added: "BAT+"
- board text added: "BATTERY"
- board text added: "DISPLAY"
- board text added: "GPS-ANTENNA"
- board text added: "SCL1"
- board text added: "SCL2"
- board text added: "SD-CARD"
- board text added: "SDA1"
- board text added: "SDA2"
- board text added: "SPEAKER"
- board text added: "SYS"
- board text added: "USB"
- board text added: "VARIOMETER | V.2.1"

Commit message: New 3D File
Parts:
- SW3, SW4, SW5, SW6: footprint Button_Switch_THT:SW_PUSH_6mm -> Button_Switch_THT:SW_PUSH_6mm_H4.3mm
Other:
- board text added: "+"
- board text added: "-"
Changed lines of the file:
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@@
     )
   )
-  (footprint "Button_Switch_THT:SW_PUSH_6mm" (layer "F.Cu")
+  (footprint "Button_Switch_THT:SW_PUSH_6mm_H4.3mm" (layer "F.Cu")
     (at 186.1554 115.3816 180)
-    (descr "https://www.omron.com/ecb/products/pdf/en-b3f.pdf")
+    (descr "tactile push button, 6x6mm e.g. PHAP33xx series, height=4.3mm")
     (tags "tact sw push 6mm")
     (property "LCSC Part" "")
@@
     (property "Sheetname" "Peripherals")
     (attr through_hole)
-    (fp_text reference "SW6" (at 3.25 -2) (layer "F.SilkS")
+    (fp_text reference "SW6" (at 3.25 -2 180) (layer "F.SilkS")
         (effects (font (size 1 1) (thickness 0.15)))
     )
-    (fp_text value "BTN1" (at 3.75 6.7) (layer "F.Fab")
+    (fp_text value "BTN1" (at 3.75 6.7 180) (layer "F.Fab")
         (effects (font (size 1 1) (thickness 0.15)))
     )
-    (fp_text user "${REFERENCE}" (at 3.25 2.25) (layer "F.Fab")
+    (fp_text user "${REFERENCE}" (at 3.25 2.25 180) (layer "F.Fab")
         (effects (font (size 1 1) (thickness 0.15)))
     )
@@
     (pad "2" thru_hole circle (at 6.5 4.5 270) (size 2 2) (drill 1.1) (layers "*.Cu" "*.Mask")
       (net 109 "Net-(R48-Pad2)") (pinfunction "2") (pintype "passive"))
-    (model "${KICAD6_3DMODEL_DIR}/Button_Switch_THT.3dshapes/SW_PUSH_6mm.wrl"
+    (model "${KICAD6_3DMODEL_DIR}/Button_Switch_THT.3dshapes/SW_PUSH_6mm_H4.3mm.wrl"
       (offset (xyz 0 -4.5 -1.5))
       (scale (xyz 1 1 1))
@@
     )
   )
-  (footprint "Button_Switch_THT:SW_PUSH_6mm" (layer "F.Cu")
+  (footprint "Button_Switch_THT:SW_PUSH_6mm_H4.3mm" (layer "F.Cu")
     (at 145.6932 115.6356 180)
-    (descr "https://www.omron.com/ecb/products/pdf/en-b3f.pdf")
+    (descr "tactile push button, 6x6mm e.g. PHAP33xx series, height=4.3mm")
     (tags "tact sw push 6mm")
     (property "LCSC Part" "")
@@
     (property "Sheetname" "Peripherals")
     (attr through_hole)
-    (fp_text reference "SW4" (at 3.25 -2) (layer "F.SilkS")
+    (fp_text reference "SW4" (at 3.25 -2 180) (layer "F.SilkS")
         (effects (font (size 1 1) (thickness 0.15)))
     )
-    (fp_text value "BTN1" (at 3.75 6.7) (layer "F.Fab")
+    (fp_text value "BTN1" (at 3.75 6.7 180) (layer "F.Fab")
         (effects (font (size 1 1) (thickness 0.15)))
     )
-    (fp_text user "${REFERENCE}" (at 3.25 2.25) (layer "F.Fab")
+    (fp_text user "${REFERENCE}" (at 3.25 2.25 180) (layer "F.Fab")
         (effects (font (size 1 1) (thickness 0.15)))
     )
@@
     (pad "2" thru_hole circle (at 6.5 4.5 270) (size 2 2) (drill 1.1) (layers "*.Cu" "*.Mask")
       (net 107 "Net-(R44-Pad2)") (pinfunction "2") (pintype "passive"))
-    (model "${KICAD6_3DMODEL_DIR}/Button_Switch_THT.3dshapes/SW_PUSH_6mm.wrl"
-      (offset (xyz 0 -4.5 -1.5))
+    (model "${KICAD6_3DMODEL_DIR}/Button_Switch_THT.3dshapes/SW_PUSH_6mm_H4.3mm.wrl"
+      (offset (xyz 0 -4.5 -2))
       (scale (xyz 1 1 1))
       (rotate (xyz 180 0 0))
@@
       (net 8 "+5V") (pinfunction "B") (pintype "passive"))
   )
-  (footprint "Button_Switch_THT:SW_PUSH_6mm" (layer "F.Cu")
+  (footprint "Button_Switch_THT:SW_PUSH_6mm_H4.3mm" (layer "F.Cu")
     (at 125.5764 115.6864 180)
-    (descr "https://www.omron.com/ecb/products/pdf/en-b3f.pdf")
+    (descr "tactile push button, 6x6mm e.g. PHAP33xx series, height=4.3mm")
     (tags "tact sw push 6mm")
     (property "LCSC Part" "")
@@
     (property "Sheetname" "Peripherals")
     (attr through_hole)
-    (fp_text reference "SW3" (at 3.25 -2) (layer "F.SilkS")
+    (fp_text reference "SW3" (at 3.25 -2 180) (layer "F.SilkS")
         (effects (font (size 1 1) (thickness 0.15)))
     )
-    (fp_text value "BTN1" (at 3.75 6.7) (layer "F.Fab")
+    (fp_text value "BTN1" (at 3.75 6.7 180) (layer "F.Fab")
         (effects (font (size 1 1) (thickness 0.15)))
     )
-    (fp_text user "${REFERENCE}" (at 3.25 2.25) (layer "F.Fab")
+    (fp_text user "${REFERENCE}" (at 3.25 2.25 180) (layer "F.Fab")
         (effects (font (size 1 1) (thickness 0.15)))
     )
@@
     (pad "2" thru_hole circle (at 6.5 4.5 270) (size 2 2) (drill 1.1) (layers "*.Cu" "*.Mask")
       (net 101 "Net-(R5-Pad2)") (pinfunction "2") (pintype "passive"))
-    (model "${KICAD6_3DMODEL_DIR}/Button_Switch_THT.3dshapes/SW_PUSH_6mm.wrl"
+    (model "${KICAD6_3DMODEL_DIR}/Button_Switch_THT.3dshapes/SW_PUSH_6mm_H4.3mm.wrl"
       (offset (xyz 0 -4.5 -1.5))
       (scale (xyz 1 1 1))
@@
     (pad "2" thru_hole oval (at 0 2.54 270) (size 1.7 1.7) (drill 1) (layers "*.Cu" "*.Mask")
       (net 78 "AUDIO_OUTP") (pinfunction "Pin_2") (pintype "passive"))
-    (model "${KICAD6_3DMODEL_DIR}/Connector_PinHeader_2.54mm.3dshapes/PinHeader_1x02_P2.54mm_Vertical.wrl"
+    (model "${KICAD6_3DMODEL_DIR}/Connector_PinHeader_2.54mm.3dshapes/PinHeader_1x02_P2.54mm_Vertical.wrl" hide
       (offset (xyz 0 0 0))
       (scale (xyz 1 1 1))
@@
     )
   )
-  (footprint "Button_Switch_THT:SW_PUSH_6mm" (layer "F.Cu")
+  (footprint "Button_Switch_THT:SW_PUSH_6mm_H4.3mm" (layer "F.Cu")
     (at 165.9116 115.5086 180)
-    (descr "https://www.omron.com/ecb/products/pdf/en-b3f.pdf")
+    (descr "tactile push button, 6x6mm e.g. PHAP33xx series, height=4.3mm")
     (tags "tact sw push 6mm")
     (property "LCSC Part" "")
@@
     (property "Sheetname" "Peripherals")
     (attr through_hole)
-    (fp_text reference "SW5" (at 3.25 -2) (layer "F.SilkS")
+    (fp_text reference "SW5" (at 3.25 -2 180) (layer "F.SilkS")
         (effects (font (size 1 1) (thickness 0.15)))
     )
-    (fp_text value "BTN1" (at 3.75 6.7) (layer "F.Fab")
+    (fp_text value "BTN1" (at 3.75 6.7 180) (layer "F.Fab")
         (effects (font (size 1 1) (thickness 0.15)))
     )
-    (fp_text user "${REFERENCE}" (at 3.25 2.25) (layer "F.Fab")
+    (fp_text user "${REFERENCE}" (at 3.25 2.25 180) (layer "F.Fab")
         (effects (font (size 1 1) (thickness 0.15)))
     )
@@
     (pad "2" thru_hole circle (at 6.5 4.5 270) (size 2 2) (drill 1.1) (layers "*.Cu" "*.Mask")
       (net 108 "Net-(R46-Pad2)") (pinfunction "2") (pintype "passive"))
-    (model "${KICAD6_3DMODEL_DIR}/Button_Switch_THT.3dshapes/SW_PUSH_6mm.wrl"
-      (offset (xyz 0 -4.5 -1))
+    (model "${KICAD6_3DMODEL_DIR}/Button_Switch_THT.3dshapes/SW_PUSH_6mm_H4.3mm.wrl"
+      (offset (xyz 0 -4.5 -1.5))
       (scale (xyz 1 1 1))
-      (rotate (xyz -180 0 0))
+      (rotate (xyz 180 0 0))
     )
   )
@@
   (gr_line (start 174.1678 58.801) (end 136.0678 58.801)
     (stroke (width 0.1) (type default)) (layer "Edge.Cuts"))
+  (gr_text "-" (at 137.81 119.26) (layer "B.SilkS")
+    (effects (font (size 1 1) (thickness 0.15)) (justify left bottom mirror))
+  )
   (gr_text "GPS-ANTENNA" (at 156.82 100.98) (layer "B.SilkS")
     (effects (font (size 1 1) (thickness 0.15)) (justify left bottom mirror))
   )
+  (gr_text "+" (at 129.68 119.14) (layer "B.SilkS")
+    (effects (font (size 1 1) (thickness 0.15)) (justify left bottom mirror))
+  )
+  (gr_text "-" (at 135.85 54.89) (layer "B.SilkS")
+    (effects (font (size 1 1) (thickness 0.15)) (justify left bottom mirror))
+  )
+  (gr_text "+" (at 128.14 54.6) (layer "B.SilkS")
+    (effects (font (size 1 1) (thickness 0.15)) (justify left bottom mirror))
+  )

Commit message: Finish PCB
Parts:
- C7, C9: footprint Capacitor_SMD:C_0402_1005Metric -> Capacitor_SMD:C_0603_1608Metric
- R17, R18: footprint Resistor_SMD:R_0805_2012Metric -> Resistor_SMD:R_0603_1608Metric
- R7: footprint Inductor_SMD:L_0603_1608Metric -> Resistor_SMD:R_0603_1608Metric
- moved C9 4.06 mm to (141.4, 96.4)
- moved C7 1.00 mm to (139.7, 104.7)
Routing:
- net +3.1V_UNSW: track 185.5 -> 188.8 mm
- net Net-(IC3-SW1): track 4.97 -> 6.86 mm
- net +3.1V_SW: vias 35 -> 34
Other:
- outline, holes or cut-outs redrawn
- board text added: "GPS"
- board text added: "JLCJLCJLCJLC"

Commit message: PCB Work
Parts:
- moved C13 6.15 mm to (124.1, 57.9)
Routing:
- net +BATT: track 109.3 -> 102.7 mm
- net GND: track 186.6 -> 187.3 mm
