File: Hardware/Version 2.1/VariometerV2.2.1/VariometerV2.2.1.kicad_pcb (KiCad board)
At the start: 4 copper layers, 94.7 x 69.1 mm, 158 parts, among them IC1 ESP32-S3-WROOM, IC3 BQ24196RGER, IC4 TPS22916CNYFPR, IC5 TPS73701DCQR, J1 USB_C_Receptacle_USB2.0, J2 Conn_01x02, J4 FFC24/0.5MM, J5 U.FL-R-SMT(01), J6 SW, J7 Conn_01x02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

Commit message: Fix Screen Connector PCB
Parts:
- removed J4: FFC24/0.5MM, MainLibrary:FH12-24S-0.5SH_55_
- added J10: Conn_01x24_MountingPin, Connector_FFC-FPC:Hirose_FH12-24S-0.5SH_1x24-1MP_P0.50mm_Horizontal, F.Cu at (194.4, 75.8)
- R16: value 360R -> 270R
- moved C31 14.7 mm to (190.3, 68.4), turned to -90 degrees
- moved C32 14.6 mm to (188.8, 68.4), turned to -90 degrees
- moved C23 14.6 mm to (182.3, 81.9), turned to 90 degrees
- moved C25 13.7 mm to (184.0, 82.3), turned to 90 degrees
- moved C26 13.1 mm to (185.6, 82.4), turned to 90 degrees
- moved C27 11.0 mm to (187.0, 82.4), turned to 90 degrees
- moved C28 9.99 mm to (188.5, 82.3), turned to 90 degrees
- moved C30 9.63 mm to (189.4, 85.5)
- moved C29 9.44 mm to (190.4, 82.3), turned to 90 degrees
- moved C24 8.47 mm to (188.1, 77.4), turned to 0 degrees
- moved R34 2.57 mm to (195.3, 95.8), turned to 90 degrees
Connections:
- C23 pad 2: /Screen/PREVGL -> Net-(J10-Pin_7)
- C24 pad 2: Net-(J4-VCOM) -> +3.1V_SW
- C26 pad 2: /Screen/PREVGH -> Net-(J10-Pin_5)
- C27 pad 2: Net-(J4-VSH) -> /Screen/PREVGH
- C29 pad 2: Net-(J4-VDD) -> /Screen/PREVGL
- C30 pad 2: +3.1V_SW -> Net-(J10-Pin_1)
Routing:
- net /Screen/GDR: track 31.4 -> 47.0 mm, vias 4 -> 6
- net Net-(J10-Pin_7): track 0.00 -> 11.4 mm
- net /Screen/RESE: track 23.3 -> 34.1 mm, vias 2 -> 4
- net /Screen/PREVGL: track 47.8 -> 37.3 mm
- net Net-(J10-Pin_5): track 0.00 -> 7.93 mm
- net Net-(J4-VSH): track 6.19 -> 0.00 mm
- net /Screen/PREVGH: track 40.2 -> 34.2 mm, vias 0 -> 2
- net Net-(J4-VDD): track 5.65 -> 0.00 mm
- net Net-(J10-Pin_1): track 0.00 -> 4.94 mm
- net Net-(J10-Pin_6): track 5.25 -> 9.67 mm
- net Net-(J10-Pin_20): track 2.86 -> 6.00 mm
- net Net-(J4-VCOM): track 2.34 -> 0.00 mm
- net LCD_DC: track 31.8 -> 30.0 mm
- net LCD_BUSY: track 30.6 -> 29.1 mm
- net Net-(J10-Pin_3): track 6.01 -> 4.58 mm
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Other:
- board text added: "Screen"
- board text removed: "DISPLAY"
