File: Hardware/Version 2.1/VariometerV2.2.1/Screen.kicad_sch (KiCad schematic)
At the start: 0 parts

Commit message: Working on PCB
Parts:
- added C23, C24, C25, C26, C27, C28, C29, C30, C31, C32, C34: 1uF, symbol Device:C_Small
- added C33: 4.7Uf, symbol Device:C_Small
- added D1 (x3): B5819W SL, Diode_SMD:D_SOD-123, symbol Device:D_Schottky_Small
- added J9: PFC24/0.5MM, symbol Main_LibraryVario:PFC24/0.5MM
- added L2: 68uH, symbol Device:L_Small
- added Q3: AO3400A, Package_TO_SOT_SMD:SOT-23, symbol Transistor_FET:AO3400A
- added R34: 0.47R, symbol Device:R_Small
- added R35: 10k, symbol Device:R_Small
Connections:
- new net: C24.2, J9.24 (VCOM)
- new net: C27.2, J9.20 (VSH)
- new net: C31.2, J9.5 (VGH)
- new net: C28.2, J9.19 (VPP)
- new net: C34.1, D1.2 (A), L2.2, Q3.3 (D)
- new net: C34.2, D1.1 (K), D1.2 (A)
- new net: C29.2, J9.18 (VDD)
- new net: C25.2, J9.22 (VSL)
- new net: C32.2, J9.4 (VGL)
- new net +3.1V_SW: C30.2, C33.1, J9.15 (VDDIO), J9.16 (VCI), L2.1
- new net BS: J9.8 (BS)
- new net GDR: J9.2 (GDR), Q3.1 (G), R35.2
- new net GND: C23.1, C24.1, C25.1, C26.1, C27.1, C28.1, C29.1, C30.1, C31.1, C32.1, C33.2, D1.1 (K), J9.17 (VSS), R34.1, R35.1
- new net LCD_BUSY: J9.9 (BUSY)
- new net LCD_CLK: J9.13 (SCLK)
- new net LCD_CS: J9.12 (CS)
- new net LCD_DC: J9.11 (D/C)
- new net LCD_DIN: J9.14 (SDI)
- new net LCD_RST: J9.10 (RST)
- new net PREVGH: C26.2, D1.1 (K), J9.21 (PREVGH)
- new net PREVGL: C23.2, D1.2 (A), J9.23 (PREVGL)
- new net RESE: J9.3 (RESE), Q3.2 (S), R34.2
- no-connect marks 0 -> 3
Other:
- note added: "?"
- note added: "Screen Connector"
- title: (none) -> Screen

Commit message: Update Schematics
Parts:
- removed J9: PFC24/0.5MM, symbol Main_LibraryVario:PFC24/0.5MM
- added J4: FFC24/0.5MM, MainLibrary:FH12-24S-0.5SH_55_, symbol Main_LibraryVario:FFC24/0.5MM
- C23, C24, C25, C26, C27, C28, C29, C31, C32: footprint (none) -> Capacitor_SMD:C_0402_1005Metric
- C30: value 1uF -> 10uF; footprint (none) -> Capacitor_SMD:C_0603_1608Metric
- C33: footprint (none) -> Capacitor_SMD:C_0603_1608Metric
- C34: value 1uF -> 4.7uF; footprint (none) -> Capacitor_SMD:C_0603_1608Metric
- Q3: footprint Package_TO_SOT_SMD:SOT-23 -> (none)
Connections:
- net +3.1V_SW: now also J4.15 (VDDIO), J4.16 (VCI)
- net BS: now also J4.8 (BS)
- net GDR: now also J4.2 (GDR)
- net GND: now also J4.17 (VSS), J4.25 (SHIELD), J4.26 (SHIELD)
- net LCD_BUSY: now also J4.9 (BUSY)
- net LCD_CLK: now also J4.13 (SCLK)
- net LCD_CS: now also J4.12 (CS)
- net LCD_DC: now also J4.11 (D/C)
- net LCD_DIN: now also J4.14 (SDI)
- net LCD_RST: now also J4.10 (RST)
- net PREVGH: now also J4.21 (PREVGH)
- net PREVGL: now also J4.23 (PREVGL)
- net RESE: now also J4.3 (RESE)
- net at C24.2: now also J4.24 (VCOM)
- net at C27.2: now also J4.20 (VSH)
- net at C31.2: now also J4.5 (VGH)
- net at C28.2: now also J4.19 (VPP)
- net at C29.2: now also J4.18 (VDD)
- net at C25.2: now also J4.22 (VSL)
- net at C32.2: now also J4.4 (VGL)
Other:
- note removed: "?"

Commit message: Working on PCB
Parts:
- Q3: footprint (none) -> Package_TO_SOT_SMD:SOT-23
- R35: footprint (none) -> Resistor_SMD:R_0603_1608Metric
Changed lines of the file:
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@@
       (effects (font (size 1.27 1.27)))
     )
-    (property "Footprint" "" (at 83.82 85.09 0)
+    (property "Footprint" "Resistor_SMD:R_0603_1608Metric" (at 83.82 85.09 0)
       (effects (font (size 1.27 1.27)) hide)
     )
@@
       (effects (font (size 1.27 1.27)) (justify left))
     )
-    (property "Footprint" "" (at 106.68 83.185 0)
+    (property "Footprint" "Package_TO_SOT_SMD:SOT-23" (at 106.68 83.185 0)
       (effects (font (size 1.27 1.27) italic) (justify left) hide)
     )

Commit message: PCB
Parts:
- removed L2: 68uH, symbol Device:L_Small
- added L3: SRN6045TA-680M, MainLibrary:SRN6045TA, symbol Main_LibraryVario:SRN6045TA-680M
- C23, C24, C25, C26, C27, C28, C29, C31, C32: LCSC Part (none) -> C52923
- C30: LCSC Part (none) -> C19702
- C33: value 4.7Uf -> 4.7uF; LCSC Part (none) -> C19666
- C34: LCSC Part (none) -> C19666
- D1: JLCPCB Part # C8598 -> (none); LCSC Part (none) -> C8598
- J4: LCSC Part (none) -> C202112
- Q3: JLCPCB Part # C20917 -> (none); LCSC Part (none) -> C20917
- R34: footprint (none) -> Resistor_SMD:R_0805_2012Metric
- R35: LCSC Part (none) -> C25804
Connections:
- net +3.1V_SW: now also L3.1
- net at C34.1, D1.2 (A), Q3.3 (D): now also L3.2
Other:
- moved on the sheet: C33

Commit message: Start on pcb
Connections:
- net BS is gone; now on net GND: J4.8 (BS)
Changed lines of the file:
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@@
     (stroke (width 0) (type default))
   )
-  (wire (pts (xy 204.47 73.66) (xy 209.55 73.66))
+  (wire (pts (xy 194.31 73.66) (xy 209.55 73.66))
     (stroke (width 0) (type default))
   )
@@
   )
   (label "PREVGH" (at 185.42 106.68 0) (fields_autoplaced)
-    (effects (font (size 1.27 1.27)) (justify left bottom))
-  )
-  (label "BS" (at 204.47 73.66 0) (fields_autoplaced)
     (effects (font (size 1.27 1.27)) (justify left bottom))
   )
@@
     )
   )
+  (symbol (lib_id "power:GND") (at 194.31 73.66 270) (unit 1)
+    (in_bom yes) (on_board yes) (dnp no) (fields_autoplaced)
+    (property "Reference" "#PWR0109" (at 187.96 73.66 0)
+      (effects (font (size 1.27 1.27)) hide)
+    )
+    (property "Value" "GND" (at 190.5 74.295 90)
+      (effects (font (size 1.27 1.27)) (justify right))
+    )
+    (property "Footprint" "" (at 194.31 73.66 0)
+      (effects (font (size 1.27 1.27)) hide)
+    )
+    (property "Datasheet" "" (at 194.31 73.66 0)
+      (effects (font (size 1.27 1.27)) hide)
+    )
+    (pin "1")
+    (instances
+      (project "VariometerV2.2.1"
+        (path "/9d9a2a31-8397-4ba2-ad51-8bee2c0fd904/523adc66-5baf-476b-9937-df31f7f6507b"
+          (reference "#PWR0109") (unit 1)
+        )
+      )
+    )
+  )
   (symbol (lib_id "Device:C_Small") (at 179.07 121.92 180) (unit 1)
     (in_bom yes) (on_board yes) (dnp no)
@@
   (symbol (lib_id "Main_LibraryVario:SRN6045TA-680M") (at 81.28 95.25 0) (unit 1)
     (in_bom yes) (on_board yes) (dnp no) (fields_autoplaced)
-    (property "Reference" "L3" (at 91.44 90.17 0)
+    (property "Reference" "L3" (at 91.44 88.9 0)
       (effects (font (size 1.27 1.27)))
     )
-    (property "Value" "SRN6045TA-680M" (at 91.44 92.71 0)
+    (property "Value" "SRN6045TA-680M" (at 91.44 91.44 0)
       (effects (font (size 1.27 1.27)))
     )

Commit message: Finish PCB
Parts:
- J4: LCSC Part C202112 -> C519265
- L3, R34: LCSC Part (none) -> 0
Changed lines of the file:
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@@
       (effects (font (size 1.27 1.27)) (justify left top) hide)
     )
-    (property "LCSC Part" "" (at 81.28 95.25 0)
+    (property "LCSC Part" "0" (at 81.28 95.25 0)
       (effects (font (size 1.27 1.27)) hide)
     )
@@
       (effects (font (size 1.27 1.27)) hide)
     )
-    (property "LCSC Part" "" (at 104.14 72.39 0)
+    (property "LCSC Part" "0" (at 104.14 72.39 0)
       (effects (font (size 1.27 1.27)) hide)
     )
@@
       (effects (font (size 1.27 1.27)) hide)
     )
-    (property "LCSC Part" "C202112" (at 215.9 71.12 0)
+    (property "LCSC Part" "C519265" (at 215.9 71.12 0)
       (effects (font (size 1.27 1.27)) hide)
     )

Commit message: Fix Screen Connector PCB
Parts:
- removed J4: FFC24/0.5MM, MainLibrary:FH12-24S-0.5SH_55_, symbol Main_LibraryVario:FFC24/0.5MM
- added J10: Conn_01x24_MountingPin, Connector_FFC-FPC:Hirose_FH12-24S-0.5SH_1x24-1MP_P0.50mm_Horizontal, symbol Connector_Generic_MountingPin:Conn_01x24_MountingPin
Connections:
- net +3.1V_SW: now also C24.2, J10.10 (Pin_10), J10.9 (Pin_9); no longer C30.2
- net GDR: now also J10.23 (Pin_23)
- net GND: now also J10.17 (Pin_17), J10.8 (Pin_8), J10.MP (MountPin)
- net LCD_BUSY: now also J10.16 (Pin_16)
- net LCD_CLK: now also J10.12 (Pin_12)
- net LCD_CS: now also J10.13 (Pin_13)
- net LCD_DC: now also J10.14 (Pin_14)
- net LCD_DIN: now also J10.11 (Pin_11)
- net LCD_RST: now also J10.15 (Pin_15)
- net PREVGH: now also C27.2, J10.4 (Pin_4); no longer C26.2
- net PREVGL: now also C29.2, J10.2 (Pin_2); no longer C23.2
- net RESE: now also J10.22 (Pin_22)
- net at C31.2: now also J10.21 (Pin_21)
- net at C28.2: now also J10.3 (Pin_3)
- net at C25.2: now also J10.6 (Pin_6)
- net at C32.2: now also J10.20 (Pin_20)
- new net: C30.2, J10.1 (Pin_1)
- new net: C26.2, J10.5 (Pin_5)
- new net: C23.2, J10.7 (Pin_7)
Other:
- moved on the sheet: C23, C24, C25, C26, C27, C28, C29, C30, C31, C32
